Commit message: Remove material from visual to not overload .dae file's colors.

File: urdf/ur_simulation_macro.xacro (robot description, xacro)
@@ -104,7 +104,4 @@
           <mesh filename="file://$(find ur_description)/meshes/${name}/visual/base.dae"/>
         </geometry>
-        <material name="${base_visual_material_name}">
-          <color rgba="${base_visual_material_color}"/>
-        </material>
       </visual>
       <collision>
@@ -124,7 +121,4 @@
           <mesh filename="file://$(find ur_description)/meshes/${name}/visual/shoulder.dae"/>
         </geometry>
-        <material name="${shoulder_visual_material_name}">
-          <color rgba="${shoulder_visual_material_color}"/>
-        </material>
       </visual>
       <collision>
@@ -144,7 +138,4 @@
           <mesh filename="file://$(find ur_description)/meshes/${name}/visual/upperarm.dae"/>
         </geometry>
-        <material name="${upper_arm_visual_material_name}">
-          <color rgba="${upper_arm_visual_material_color}"/>
-        </material>
       </visual>
       <collision>
@@ -164,7 +155,4 @@
           <mesh filename="file://$(find ur_description)/meshes/${name}/visual/forearm.dae"/>
         </geometry>
-        <material name="${forearm_visual_material_name}">
-          <color rgba="${forearm_visual_material_color}"/>
-        </material>
       </visual>
       <collision>
@@ -184,7 +172,4 @@
           <mesh filename="file://$(find ur_description)/meshes/${name}/visual/wrist1.dae"/>
         </geometry>
-        <material name="${wrist_1_visual_material_name}">
-          <color rgba="${wrist_1_visual_material_color}"/>
-        </material>
       </visual>
       <collision>
@@ -204,7 +189,4 @@
           <mesh filename="file://$(find ur_description)/meshes/${name}/visual/wrist2.dae"/>
         </geometry>
-        <material name="${wrist_2_visual_material_name}">
-          <color rgba="${wrist_2_visual_material_color}"/>
-        </material>
       </visual>
       <collision>
@@ -224,7 +206,4 @@
           <mesh filename="file://$(find ur_description)/meshes/${name}/visual/wrist3.dae"/>
         </geometry>
-        <material name="${wrist_3_visual_material_name}">
-          <color rgba="${wrist_3_visual_material_color}"/>
-        </material>
       </visual>
       <collision>
