Commit message: Add support for gpios, update MoveIt and ros2_control launching (#66)
* Add ur_msgs as dependency.

* Bare bone tool io controller.

* Register all non-joint interfaces.

* Fix typo.

* Configure state and command interfaces in gpio controller.

* Fix clang issue.

* Register needed services and publishers.

* Reorganize state and command interfaces for easier enumeration.

* Update licence.

* Include success check for io service.

* Fix ci.

* Publish data of interest.

* Clang tidy.

* Apply suggestions from code review

* Launch Arguments for xacro are working, not all params added

* Moved files and one step further with the Arguemnts

* Add launch for all version of UR robots

* Small updated from offline review

* Some rewrapping and testing GPIO controller.

* Reduce unintended changes

* Readme grammar check and minor re-org

* Minor comment and typo cleanup

* Reduce duplication of default launch args

* Initial add of moveit configs

* Added MoveIt configs and example launch file

* Remove unused mongodb node

* Enabled monogodb

* Add condistion check for dashboard client and start command for MoveIt.

* Added protection to add false joints

* Debug io controller and interfaces

* Use scaled controller in example

* Removed dashboard client node from default start

* Updated README and use fixed frame in MoveIt.

* [WIP] Hard-code launch config for UR5e

* RViz MoveIt plugin actually loads. Controllers do not.

* Revert changes and try correct MoveIt.

* Set speed scaling in percetange.

* Separete control and moveit launch files an correct MoveIt configuration

* Add again planning scene parameters

Co-authored-by: Lovro <lovro.ivanov@gmail.com>
Co-authored-by: AndyZe <zelenak@picknik.ai>

File: urdf/ur.ros2_control.xacro (robot description, xacro)
@@ -1,6 +1,6 @@
 <?xml version="1.0"?>
 <robot xmlns:xacro="http://www.ros.org/wiki/xacro">
-  <xacro:macro name="ur5_system_position_only" params="name prefix
-    use_fake_hardware:=^|false fake_sensor_commands:=^|false
+  <xacro:macro name="ur_ros2_control" params="name prefix
+    use_fake_hardware:=false fake_sensor_commands:=false
     script_filename output_recipe_filename
     input_recipe_filename tf_prefix
@@ -125,4 +125,102 @@
         <state_interface name="torque.z"/>
       </sensor>
+      <!-- NOTE The following are joints used only for testing with fake hardware and will change in the future -->
+      <joint name="speed_scaling">
+        <state_interface name="speed_scaling_factor"/>
+        <command_interface name="speed_scaling_factor_cmd"/>
+        <command_interface name="scaling_async_success"/>
+      </joint>
+      <joint name="gpio">
+        <command_interface name="standard_digital_output_cmd_0"/>
+        <command_interface name="standard_digital_output_cmd_1"/>
+        <command_interface name="standard_digital_output_cmd_2"/>
+        <command_interface name="standard_digital_output_cmd_3"/>
+        <command_interface name="standard_digital_output_cmd_4"/>
+        <command_interface name="standard_digital_output_cmd_5"/>
+        <command_interface name="standard_digital_output_cmd_6"/>
+        <command_interface name="standard_digital_output_cmd_7"/>
+        <command_interface name="standard_digital_output_cmd_8"/>
+        <command_interface name="standard_digital_output_cmd_9"/>
+        <command_interface name="standard_digital_output_cmd_10"/>
+        <command_interface name="standard_digital_output_cmd_11"/>
+        <command_interface name="standard_digital_output_cmd_12"/>
+        <command_interface name="standard_digital_output_cmd_13"/>
+        <command_interface name="standard_digital_output_cmd_14"/>
+        <command_interface name="standard_digital_output_cmd_15"/>
+        <command_interface name="standard_digital_output_cmd_16"/>
+        <command_interface name="standard_digital_output_cmd_17"/>
+        <command_interface name="standard_analog_output_cmd_0"/>
+        <command_interface name="standard_analog_output_cmd_1"/>
+        <command_interface name="io_async_success"/>
+        <state_interface name="digital_output_0"/>
+        <state_interface name="digital_output_1"/>
+        <state_interface name="digital_output_2"/>
+        <state_interface name="digital_output_3"/>
+        <state_interface name="digital_output_4"/>
+        <state_interface name="digital_output_5"/>
+        <state_interface name="digital_output_6"/>
+        <state_interface name="digital_output_7"/>
+        <state_interface name="digital_output_8"/>
+        <state_interface name="digital_output_9"/>
+        <state_interface name="digital_output_10"/>
+        <state_interface name="digital_output_11"/>
+        <state_interface name="digital_output_12"/>
+        <state_interface name="digital_output_13"/>
+        <state_interface name="digital_output_14"/>
+        <state_interface name="digital_output_15"/>
+        <state_interface name="digital_output_16"/>
+        <state_interface name="digital_output_17"/>
+        <state_interface name="digital_input_0"/>
+        <state_interface name="digital_input_1"/>
+        <state_interface name="digital_input_2"/>
+        <state_interface name="digital_input_3"/>
+        <state_interface name="digital_input_4"/>
+        <state_interface name="digital_input_5"/>
+        <state_interface name="digital_input_6"/>
+        <state_interface name="digital_input_7"/>
+        <state_interface name="digital_input_8"/>
+        <state_interface name="digital_input_9"/>
+        <state_interface name="digital_input_10"/>
+        <state_interface name="digital_input_11"/>
+        <state_interface name="digital_input_12"/>
+        <state_interface name="digital_input_13"/>
+        <state_interface name="digital_input_14"/>
+        <state_interface name="digital_input_15"/>
+        <state_interface name="digital_input_16"/>
+        <state_interface name="digital_input_17"/>
+        <state_interface name="standard_analog_output_0"/>
+        <state_interface name="standard_analog_output_1"/>
+        <state_interface name="standard_analog_input_0"/>
+        <state_interface name="standard_analog_input_1"/>
+        <state_interface name="analog_io_type_0"/>
+        <state_interface name="analog_io_type_1"/>
+        <state_interface name="analog_io_type_2"/>
+        <state_interface name="analog_io_type_3"/>
+        <state_interface name="tool_mode"/>
+        <state_interface name="tool_output_voltage"/>
+        <state_interface name="tool_output_current"/>
+        <state_interface name="tool_temperature"/>
+        <state_interface name="tool_analog_input_0"/>
+        <state_interface name="tool_analog_input_1"/>
+        <state_interface name="tool_analog_input_type_0"/>
+        <state_interface name="tool_analog_input_type_1"/>
+        <state_interface name="robot_mode"/>
+        <state_interface name="robot_status_bit_0"/>
+        <state_interface name="robot_status_bit_1"/>
+        <state_interface name="robot_status_bit_2"/>
+        <state_interface name="robot_status_bit_3"/>
+        <state_interface name="safety_mode"/>
+        <state_interface name="safety_status_bit_0"/>
+        <state_interface name="safety_status_bit_1"/>
+        <state_interface name="safety_status_bit_2"/>
+        <state_interface name="safety_status_bit_3"/>
+        <state_interface name="safety_status_bit_4"/>
+        <state_interface name="safety_status_bit_5"/>
+        <state_interface name="safety_status_bit_6"/>
+        <state_interface name="safety_status_bit_7"/>
+        <state_interface name="safety_status_bit_8"/>
+        <state_interface name="safety_status_bit_9"/>
+        <state_interface name="safety_status_bit_10"/>
+      </joint>
     </ros2_control>
   </xacro:macro>

File: urdf/ur.urdf.xacro (robot description, xacro)
@@ -2,5 +2,5 @@
 <robot xmlns:xacro="http://wiki.ros.org/xacro" name="$(arg name)">
    <!-- robot name parameter -->
-   <xacro:arg name="name" default=""/>
+   <xacro:arg name="name" default="ur"/>
    <!-- import main macro -->
    <xacro:include filename="$(find ur_description)/urdf/ur_macro.xacro"/>

File: urdf/ur5_robot.urdf.xacro (robot description, xacro)
@@ -13,5 +13,5 @@
     <xacro:arg name="robot_ip" default="10.0.1.186"/>
     <!-- ros2 control include -->
-    <xacro:include filename="$(find ur_ros2_control_demos)/urdf/ur5_system_position_only.ros2_control.xacro" />
+    <xacro:include filename="$(find ur_bringup)/urdf/ur5_system_position_only.ros2_control.xacro" />
     <!-- ros2 control instance -->
     <xacro:ur5_system_position_only name="URPositionHardwareInterface" prefix=""

File: urdf/ur_macro.xacro (robot description, xacro)
@@ -71,5 +71,5 @@
     <xacro:include filename="$(find ur_description)/urdf/ur.ros2_control.xacro" />
     <!-- ros2 control instance -->
-    <xacro:ur5_system_position_only
+    <xacro:ur_ros2_control
       name="URPositionHardwareInterface" prefix="$(arg prefix)"
       use_fake_hardware="$(arg use_fake_hardware)"

Commit message: Allows setting initial joint positions for Generic system (#154)
* added the initial_positions argument with default dictionary

* documented the use of the initial_positions argument

* Apply suggestions from code review

* Update README.md

* added initial_positions yaml file to serve as an example

* Additional changes to ros2 control xacro.

* Fix pre-commit.

Co-authored-by: Denis Štogl <destogl@users.noreply.github.com>
Co-authored-by: Lovro <lovro.ivanov@gmail.com>

File: urdf/ur.ros2_control.xacro (robot description, xacro)
@@ -4,4 +4,5 @@
     use_fake_hardware:=false fake_sensor_commands:=false
     headless_mode:=false
+    initial_positions:=${dict(shoulder_pan_joint=0.0,shoulder_lift_joint=-1.57,elbow_joint=0.0,wrist_1_joint=-1.57,wrist_2_joint=0.0,wrist_3_joint=0.0)}
     script_filename output_recipe_filename
     input_recipe_filename tf_prefix
@@ -51,5 +52,5 @@
         <state_interface name="velocity"/>
         <state_interface name="effort"/>
-        <param name="initial_position">0.0</param>  <!-- initial position for the FakeSystem -->
+        <param name="initial_position">${initial_positions['shoulder_pan_joint']}</param>  <!-- initial position for the FakeSystem -->
       </joint>
       <joint name="${prefix}shoulder_lift_joint">
@@ -65,5 +66,5 @@
         <state_interface name="velocity"/>
         <state_interface name="effort"/>
-        <param name="initial_position">-1.57</param>  <!-- initial position for the FakeSystem -->
+        <param name="initial_position">${initial_positions['shoulder_lift_joint']}</param>  <!-- initial position for the FakeSystem -->
       </joint>
       <joint name="${prefix}elbow_joint">
@@ -79,5 +80,5 @@
         <state_interface name="velocity"/>
         <state_interface name="effort"/>
-        <param name="initial_position">0.0</param>  <!-- initial position for the FakeSystem -->
+        <param name="initial_position">${initial_positions['elbow_joint']}</param>  <!-- initial position for the FakeSystem -->
       </joint>
       <joint name="${prefix}wrist_1_joint">
@@ -93,5 +94,5 @@
         <state_interface name="velocity"/>
         <state_interface name="effort"/>
-        <param name="initial_position">-1.57</param>  <!-- initial position for the FakeSystem -->
+        <param name="initial_position">${initial_positions['wrist_1_joint']}</param>  <!-- initial position for the FakeSystem -->
       </joint>
       <joint name="${prefix}wrist_2_joint">
@@ -107,5 +108,5 @@
         <state_interface name="velocity"/>
         <state_interface name="effort"/>
-        <param name="initial_position">0.0</param>  <!-- initial position for the FakeSystem -->
+        <param name="initial_position">${initial_positions['wrist_2_joint']}</param>  <!-- initial position for the FakeSystem -->
       </joint>
       <joint name="${prefix}wrist_3_joint">
@@ -121,5 +122,5 @@
         <state_interface name="velocity"/>
         <state_interface name="effort"/>
-        <param name="initial_position">0.0</param>  <!-- initial position for the FakeSystem -->
+        <param name="initial_position">${initial_positions['wrist_3_joint']}</param>  <!-- initial position for the FakeSystem -->
       </joint>
       <sensor name="tcp_fts_sensor">

File: urdf/ur.urdf.xacro (robot description, xacro)
@@ -19,4 +19,7 @@
    <xacro:arg name="fake_sensor_commands" default="false" />
    <xacro:arg name="headless_mode" default="false" />
+   <!-- initial position -->
+   <xacro:arg name="initial_positions_file" default="$(find ur_description)/config/initial_positions.yaml"/>
+   <xacro:property name="initial_positions_file" default="$(arg initial_positions_file)"/>
    <!-- arm -->
    <xacro:ur_robot
@@ -32,4 +35,5 @@
      use_fake_hardware="$(arg use_fake_hardware)"
      fake_sensor_commands="$(arg fake_sensor_commands)"
-     headless_mode="$(arg headless_mode)" />
+     headless_mode="$(arg headless_mode)"
+     initial_positions="${load_yaml(initial_positions_file)}" />
 </robot>

File: urdf/ur_macro.xacro (robot description, xacro)
@@ -56,6 +56,6 @@
     use_fake_hardware:=false
     fake_sensor_commands:=false
-    headless_mode:=false"
-  >
+    headless_mode:=false
+    initial_positions:=${dict(shoulder_pan_joint=0.0,shoulder_lift_joint=-1.57,elbow_joint=0.0,wrist_1_joint=-1.57,wrist_2_joint=0.0,wrist_3_joint=0.0)}">
     <!-- Load configuration data from the provided .yaml files -->
     <xacro:read_model_data
@@ -75,4 +75,5 @@
       name="URPositionHardwareInterface" prefix="${prefix}"
       use_fake_hardware="$(arg use_fake_hardware)"
+      initial_positions="${initial_positions}"
       fake_sensor_commands="$(arg fake_sensor_commands)"
       headless_mode="$(arg headless_mode)"

Commit message: Add missing command and state interfaces to get everything working with the fake hardware and add some comment into xacro file to be clearer. (#221)

File: urdf/ur.ros2_control.xacro (robot description, xacro)
@@ -231,4 +231,11 @@
         <state_interface name="safety_status_bit_10"/>
       </joint>
+      <joint name="resend_robot_program">
+        <command_interface name="resend_robot_program_cmd"/>
+        <command_interface name="resend_robot_program_async_success"/>
+      </joint>
+      <joint name="system_interface">
+        <state_interface name="initialized"/>
+      </joint>
     </ros2_control>
   </xacro:macro>

File: urdf/ur.urdf.xacro (robot description, xacro)
@@ -19,6 +19,7 @@
    <xacro:arg name="fake_sensor_commands" default="false" />
    <xacro:arg name="headless_mode" default="false" />
-   <!-- initial position -->
+   <!-- initial position for fake hardware -->
    <xacro:arg name="initial_positions_file" default="$(find ur_description)/config/initial_positions.yaml"/>
+   <!-- convert to property to use substitution in function -->
    <xacro:property name="initial_positions_file" default="$(arg initial_positions_file)"/>
    <!-- arm -->
