Commit message: Add URDF files for simulation.

File: urdf/ur.ros2_control.xacro (robot description, xacro)
@@ -1,6 +1,10 @@
 <?xml version="1.0"?>
 <robot xmlns:xacro="http://www.ros.org/wiki/xacro">
-  <xacro:macro name="ur_ros2_control" params="name prefix
+  <xacro:macro name="ur_ros2_control" params="
+    name
+    prefix
     use_fake_hardware:=false fake_sensor_commands:=false
+    gazebo_sim:=false
+    ignition_sim:=false
     headless_mode:=false
     initial_positions:=${dict(shoulder_pan_joint=0.0,shoulder_lift_joint=-1.57,elbow_joint=0.0,wrist_1_joint=-1.57,wrist_2_joint=0.0,wrist_3_joint=0.0)}
@@ -11,4 +15,10 @@
     <ros2_control name="${name}" type="system">
       <hardware>
+        <xacro:if value="${gazebo_sim}">
+          <plugin>gazebo_ros2_control/GazeboSystem</plugin>
+        </xacro:if>
+        <xacro:if value="${ignition_sim}">
+          <plugin>ignition_ros2_control/IgnitionSystem</plugin>
+        </xacro:if>
         <xacro:if value="${use_fake_hardware}">
           <plugin>fake_components/GenericSystem</plugin>
@@ -16,5 +26,5 @@
           <param name="state_following_offset">0.0</param>
         </xacro:if>
-        <xacro:unless value="${use_fake_hardware}">
+        <xacro:unless value="${use_fake_hardware or gazebo_sim or ignition_sim}">
           <plugin>ur_robot_driver/URPositionHardwareInterface</plugin>
           <param name="robot_ip">${robot_ip}</param>
@@ -125,118 +135,120 @@
         <param name="initial_position">${initial_positions['wrist_3_joint']}</param>  <!-- initial position for the FakeSystem -->
       </joint>
-      <sensor name="tcp_fts_sensor">
-        <state_interface name="force.x"/>
-        <state_interface name="force.y"/>
-        <state_interface name="force.z"/>
-        <state_interface name="torque.x"/>
-        <state_interface name="torque.y"/>
-        <state_interface name="torque.z"/>
-      </sensor>
-      <!-- NOTE The following are joints used only for testing with fake hardware and will change in the future -->
-      <joint name="speed_scaling">
-        <state_interface name="speed_scaling_factor"/>
-        <param name="initial_speed_scaling_factor">1</param>
-        <command_interface name="target_speed_fraction_cmd"/>
-        <command_interface name="target_speed_fraction_async_success"/>
-      </joint>
-      <joint name="gpio">
-        <command_interface name="standard_digital_output_cmd_0"/>
-        <command_interface name="standard_digital_output_cmd_1"/>
-        <command_interface name="standard_digital_output_cmd_2"/>
-        <command_interface name="standard_digital_output_cmd_3"/>
-        <command_interface name="standard_digital_output_cmd_4"/>
-        <command_interface name="standard_digital_output_cmd_5"/>
-        <command_interface name="standard_digital_output_cmd_6"/>
-        <command_interface name="standard_digital_output_cmd_7"/>
-        <command_interface name="standard_digital_output_cmd_8"/>
-        <command_interface name="standard_digital_output_cmd_9"/>
-        <command_interface name="standard_digital_output_cmd_10"/>
-        <command_interface name="standard_digital_output_cmd_11"/>
-        <command_interface name="standard_digital_output_cmd_12"/>
-        <command_interface name="standard_digital_output_cmd_13"/>
-        <command_interface name="standard_digital_output_cmd_14"/>
-        <command_interface name="standard_digital_output_cmd_15"/>
-        <command_interface name="standard_digital_output_cmd_16"/>
-        <command_interface name="standard_digital_output_cmd_17"/>
-        <command_interface name="standard_analog_output_cmd_0"/>
-        <command_interface name="standard_analog_output_cmd_1"/>
-        <command_interface name="io_async_success"/>
-        <state_interface name="digital_output_0"/>
-        <state_interface name="digital_output_1"/>
-        <state_interface name="digital_output_2"/>
-        <state_interface name="digital_output_3"/>
-        <state_interface name="digital_output_4"/>
-        <state_interface name="digital_output_5"/>
-        <state_interface name="digital_output_6"/>
-        <state_interface name="digital_output_7"/>
-        <state_interface name="digital_output_8"/>
-        <state_interface name="digital_output_9"/>
-        <state_interface name="digital_output_10"/>
-        <state_interface name="digital_output_11"/>
-        <state_interface name="digital_output_12"/>
-        <state_interface name="digital_output_13"/>
-        <state_interface name="digital_output_14"/>
-        <state_interface name="digital_output_15"/>
-        <state_interface name="digital_output_16"/>
-        <state_interface name="digital_output_17"/>
-        <state_interface name="digital_input_0"/>
-        <state_interface name="digital_input_1"/>
-        <state_interface name="digital_input_2"/>
-        <state_interface name="digital_input_3"/>
-        <state_interface name="digital_input_4"/>
-        <state_interface name="digital_input_5"/>
-        <state_interface name="digital_input_6"/>
-        <state_interface name="digital_input_7"/>
-        <state_interface name="digital_input_8"/>
-        <state_interface name="digital_input_9"/>
-        <state_interface name="digital_input_10"/>
-        <state_interface name="digital_input_11"/>
-        <state_interface name="digital_input_12"/>
-        <state_interface name="digital_input_13"/>
-        <state_interface name="digital_input_14"/>
-        <state_interface name="digital_input_15"/>
-        <state_interface name="digital_input_16"/>
-        <state_interface name="digital_input_17"/>
-        <state_interface name="standard_analog_output_0"/>
-        <state_interface name="standard_analog_output_1"/>
-        <state_interface name="standard_analog_input_0"/>
-        <state_interface name="standard_analog_input_1"/>
-        <state_interface name="analog_io_type_0"/>
-        <state_interface name="analog_io_type_1"/>
-        <state_interface name="analog_io_type_2"/>
-        <state_interface name="analog_io_type_3"/>
-        <state_interface name="tool_mode"/>
-        <state_interface name="tool_output_voltage"/>
-        <state_interface name="tool_output_current"/>
-        <state_interface name="tool_temperature"/>
-        <state_interface name="tool_analog_input_0"/>
-        <state_interface name="tool_analog_input_1"/>
-        <state_interface name="tool_analog_input_type_0"/>
-        <state_interface name="tool_analog_input_type_1"/>
-        <state_interface name="robot_mode"/>
-        <state_interface name="robot_status_bit_0"/>
-        <state_interface name="robot_status_bit_1"/>
-        <state_interface name="robot_status_bit_2"/>
-        <state_interface name="robot_status_bit_3"/>
-        <state_interface name="safety_mode"/>
-        <state_interface name="safety_status_bit_0"/>
-        <state_interface name="safety_status_bit_1"/>
-        <state_interface name="safety_status_bit_2"/>
-        <state_interface name="safety_status_bit_3"/>
-        <state_interface name="safety_status_bit_4"/>
-        <state_interface name="safety_status_bit_5"/>
-        <state_interface name="safety_status_bit_6"/>
-        <state_interface name="safety_status_bit_7"/>
-        <state_interface name="safety_status_bit_8"/>
-        <state_interface name="safety_status_bit_9"/>
-        <state_interface name="safety_status_bit_10"/>
-      </joint>
-      <joint name="resend_robot_program">
-        <command_interface name="resend_robot_program_cmd"/>
-        <command_interface name="resend_robot_program_async_success"/>
-      </joint>
-      <joint name="system_interface">
-        <state_interface name="initialized"/>
-      </joint>
+      <xacro:unless value="${gazebo_sim or ignition_sim}">
+        <sensor name="tcp_fts_sensor">
+          <state_interface name="force.x"/>
+          <state_interface name="force.y"/>
+          <state_interface name="force.z"/>
+          <state_interface name="torque.x"/>
+          <state_interface name="torque.y"/>
+          <state_interface name="torque.z"/>
+        </sensor>
+        <!-- NOTE The following are joints used only for testing with fake hardware and will change in the future -->
+        <joint name="speed_scaling">
+          <state_interface name="speed_scaling_factor"/>
+          <param name="initial_speed_scaling_factor">1</param>
+          <command_interface name="target_speed_fraction_cmd"/>
+          <command_interface name="target_speed_fraction_async_success"/>
+        </joint>
+        <joint name="gpio">
+          <command_interface name="standard_digital_output_cmd_0"/>
+          <command_interface name="standard_digital_output_cmd_1"/>
+          <command_interface name="standard_digital_output_cmd_2"/>
+          <command_interface name="standard_digital_output_cmd_3"/>
+          <command_interface name="standard_digital_output_cmd_4"/>
+          <command_interface name="standard_digital_output_cmd_5"/>
+          <command_interface name="standard_digital_output_cmd_6"/>
+          <command_interface name="standard_digital_output_cmd_7"/>
+          <command_interface name="standard_digital_output_cmd_8"/>
+          <command_interface name="standard_digital_output_cmd_9"/>
+          <command_interface name="standard_digital_output_cmd_10"/>
+          <command_interface name="standard_digital_output_cmd_11"/>
+          <command_interface name="standard_digital_output_cmd_12"/>
+          <command_interface name="standard_digital_output_cmd_13"/>
+          <command_interface name="standard_digital_output_cmd_14"/>
+          <command_interface name="standard_digital_output_cmd_15"/>
+          <command_interface name="standard_digital_output_cmd_16"/>
+          <command_interface name="standard_digital_output_cmd_17"/>
+          <command_interface name="standard_analog_output_cmd_0"/>
+          <command_interface name="standard_analog_output_cmd_1"/>
+          <command_interface name="io_async_success"/>
+          <state_interface name="digital_output_0"/>
+          <state_interface name="digital_output_1"/>
+          <state_interface name="digital_output_2"/>
+          <state_interface name="digital_output_3"/>
+          <state_interface name="digital_output_4"/>
+          <state_interface name="digital_output_5"/>
+          <state_interface name="digital_output_6"/>
+          <state_interface name="digital_output_7"/>
+          <state_interface name="digital_output_8"/>
+          <state_interface name="digital_output_9"/>
+          <state_interface name="digital_output_10"/>
+          <state_interface name="digital_output_11"/>
+          <state_interface name="digital_output_12"/>
+          <state_interface name="digital_output_13"/>
+          <state_interface name="digital_output_14"/>
+          <state_interface name="digital_output_15"/>
+          <state_interface name="digital_output_16"/>
+          <state_interface name="digital_output_17"/>
+          <state_interface name="digital_input_0"/>
+          <state_interface name="digital_input_1"/>
+          <state_interface name="digital_input_2"/>
+          <state_interface name="digital_input_3"/>
+          <state_interface name="digital_input_4"/>
+          <state_interface name="digital_input_5"/>
+          <state_interface name="digital_input_6"/>
+          <state_interface name="digital_input_7"/>
+          <state_interface name="digital_input_8"/>
+          <state_interface name="digital_input_9"/>
+          <state_interface name="digital_input_10"/>
+          <state_interface name="digital_input_11"/>
+          <state_interface name="digital_input_12"/>
+          <state_interface name="digital_input_13"/>
+          <state_interface name="digital_input_14"/>
+          <state_interface name="digital_input_15"/>
+          <state_interface name="digital_input_16"/>
+          <state_interface name="digital_input_17"/>
+          <state_interface name="standard_analog_output_0"/>
+          <state_interface name="standard_analog_output_1"/>
+          <state_interface name="standard_analog_input_0"/>
+          <state_interface name="standard_analog_input_1"/>
+          <state_interface name="analog_io_type_0"/>
+          <state_interface name="analog_io_type_1"/>
+          <state_interface name="analog_io_type_2"/>
+          <state_interface name="analog_io_type_3"/>
+          <state_interface name="tool_mode"/>
+          <state_interface name="tool_output_voltage"/>
+          <state_interface name="tool_output_current"/>
+          <state_interface name="tool_temperature"/>
+          <state_interface name="tool_analog_input_0"/>
+          <state_interface name="tool_analog_input_1"/>
+          <state_interface name="tool_analog_input_type_0"/>
+          <state_interface name="tool_analog_input_type_1"/>
+          <state_interface name="robot_mode"/>
+          <state_interface name="robot_status_bit_0"/>
+          <state_interface name="robot_status_bit_1"/>
+          <state_interface name="robot_status_bit_2"/>
+          <state_interface name="robot_status_bit_3"/>
+          <state_interface name="safety_mode"/>
+          <state_interface name="safety_status_bit_0"/>
+          <state_interface name="safety_status_bit_1"/>
+          <state_interface name="safety_status_bit_2"/>
+          <state_interface name="safety_status_bit_3"/>
+          <state_interface name="safety_status_bit_4"/>
+          <state_interface name="safety_status_bit_5"/>
+          <state_interface name="safety_status_bit_6"/>
+          <state_interface name="safety_status_bit_7"/>
+          <state_interface name="safety_status_bit_8"/>
+          <state_interface name="safety_status_bit_9"/>
+          <state_interface name="safety_status_bit_10"/>
+        </joint>
+        <joint name="resend_robot_program">
+          <command_interface name="resend_robot_program_cmd"/>
+          <command_interface name="resend_robot_program_async_success"/>
+        </joint>
+        <joint name="system_interface">
+          <state_interface name="initialized"/>
+        </joint>
+      </xacro:unless>
     </ros2_control>
   </xacro:macro>

Commit message: Update simulation flag names.

File: urdf/ur.ros2_control.xacro (robot description, xacro)
@@ -5,6 +5,6 @@
     prefix
     use_fake_hardware:=false fake_sensor_commands:=false
-    gazebo_sim:=false
-    ignition_sim:=false
+    sim_gazebo:=false
+    sim_ignition:=false
     headless_mode:=false
     initial_positions:=${dict(shoulder_pan_joint=0.0,shoulder_lift_joint=-1.57,elbow_joint=0.0,wrist_1_joint=-1.57,wrist_2_joint=0.0,wrist_3_joint=0.0)}
@@ -15,9 +15,9 @@
     <ros2_control name="${name}" type="system">
       <hardware>
-        <xacro:if value="${gazebo_sim}">
+        <xacro:if value="${sim_gazebo}">
           <plugin>gazebo_ros2_control/GazeboSystem</plugin>
         </xacro:if>
-        <xacro:if value="${ignition_sim}">
-          <plugin>ignition_ros2_control/IgnitionSystem</plugin>
+        <xacro:if value="${sim_ignition}">
+          <plugin>ign_ros2_control/IgnitionSystem</plugin>
         </xacro:if>
         <xacro:if value="${use_fake_hardware}">
@@ -26,5 +26,5 @@
           <param name="state_following_offset">0.0</param>
         </xacro:if>
-        <xacro:unless value="${use_fake_hardware or gazebo_sim or ignition_sim}">
+        <xacro:unless value="${use_fake_hardware or sim_gazebo or sim_ignition}">
           <plugin>ur_robot_driver/URPositionHardwareInterface</plugin>
           <param name="robot_ip">${robot_ip}</param>
@@ -60,8 +60,10 @@
           <param name="max">3.15</param>
         </command_interface>
-        <state_interface name="position"/>
-        <state_interface name="velocity"/>
-        <state_interface name="effort"/>
-        <param name="initial_position">${initial_positions['shoulder_pan_joint']}</param>  <!-- initial position for the FakeSystem -->
+        <state_interface name="position">
+          <!-- initial position for the FakeSystem and simulation -->
+          <param name="initial_value">${initial_positions['shoulder_pan_joint']}</param>
+        </state_interface>
+        <state_interface name="velocity"/>
+        <state_interface name="effort"/>
       </joint>
       <joint name="${prefix}shoulder_lift_joint">
@@ -74,8 +76,10 @@
           <param name="max">3.15</param>
         </command_interface>
-        <state_interface name="position"/>
-        <state_interface name="velocity"/>
-        <state_interface name="effort"/>
-        <param name="initial_position">${initial_positions['shoulder_lift_joint']}</param>  <!-- initial position for the FakeSystem -->
+        <state_interface name="position">
+          <!-- initial position for the FakeSystem and simulation -->
+          <param name="initial_value">${initial_positions['shoulder_lift_joint']}</param>
+        </state_interface>
+        <state_interface name="velocity"/>
+        <state_interface name="effort"/>
       </joint>
       <joint name="${prefix}elbow_joint">
@@ -88,8 +92,10 @@
           <param name="max">3.15</param>
         </command_interface>
-        <state_interface name="position"/>
-        <state_interface name="velocity"/>
-        <state_interface name="effort"/>
-        <param name="initial_position">${initial_positions['elbow_joint']}</param>  <!-- initial position for the FakeSystem -->
+        <state_interface name="position">
+          <!-- initial position for the FakeSystem and simulation -->
+          <param name="initial_value">${initial_positions['elbow_joint']}</param>
+        </state_interface>
+        <state_interface name="velocity"/>
+        <state_interface name="effort"/>
       </joint>
       <joint name="${prefix}wrist_1_joint">
@@ -102,8 +108,10 @@
           <param name="max">3.2</param>
         </command_interface>
-        <state_interface name="position"/>
-        <state_interface name="velocity"/>
-        <state_interface name="effort"/>
-        <param name="initial_position">${initial_positions['wrist_1_joint']}</param>  <!-- initial position for the FakeSystem -->
+        <state_interface name="position">
+          <!-- initial position for the FakeSystem and simulation -->
+          <param name="initial_value">${initial_positions['wrist_1_joint']}</param>
+        </state_interface>
+        <state_interface name="velocity"/>
+        <state_interface name="effort"/>
       </joint>
       <joint name="${prefix}wrist_2_joint">
@@ -116,8 +124,10 @@
           <param name="max">3.2</param>
         </command_interface>
-        <state_interface name="position"/>
-        <state_interface name="velocity"/>
-        <state_interface name="effort"/>
-        <param name="initial_position">${initial_positions['wrist_2_joint']}</param>  <!-- initial position for the FakeSystem -->
+        <state_interface name="position">
+          <!-- initial position for the FakeSystem and simulation -->
+          <param name="initial_value">${initial_positions['wrist_2_joint']}</param>
+        </state_interface>
+        <state_interface name="velocity"/>
+        <state_interface name="effort"/>
       </joint>
       <joint name="${prefix}wrist_3_joint">
@@ -130,10 +140,12 @@
           <param name="max">3.2</param>
         </command_interface>
-        <state_interface name="position"/>
-        <state_interface name="velocity"/>
-        <state_interface name="effort"/>
-        <param name="initial_position">${initial_positions['wrist_3_joint']}</param>  <!-- initial position for the FakeSystem -->
-      </joint>
-      <xacro:unless value="${gazebo_sim or ignition_sim}">
+        <state_interface name="position">
+          <!-- initial position for the FakeSystem and simulation -->
+          <param name="initial_value">${initial_positions['wrist_3_joint']}</param>
+        </state_interface>
+        <state_interface name="velocity"/>
+        <state_interface name="effort"/>
+      </joint>
+      <xacro:unless value="${sim_gazebo or sim_ignition}">
         <sensor name="tcp_fts_sensor">
           <state_interface name="force.x"/>

File: urdf/ur_simulation.urdf.xacro (robot description, xacro)
@@ -3,4 +3,5 @@
   <!-- robot name parameter -->
   <xacro:arg name="name" default="ur"/>
+  <xacro:arg name="ur_type" default="ur5e"/>
   <!-- import main macro -->
   <xacro:include filename="$(find ur_description)/urdf/ur_simulation_macro.xacro"/>
@@ -23,6 +24,6 @@
   <xacro:arg name="initial_positions_file" default="$(find ur_description)/config/initial_positions.yaml"/>
   <!-- Simulation parameter -->
-  <xacro:arg name="gazebo_sim" default="false" />
-  <xacro:arg name="ignition_sim" default="false" />
+  <xacro:arg name="sim_gazebo" default="false" />
+  <xacro:arg name="sim_ignition" default="false" />
   <xacro:arg name="simulation_controllers" default="$(find ur_bringup)/config/ur_controllers.yaml" />
   <!-- convert to property to use substitution in function -->
@@ -32,5 +33,5 @@
   <!-- arm -->
   <xacro:ur_robot
-    name="$(arg name)"
+    name="$(arg ur_type)"
     prefix="$(arg prefix)"
     parent="world"
@@ -48,9 +49,9 @@
     initial_positions="${load_yaml(initial_positions_file)}"
     use_tool_communication="$(arg use_tool_communication)"
-    gazebo_sim="$(arg gazebo_sim)"
-    ignition_sim="$(arg ignition_sim)" >
+    sim_gazebo="$(arg sim_gazebo)"
+    sim_ignition="$(arg sim_ignition)" >
     <origin xyz="0 0 0" rpy="0 0 0" />          <!-- position robot in the world -->
   </xacro:ur_robot>
-  <xacro:if value="$(arg gazebo_sim)">
+  <xacro:if value="$(arg sim_gazebo)">
     <!-- Gazebo plugins -->
     <gazebo reference="world">
@@ -62,10 +63,10 @@
     </gazebo>
   </xacro:if>
-  <xacro:if value="$(arg ignition_sim)">
+  <xacro:if value="$(arg sim_ignition)">
     <!-- Gazebo plugins -->
     <gazebo reference="world">
     </gazebo>
     <gazebo>
-      <plugin filename="libignition_ros2_control-system.so" name="ignition_ros2_control::IgnitionROS2ControlPlugin">
+      <plugin filename="libign_ros2_control-system.so" name="ign_ros2_control::IgnitionROS2ControlPlugin">
         <parameters>$(arg simulation_controllers)</parameters>
         <controller_manager_node_name>$(arg prefix)controller_manager</controller_manager_node_name>

File: urdf/ur_simulation_macro.xacro (robot description, xacro)
@@ -59,6 +59,6 @@
     use_fake_hardware:=false
     fake_sensor_commands:=false
-    gazebo_sim:=false
-    ignition_sim:=false
+    sim_gazebo:=false
+    sim_ignition:=false
     headless_mode:=false
     initial_positions:=${dict(shoulder_pan_joint=0.0,shoulder_lift_joint=-1.57,elbow_joint=0.0,wrist_1_joint=-1.57,wrist_2_joint=0.0,wrist_3_joint=0.0)}
@@ -82,6 +82,6 @@
       use_fake_hardware="$(arg use_fake_hardware)"
       fake_sensor_commands="$(arg fake_sensor_commands)"
-      gazebo_sim="$(arg gazebo_sim)"
-      ignition_sim="$(arg ignition_sim)"
+      sim_gazebo="$(arg sim_gazebo)"
+      sim_ignition="$(arg sim_ignition)"
       headless_mode="$(arg headless_mode)"
       initial_positions="${initial_positions}"
