Commit message: Port 'gpio'-changes from UniversalRobots/Universal_Robots_ROS2_Driver#224

File: urdf/ur.ros2_control.xacro (robot description, xacro)
@@ -159,11 +159,11 @@
         </sensor>
         <!-- NOTE The following are joints used only for testing with fake hardware and will change in the future -->
-        <joint name="speed_scaling">
+        <gpio name="speed_scaling">
           <state_interface name="speed_scaling_factor"/>
           <param name="initial_speed_scaling_factor">1</param>
           <command_interface name="target_speed_fraction_cmd"/>
           <command_interface name="target_speed_fraction_async_success"/>
-        </joint>
-        <joint name="gpio">
+        </gpio>
+        <gpio name="gpio">
           <command_interface name="standard_digital_output_cmd_0"/>
           <command_interface name="standard_digital_output_cmd_1"/>
@@ -256,5 +256,5 @@
           <state_interface name="safety_status_bit_9"/>
           <state_interface name="safety_status_bit_10"/>
-        </joint>
+        </gpio>
         <gpio name="payload">
           <command_interface name="mass"/>
@@ -264,11 +264,11 @@
           <command_interface name="payload_async_success"/>
         </gpio>
-        <joint name="resend_robot_program">
+        <gpio name="resend_robot_program">
           <command_interface name="resend_robot_program_cmd"/>
           <command_interface name="resend_robot_program_async_success"/>
-        </joint>
-        <joint name="system_interface">
+        </gpio>
+        <gpio name="system_interface">
           <state_interface name="initialized"/>
-        </joint>
+        </gpio>
       </xacro:unless>
     </ros2_control>

File: urdf/ur.urdf.xacro (robot description, xacro)
@@ -33,5 +33,5 @@
    <xacro:arg name="sim_ignition" default="false" />
    <xacro:arg name="simulation_controllers" default="" />
-   <!-- initial position for fake hardware -->
+   <!-- initial position for simulations (Fake Hardware, Gazebo, Ignition) -->
    <xacro:arg name="initial_positions_file" default="$(find ur_description)/config/initial_positions.yaml"/>
    <!-- convert to property to use substitution in function -->

Commit message: Add dynamics per joint. Change pid params.

File: urdf/ur.ros2_control.xacro (robot description, xacro)
@@ -76,12 +76,20 @@
         <xacro:if value="${sim_ignition}">
           <!-- initial PID values for the IgnitionSystem and simulation -->
-          <param name="p">10000.0</param>
-          <param name="i">0.0</param>
-          <param name="d">5.0</param>
-          <param name="iMax">75</param>
-          <param name="iMin">-75</param>
-          <param name="cmdMax">150</param>
-          <param name="cmdMin">-150</param>
-          <param name="cmdOffset">0.0</param>
+          <param name="p_pos">10.0</param>
+          <param name="i_pos">0.0</param>
+          <param name="d_pos">0.01</param>
+          <param name="iMax_pos">1.57</param>
+          <param name="iMin_pos">-1.57</param>
+          <param name="cmdMax_pos">3.14</param>
+          <param name="cmdMin_pos">-3.14</param>
+          <param name="cmdOffset_pos">0.0</param>
+          <param name="p_vel">50.0</param>
+          <param name="i_vel">100.0</param>
+          <param name="d_vel">0.0</param>
+          <param name="iMax_vel">75.0</param>
+          <param name="iMin_vel">-75.0</param>
+          <param name="cmdMax_vel">150.0</param>
+          <param name="cmdMin_vel">-150.0</param>
+          <param name="cmdOffset_vel">0.0</param>
         </xacro:if>
       </joint>
@@ -103,12 +111,20 @@
         <xacro:if value="${sim_ignition}">
           <!-- initial PID values for the IgnitionSystem and simulation -->
-          <param name="p">10000.0</param>
-          <param name="i">0.0</param>
-          <param name="d">5.0</param>
-          <param name="iMax">75</param>
-          <param name="iMin">-75</param>
-          <param name="cmdMax">150</param>
-          <param name="cmdMin">-150</param>
-          <param name="cmdOffset">0.0</param>
+          <param name="p_pos">10.0</param>
+          <param name="i_pos">0.0</param>
+          <param name="d_pos">0.01</param>
+          <param name="iMax_pos">1.57</param>
+          <param name="iMin_pos">-1.57</param>
+          <param name="cmdMax_pos">3.14</param>
+          <param name="cmdMin_pos">-3.14</param>
+          <param name="cmdOffset_pos">0.0</param>
+          <param name="p_vel">300.0</param>
+          <param name="i_vel">90.0</param>
+          <param name="d_vel">0.0</param>
+          <param name="iMax_vel">75.0</param>
+          <param name="iMin_vel">-75.0</param>
+          <param name="cmdMax_vel">150.0</param>
+          <param name="cmdMin_vel">-150.0</param>
+          <param name="cmdOffset_vel">0.0</param>
         </xacro:if>
       </joint>
@@ -130,12 +146,20 @@
         <xacro:if value="${sim_ignition}">
           <!-- initial PID values for the IgnitionSystem and simulation -->
-          <param name="p">10000.0</param>
-          <param name="i">0.0</param>
-          <param name="d">5.0</param>
-          <param name="iMax">75</param>
-          <param name="iMin">-75</param>
-          <param name="cmdMax">150</param>
-          <param name="cmdMin">-150</param>
-          <param name="cmdOffset">0.0</param>
+          <param name="p_pos">10.0</param>
+          <param name="i_pos">0.0</param>
+          <param name="d_pos">0.01</param>
+          <param name="iMax_pos">1.57</param>
+          <param name="iMin_pos">-1.57</param>
+          <param name="cmdMax_pos">3.14</param>
+          <param name="cmdMin_pos">-3.14</param>
+          <param name="cmdOffset_pos">0.0</param>
+          <param name="p_vel">50.0</param>
+          <param name="i_vel">100.0</param>
+          <param name="d_vel">0.0</param>
+          <param name="iMax_vel">75.0</param>
+          <param name="iMin_vel">-75.0</param>
+          <param name="cmdMax_vel">150.0</param>
+          <param name="cmdMin_vel">-150.0</param>
+          <param name="cmdOffset_vel">0.0</param>
         </xacro:if>
       </joint>
@@ -157,12 +181,20 @@
         <xacro:if value="${sim_ignition}">
           <!-- initial PID values for the IgnitionSystem and simulation -->
-          <param name="p">500.0</param>
-          <param name="i">0.0</param>
-          <param name="d">5.0</param>
-          <param name="iMax">14</param>
-          <param name="iMin">-14</param>
-          <param name="cmdMax">28</param>
-          <param name="cmdMin">-28</param>
-          <param name="cmdOffset">0.0</param>
+          <param name="p_pos">10.0</param>
+          <param name="i_pos">0.0</param>
+          <param name="d_pos">0.001</param>
+          <param name="iMax_pos">1.57</param>
+          <param name="iMin_pos">-1.57</param>
+          <param name="cmdMax_pos">3.14</param>
+          <param name="cmdMin_pos">-3.14</param>
+          <param name="cmdOffset_pos">0.0</param>
+          <param name="p_vel">10.0</param>
+          <param name="i_vel">10.0</param>
+          <param name="d_vel">0.0</param>
+          <param name="iMax_vel">14.0</param>
+          <param name="iMin_vel">-14.0</param>
+          <param name="cmdMax_vel">28.0</param>
+          <param name="cmdMin_vel">-28.0</param>
+          <param name="cmdOffset_vel">0.0</param>
         </xacro:if>
       </joint>
@@ -184,12 +216,20 @@
         <xacro:if value="${sim_ignition}">
           <!-- initial PID values for the IgnitionSystem and simulation -->
-          <param name="p">500.0</param>
-          <param name="i">0.0</param>
-          <param name="d">5.0</param>
-          <param name="iMax">14</param>
-          <param name="iMin">-14</param>
-          <param name="cmdMax">28</param>
-          <param name="cmdMin">-28</param>
-          <param name="cmdOffset">0.0</param>
+          <param name="p_pos">10.0</param>
+          <param name="i_pos">0.0</param>
+          <param name="d_pos">0.001</param>
+          <param name="iMax_pos">1.57</param>
+          <param name="iMin_pos">-1.57</param>
+          <param name="cmdMax_pos">3.14</param>
+          <param name="cmdMin_pos">-3.14</param>
+          <param name="cmdOffset_pos">0.0</param>
+          <param name="p_vel">5.0</param>
+          <param name="i_vel">10.0</param>
+          <param name="d_vel">0.0</param>
+          <param name="iMax_vel">14.0</param>
+          <param name="iMin_vel">-14.0</param>
+          <param name="cmdMax_vel">28.0</param>
+          <param name="cmdMin_vel">-28.0</param>
+          <param name="cmdOffset_vel">0.0</param>
         </xacro:if>
       </joint>
@@ -211,12 +251,20 @@
         <xacro:if value="${sim_ignition}">
           <!-- initial PID values for the IgnitionSystem and simulation -->
-          <param name="p">300.0</param>
-          <param name="i">0.0</param>
-          <param name="d">0.0</param>
-          <param name="iMax">14</param>
-          <param name="iMin">-14</param>
-          <param name="cmdMax">28</param>
-          <param name="cmdMin">-28</param>
-          <param name="cmdOffset">0.0</param>
+          <param name="p_pos">10.0</param>
+          <param name="i_pos">0.0</param>
+          <param name="d_pos">0.0001</param>
+          <param name="iMax_pos">1.57</param>
+          <param name="iMin_pos">-1.57</param>
+          <param name="cmdMax_pos">3.14</param>
+          <param name="cmdMin_pos">-3.14</param>
+          <param name="cmdOffset_pos">0.0</param>
+          <param name="p_vel">5.0</param>
+          <param name="i_vel">10.0</param>
+          <param name="d_vel">0.0</param>
+          <param name="iMax_vel">14.0</param>
+          <param name="iMin_vel">-14.0</param>
+          <param name="cmdMax_vel">28.0</param>
+          <param name="cmdMin_vel">-28.0</param>
+          <param name="cmdOffset_vel">0.0</param>
         </xacro:if>
       </joint>

File: urdf/ur_macro.xacro (robot description, xacro)
@@ -272,5 +272,5 @@
          <safety_controller soft_lower_limit="${shoulder_pan_lower_limit + safety_pos_margin}" soft_upper_limit="${shoulder_pan_upper_limit - safety_pos_margin}" k_position="${safety_k_position}" k_velocity="0.0"/>
       </xacro:if>
-      <dynamics damping="0" friction="0"/>
+      <dynamics damping="21.75" friction="3.48"/>
     </joint>
     <joint name="${prefix}shoulder_lift_joint" type="revolute">
@@ -284,5 +284,5 @@
          <safety_controller soft_lower_limit="${shoulder_lift_lower_limit + safety_pos_margin}" soft_upper_limit="${shoulder_lift_upper_limit - safety_pos_margin}" k_position="${safety_k_position}" k_velocity="0.0"/>
       </xacro:if>
-      <dynamics damping="0" friction="0"/>
+      <dynamics damping="21.75" friction="3.48"/>
     </joint>
     <joint name="${prefix}elbow_joint" type="revolute">
@@ -296,5 +296,5 @@
          <safety_controller soft_lower_limit="${elbow_joint_lower_limit + safety_pos_margin}" soft_upper_limit="${elbow_joint_upper_limit - safety_pos_margin}" k_position="${safety_k_position}" k_velocity="0.0"/>
       </xacro:if>
-      <dynamics damping="0" friction="0"/>
+      <dynamics damping="21.75" friction="3.48"/>
     </joint>
     <joint name="${prefix}wrist_1_joint" type="revolute">
@@ -308,5 +308,5 @@
          <safety_controller soft_lower_limit="${wrist_1_lower_limit + safety_pos_margin}" soft_upper_limit="${wrist_1_upper_limit - safety_pos_margin}" k_position="${safety_k_position}" k_velocity="0.0"/>
       </xacro:if>
-      <dynamics damping="0" friction="0"/>
+      <dynamics damping="3.0" friction="0.48"/>
     </joint>
     <joint name="${prefix}wrist_2_joint" type="revolute">
@@ -320,5 +320,5 @@
          <safety_controller soft_lower_limit="${wrist_2_lower_limit + safety_pos_margin}" soft_upper_limit="${wrist_2_upper_limit - safety_pos_margin}" k_position="${safety_k_position}" k_velocity="0.0"/>
       </xacro:if>
-      <dynamics damping="0" friction="0"/>
+      <dynamics damping="3.0" friction="0.48"/>
     </joint>
     <joint name="${prefix}wrist_3_joint" type="revolute">
@@ -332,5 +332,5 @@
          <safety_controller soft_lower_limit="${wrist_3_lower_limit + safety_pos_margin}" soft_upper_limit="${wrist_3_upper_limit - safety_pos_margin}" k_position="${safety_k_position}" k_velocity="0.0"/>
       </xacro:if>
-      <dynamics damping="0" friction="0"/>
+      <dynamics damping="3.0" friction="0.48"/>
     </joint>
     <link name="${prefix}ft_frame"/>

Commit message: Detangle ros2_control from kinematic model
Signed-off-by: Christoph Hellmann Santos <christoph.hellmann.santos@ipa.fraunhofer.de>

File: urdf/ur.ros2_control.xacro (robot description, xacro)
@@ -1,4 +1,5 @@
 <?xml version="1.0"?>
 <robot xmlns:xacro="http://www.ros.org/wiki/xacro">
+  <xacro:include filename="$(find ur_description)/urdf/inc/ur_transmissions.xacro" />
   <xacro:macro name="ur_ros2_control" params="
     name
@@ -18,5 +19,9 @@
     script_sender_port:=50002
     reverse_ip:=0.0.0.0
-    script_command_port:=50004">
+    script_command_port:=50004
+    transmission_hw_interface:=hardware_interface/PositionJointInterface
+    ">
+    <!-- Add URDF transmission elements (for ros_control) -->
+    <!--<xacro:ur_arm_transmission prefix="${prefix}" hw_interface="${transmission_hw_interface}" />-->
     <ros2_control name="${name}" type="system">
       <hardware>

File: urdf/ur.urdf.xacro (robot description, xacro)
@@ -3,6 +3,8 @@
    <!-- robot name parameter -->
    <xacro:arg name="name" default="ur"/>
-   <!-- import main macro -->
+   <!-- include arm -->
    <xacro:include filename="$(find ur_description)/urdf/ur_macro.xacro"/>
+   <!-- include ros2 control -->
+   <xacro:include filename="$(find ur_description)/urdf/ur.ros2_control.xacro" />
    <!-- possible 'ur_type' values: ur3, ur3e, ur5, ur5e, ur10, ur10e, ur16e -->
    <!-- the default value should raise an error in case this was called without defining the type -->
@@ -46,19 +48,29 @@
    <!-- convert to property to use substitution in function -->
    <xacro:property name="initial_positions_file" default="$(arg initial_positions_file)"/>
+   <xacro:property name="sim_gazebo" default="$(arg sim_gazebo)"/>
+   <xacro:property name="sim_ignition" default="$(arg sim_ignition)"/>
    <!-- create link fixed to the "world" -->
    <link name="world" />
-   <!-- arm -->
+   <!-- load model data -->
+   <xacro:read_model_data
+     joint_limits_parameters_file="$(arg joint_limit_params)"
+     kinematics_parameters_file="$(arg kinematics_params)"
+     physical_parameters_file="$(arg physical_params)"
+     visual_parameters_file="$(arg visual_params)"
+     force_abs_paths="${sim_gazebo or sim_ignition}"/>
+   <!-- arm instance -->
    <xacro:ur_robot
      name="$(arg name)"
      prefix="$(arg prefix)"
      parent="world"
-     joint_limits_parameters_file="$(arg joint_limit_params)"
-     kinematics_parameters_file="$(arg kinematics_params)"
-     physical_parameters_file="$(arg physical_params)"
-     visual_parameters_file="$(arg visual_params)"
-     transmission_hw_interface="$(arg transmission_hw_interface)"
      safety_limits="$(arg safety_limits)"
      safety_pos_margin="$(arg safety_pos_margin)"
      safety_k_position="$(arg safety_k_position)"
+     >
+     <origin xyz="0 0 0" rpy="0 0 0" />          <!-- position robot in the world -->
+   </xacro:ur_robot>
+   <!-- ros2 control instance -->
+   <xacro:ur_ros2_control
+     name="$(arg name)" prefix="$(arg prefix)"
      use_fake_hardware="$(arg use_fake_hardware)"
      fake_sensor_commands="$(arg fake_sensor_commands)"
@@ -82,7 +94,7 @@
      reverse_ip="$(arg reverse_ip)"
      script_command_port="$(arg script_command_port)"
-     >
-     <origin xyz="0 0 0" rpy="0 0 0" />          <!-- position robot in the world -->
-   </xacro:ur_robot>
+     tf_prefix=""
+     hash_kinematics="${kinematics_hash}"
+     />
    <xacro:if value="$(arg sim_gazebo)">
     <!-- Gazebo plugins -->

File: urdf/ur_macro.xacro (robot description, xacro)
@@ -49,9 +49,4 @@
     parent
     *origin
-    joint_limits_parameters_file
-    kinematics_parameters_file
-    physical_parameters_file
-    visual_parameters_file
-    transmission_hw_interface:=hardware_interface/PositionJointInterface
     safety_limits:=false
     safety_pos_margin:=0.15
@@ -80,45 +75,4 @@
     reverse_ip:=0.0.0.0
     script_command_port:=50004">
-    <!-- Load configuration data from the provided .yaml files -->
-    <xacro:read_model_data
-      joint_limits_parameters_file="${joint_limits_parameters_file}"
-      kinematics_parameters_file="${kinematics_parameters_file}"
-      physical_parameters_file="${physical_parameters_file}"
-      visual_parameters_file="${visual_parameters_file}"
-      force_abs_paths="${sim_gazebo or sim_ignition}"/>
-    <!-- ros2 control include -->
-    <xacro:include filename="$(find ur_description)/urdf/ur.ros2_control.xacro" />
-    <!-- ros2 control instance -->
-    <xacro:ur_ros2_control
-      name="${name}" prefix="${prefix}"
-      use_fake_hardware="${use_fake_hardware}"
-      initial_positions="${initial_positions}"
-      fake_sensor_commands="${fake_sensor_commands}"
-      headless_mode="${headless_mode}"
-      sim_gazebo="${sim_gazebo}"
-      sim_ignition="${sim_ignition}"
-      script_filename="${script_filename}"
-      output_recipe_filename="${output_recipe_filename}"
-      input_recipe_filename="${input_recipe_filename}"
-      tf_prefix=""
-      hash_kinematics="${kinematics_hash}"
-      robot_ip="${robot_ip}"
-      use_tool_communication="${use_tool_communication}"
-      tool_voltage="${tool_voltage}"
-      tool_parity="${tool_parity}"
-      tool_baud_rate="${tool_baud_rate}"
-      tool_stop_bits="${tool_stop_bits}"
-      tool_rx_idle_chars="${tool_rx_idle_chars}"
-      tool_tx_idle_chars="${tool_tx_idle_chars}"
-      tool_device_name="${tool_device_name}"
-      tool_tcp_port="${tool_tcp_port}"
-      reverse_port="${reverse_port}"
-      script_sender_port="${script_sender_port}"
-      reverse_ip="${reverse_ip}"
-      script_command_port="${script_command_port}"
-      />
-    <!-- Add URDF transmission elements (for ros_control) -->
-    <!--<xacro:ur_arm_transmission prefix="${prefix}" hw_interface="${transmission_hw_interface}" />-->
-    <!-- Placeholder for ros2_control transmission which don't yet exist -->
     <!-- links -  main serial chain -->
     <link name="${prefix}base_link"/>
