Commit message: Replace duplicated `prefix` parameter with `tf_prefix`

File: urdf/ur.ros2_control.xacro (robot description, xacro)
@@ -3,5 +3,4 @@
   <xacro:macro name="ur_ros2_control" params="
     name
-    prefix
     use_fake_hardware:=false fake_sensor_commands:=false
     sim_gazebo:=false
@@ -38,5 +37,4 @@
         <xacro:unless value="${use_fake_hardware or sim_gazebo or sim_ignition}">
           <plugin>ur_robot_driver/URPositionHardwareInterface</plugin>
-          <param name="prefix">${prefix}</param>
           <param name="robot_ip">${robot_ip}</param>
           <param name="script_filename">${script_filename}</param>
@@ -66,5 +64,5 @@
         </xacro:unless>
       </hardware>
-      <joint name="${prefix}shoulder_pan_joint">
+      <joint name="${tf_prefix}shoulder_pan_joint">
         <command_interface name="position">
           <param name="min">{-2*pi}</param>
@@ -82,5 +80,5 @@
         <state_interface name="effort"/>
       </joint>
-      <joint name="${prefix}shoulder_lift_joint">
+      <joint name="${tf_prefix}shoulder_lift_joint">
         <command_interface name="position">
           <param name="min">{-2*pi}</param>
@@ -98,5 +96,5 @@
         <state_interface name="effort"/>
       </joint>
-      <joint name="${prefix}elbow_joint">
+      <joint name="${tf_prefix}elbow_joint">
         <command_interface name="position">
           <param name="min">{-pi}</param>
@@ -114,5 +112,5 @@
         <state_interface name="effort"/>
       </joint>
-      <joint name="${prefix}wrist_1_joint">
+      <joint name="${tf_prefix}wrist_1_joint">
         <command_interface name="position">
           <param name="min">{-2*pi}</param>
@@ -130,5 +128,5 @@
         <state_interface name="effort"/>
       </joint>
-      <joint name="${prefix}wrist_2_joint">
+      <joint name="${tf_prefix}wrist_2_joint">
         <command_interface name="position">
           <param name="min">{-2*pi}</param>
@@ -146,5 +144,5 @@
         <state_interface name="effort"/>
       </joint>
-      <joint name="${prefix}wrist_3_joint">
+      <joint name="${tf_prefix}wrist_3_joint">
         <command_interface name="position">
           <param name="min">{-2*pi}</param>
@@ -163,5 +161,5 @@
       </joint>
       <xacro:unless value="${sim_gazebo or sim_ignition}">
-        <sensor name="${prefix}tcp_fts_sensor">
+        <sensor name="${tf_prefix}tcp_fts_sensor">
           <state_interface name="force.x"/>
           <state_interface name="force.y"/>
@@ -172,5 +170,5 @@
         </sensor>
         <!-- NOTE The following are joints used only for testing with fake hardware and will change in the future -->
-        <gpio name="${prefix}speed_scaling">
+        <gpio name="${tf_prefix}speed_scaling">
           <state_interface name="speed_scaling_factor"/>
           <param name="initial_speed_scaling_factor">1</param>
@@ -178,5 +176,5 @@
           <command_interface name="target_speed_fraction_async_success"/>
         </gpio>
-        <gpio name="${prefix}gpio">
+        <gpio name="${tf_prefix}gpio">
           <command_interface name="standard_digital_output_cmd_0"/>
           <command_interface name="standard_digital_output_cmd_1"/>
@@ -272,5 +270,5 @@
           <state_interface name="program_running"/>
         </gpio>
-        <gpio name="${prefix}payload">
+        <gpio name="${tf_prefix}payload">
           <command_interface name="mass"/>
           <command_interface name="cog.x"/>
@@ -279,13 +277,13 @@
           <command_interface name="payload_async_success"/>
         </gpio>
-        <gpio name="${prefix}resend_robot_program">
+        <gpio name="${tf_prefix}resend_robot_program">
           <command_interface name="resend_robot_program_cmd"/>
           <command_interface name="resend_robot_program_async_success"/>
         </gpio>
-        <gpio name="${prefix}zero_ftsensor">
+        <gpio name="${tf_prefix}zero_ftsensor">
           <command_interface name="zero_ftsensor_cmd"/>
           <command_interface name="zero_ftsensor_async_success"/>
         </gpio>
-        <gpio name="${prefix}system_interface">
+        <gpio name="${tf_prefix}system_interface">
           <state_interface name="initialized"/>
         </gpio>

File: urdf/ur.urdf.xacro (robot description, xacro)
@@ -9,5 +9,5 @@
    <xacro:arg name="ur_type" default="ur5x"/>
    <!-- parameters -->
-   <xacro:arg name="prefix" default="" />
+   <xacro:arg name="tf_prefix" default="" />
    <xacro:arg name="joint_limit_params" default="$(find ur_description)/config/$(arg ur_type)/joint_limits.yaml"/>
    <xacro:arg name="kinematics_params" default="$(find ur_description)/config/$(arg ur_type)/default_kinematics.yaml"/>
@@ -51,5 +51,5 @@
    <xacro:ur_robot
      name="$(arg name)"
-     prefix="$(arg prefix)"
+     tf_prefix="$(arg tf_prefix)"
      parent="world"
      joint_limits_parameters_file="$(arg joint_limit_params)"
@@ -102,5 +102,5 @@
       <plugin filename="libign_ros2_control-system.so" name="ign_ros2_control::IgnitionROS2ControlPlugin">
         <parameters>$(arg simulation_controllers)</parameters>
-        <controller_manager_node_name>$(arg prefix)controller_manager</controller_manager_node_name>
+        <controller_manager_node_name>$(arg tf_prefix)controller_manager</controller_manager_node_name>
       </plugin>
     </gazebo>

File: urdf/ur_macro.xacro (robot description, xacro)
@@ -46,5 +46,5 @@
   <xacro:macro name="ur_robot" params="
     name
-    prefix
+    tf_prefix
     parent
     *origin
@@ -95,5 +95,5 @@
     <!-- ros2 control instance -->
     <xacro:ur_ros2_control
-      name="${name}" prefix="${prefix}"
+      name="${name}"
       use_fake_hardware="${use_fake_hardware}"
       initial_positions="${initial_positions}"
@@ -105,5 +105,5 @@
       output_recipe_filename="${output_recipe_filename}"
       input_recipe_filename="${input_recipe_filename}"
-      tf_prefix=""
+      tf_prefix="${tf_prefix}"
       hash_kinematics="${kinematics_hash}"
       robot_ip="${robot_ip}"
@@ -129,6 +129,6 @@
     <!-- Placeholder for ros2_control transmission which don't yet exist -->
     <!-- links -  main serial chain -->
-    <link name="${prefix}base_link"/>
-    <link name="${prefix}base_link_inertia">
+    <link name="${tf_prefix}base_link"/>
+    <link name="${tf_prefix}base_link_inertia">
       <visual>
         <origin xyz="0 0 0" rpy="0 0 ${pi}"/>
@@ -147,5 +147,5 @@
       </xacro:cylinder_inertial>
     </link>
-    <link name="${prefix}shoulder_link">
+    <link name="${tf_prefix}shoulder_link">
       <visual>
         <origin xyz="0 0 0" rpy="0 0 ${pi}"/>
@@ -164,5 +164,5 @@
       </xacro:cylinder_inertial>
     </link>
-    <link name="${prefix}upper_arm_link">
+    <link name="${tf_prefix}upper_arm_link">
       <visual>
         <origin xyz="0 0 ${shoulder_offset}" rpy="${pi/2} 0 ${-pi/2}"/>
@@ -181,5 +181,5 @@
       </xacro:cylinder_inertial>
     </link>
-    <link name="${prefix}forearm_link">
+    <link name="${tf_prefix}forearm_link">
       <visual>
         <origin xyz="0 0 ${elbow_offset}" rpy="${pi/2} 0 ${-pi/2}"/>
@@ -198,5 +198,5 @@
       </xacro:cylinder_inertial>
     </link>
-    <link name="${prefix}wrist_1_link">
+    <link name="${tf_prefix}wrist_1_link">
 	  <xacro:get_visual_params name="wrist_1" type="visual_offset"/>
       <visual>
@@ -216,5 +216,5 @@
       </xacro:cylinder_inertial>
     </link>
-    <link name="${prefix}wrist_2_link">
+    <link name="${tf_prefix}wrist_2_link">
 	  <xacro:get_visual_params name="wrist_2" type="visual_offset"/>
       <visual>
@@ -234,5 +234,5 @@
       </xacro:cylinder_inertial>
     </link>
-    <link name="${prefix}wrist_3_link">
+    <link name="${tf_prefix}wrist_3_link">
 	  <xacro:get_visual_params name="wrist_3" type="visual_offset"/>
       <visual>
@@ -253,13 +253,13 @@
     </link>
     <!-- base_joint fixes base_link to the environment -->
-    <joint name="${prefix}base_joint" type="fixed">
+    <joint name="${tf_prefix}base_joint" type="fixed">
       <xacro:insert_block name="origin" />
       <parent link="${parent}" />
-      <child link="${prefix}base_link" />
+      <child link="${tf_prefix}base_link" />
     </joint>
     <!-- joints - main serial chain -->
-    <joint name="${prefix}base_link-base_link_inertia" type="fixed">
-      <parent link="${prefix}base_link" />
-      <child link="${prefix}base_link_inertia" />
+    <joint name="${tf_prefix}base_link-base_link_inertia" type="fixed">
+      <parent link="${tf_prefix}base_link" />
+      <child link="${tf_prefix}base_link_inertia" />
       <!-- 'base_link' is REP-103 aligned (so X+ forward), while the internal
            frames of the robot/controller have X+ pointing backwards.
@@ -269,7 +269,7 @@
       <origin xyz="0 0 0" rpy="0 0 ${pi}" />
     </joint>
-    <joint name="${prefix}shoulder_pan_joint" type="revolute">
-      <parent link="${prefix}base_link_inertia" />
-      <child link="${prefix}shoulder_link" />
+    <joint name="${tf_prefix}shoulder_pan_joint" type="revolute">
+      <parent link="${tf_prefix}base_link_inertia" />
+      <child link="${tf_prefix}shoulder_link" />
       <origin xyz="${shoulder_x} ${shoulder_y} ${shoulder_z}" rpy="${shoulder_roll} ${shoulder_pitch} ${shoulder_yaw}" />
       <axis xyz="0 0 1" />
@@ -281,7 +281,7 @@
       <dynamics damping="0" friction="0"/>
     </joint>
-    <joint name="${prefix}shoulder_lift_joint" type="revolute">
-      <parent link="${prefix}shoulder_link" />
-      <child link="${prefix}upper_arm_link" />
+    <joint name="${tf_prefix}shoulder_lift_joint" type="revolute">
+      <parent link="${tf_prefix}shoulder_link" />
+      <child link="${tf_prefix}upper_arm_link" />
       <origin xyz="${upper_arm_x} ${upper_arm_y} ${upper_arm_z}" rpy="${upper_arm_roll} ${upper_arm_pitch} ${upper_arm_yaw}" />
       <axis xyz="0 0 1" />
@@ -293,7 +293,7 @@
       <dynamics damping="0" friction="0"/>
     </joint>
-    <joint name="${prefix}elbow_joint" type="revolute">
-      <parent link="${prefix}upper_arm_link" />
-      <child link="${prefix}forearm_link" />
+    <joint name="${tf_prefix}elbow_joint" type="revolute">
+      <parent link="${tf_prefix}upper_arm_link" />
+      <child link="${tf_prefix}forearm_link" />
       <origin xyz="${forearm_x} ${forearm_y} ${forearm_z}" rpy="${forearm_roll} ${forearm_pitch} ${forearm_yaw}" />
       <axis xyz="0 0 1" />
@@ -305,7 +305,7 @@
       <dynamics damping="0" friction="0"/>
     </joint>
-    <joint name="${prefix}wrist_1_joint" type="revolute">
-      <parent link="${prefix}forearm_link" />
-      <child link="${prefix}wrist_1_link" />
+    <joint name="${tf_prefix}wrist_1_joint" type="revolute">
+      <parent link="${tf_prefix}forearm_link" />
+      <child link="${tf_prefix}wrist_1_link" />
       <origin xyz="${wrist_1_x} ${wrist_1_y} ${wrist_1_z}" rpy="${wrist_1_roll} ${wrist_1_pitch} ${wrist_1_yaw}" />
       <axis xyz="0 0 1" />
@@ -317,7 +317,7 @@
       <dynamics damping="0" friction="0"/>
     </joint>
-    <joint name="${prefix}wrist_2_joint" type="revolute">
-      <parent link="${prefix}wrist_1_link" />
-      <child link="${prefix}wrist_2_link" />
+    <joint name="${tf_prefix}wrist_2_joint" type="revolute">
+      <parent link="${tf_prefix}wrist_1_link" />
+      <child link="${tf_prefix}wrist_2_link" />
       <origin xyz="${wrist_2_x} ${wrist_2_y} ${wrist_2_z}" rpy="${wrist_2_roll} ${wrist_2_pitch} ${wrist_2_yaw}" />
       <axis xyz="0 0 1" />
@@ -329,7 +329,7 @@
       <dynamics damping="0" friction="0"/>
     </joint>
-    <joint name="${prefix}wrist_3_joint" type="revolute">
-      <parent link="${prefix}wrist_2_link" />
-      <child link="${prefix}wrist_3_link" />
+    <joint name="${tf_prefix}wrist_3_joint" type="revolute">
+      <parent link="${tf_prefix}wrist_2_link" />
+      <child link="${tf_prefix}wrist_3_link" />
       <origin xyz="${wrist_3_x} ${wrist_3_y} ${wrist_3_z}" rpy="${wrist_3_roll} ${wrist_3_pitch} ${wrist_3_yaw}" />
       <axis xyz="0 0 1" />
@@ -341,13 +341,13 @@
       <dynamics damping="0" friction="0"/>
     </joint>
-    <link name="${prefix}ft_frame"/>
-    <joint name="${prefix}wrist_3_link-ft_frame" type="fixed">
-      <parent link="${prefix}wrist_3_link"/>
-      <child link="${prefix}ft_frame"/>
+    <link name="${tf_prefix}ft_frame"/>
+    <joint name="${tf_prefix}wrist_3_link-ft_frame" type="fixed">
+      <parent link="${tf_prefix}wrist_3_link"/>
+      <child link="${tf_prefix}ft_frame"/>
       <origin xyz="0 0 0" rpy="${pi} 0 0"/>
     </joint>
     <!-- ROS-Industrial 'base' frame - base_link to UR 'Base' Coordinates transform -->
-    <link name="${prefix}base"/>
-    <joint name="${prefix}base_link-base_fixed_joint" type="fixed">
+    <link name="${tf_prefix}base"/>
+    <joint name="${tf_prefix}base_link-base_fixed_joint" type="fixed">
       <!-- Note the rotation over Z of pi radians - as base_link is REP-103
            aligned (i.e., has X+ forward, Y+ left and Z+ up), this is needed
@@ -356,21 +356,21 @@
       -->
       <origin xyz="0 0 0" rpy="0 0 ${pi}"/>
-      <parent link="${prefix}base_link"/>
-      <child link="${prefix}base"/>
+      <parent link="${tf_prefix}base_link"/>
+      <child link="${tf_prefix}base"/>
     </joint>
     <!-- ROS-Industrial 'flange' frame - attachment point for EEF models -->
-    <link name="${prefix}flange" />
-    <joint name="${prefix}wrist_3-flange" type="fixed">
-      <parent link="${prefix}wrist_3_link" />
-      <child link="${prefix}flange" />
+    <link name="${tf_prefix}flange" />
+    <joint name="${tf_prefix}wrist_3-flange" type="fixed">
+      <parent link="${tf_prefix}wrist_3_link" />
+      <child link="${tf_prefix}flange" />
       <origin xyz="0 0 0" rpy="0 ${-pi/2.0} ${-pi/2.0}" />
     </joint>
     <!-- ROS-Industrial 'tool0' frame - all-zeros tool frame -->
-    <link name="${prefix}tool0"/>
-    <joint name="${prefix}flange-tool0" type="fixed">
+    <link name="${tf_prefix}tool0"/>
+    <joint name="${tf_prefix}flange-tool0" type="fixed">
       <!-- default toolframe - X+ left, Y+ up, Z+ front -->
       <origin xyz="0 0 0" rpy="${pi/2.0} 0 ${pi/2.0}"/>
-      <parent link="${prefix}flange"/>
-      <child link="${prefix}tool0"/>
+      <parent link="${tf_prefix}flange"/>
+      <child link="${tf_prefix}tool0"/>
     </joint>
   </xacro:macro>
