Commit message: Ignition Gazebo simulation for UR robots (#232)
* Make ur and ignition happy

* More ur sim stuff

* Remove pycache

* Remove visual colors, so colors are read from dae

* Better tuning

* Organizational changes, docs and a little more tuning

* More organizational changes

* Move world link outside xacro if

* pre-commit fixes

* Add ros_ign to repos

* Better tuning = less jerkiness

* Re-tuning

* Apply suggestions from code review

Co-authored-by: AndyZe <andyz@utexas.edu>

* Add comments on environment hooks

Co-authored-by: AndyZe <andyz@utexas.edu>

File: urdf/ur.urdf.xacro (robot description, xacro)
@@ -21,4 +21,6 @@
    <!-- initial position for fake hardware -->
    <xacro:arg name="initial_positions_file" default="$(find ur_description)/config/initial_positions.yaml"/>
+   <!-- Simulation parameter -->
+   <xacro:arg name="ignition" default="false" />
    <!-- convert to property to use substitution in function -->
    <xacro:property name="initial_positions_file" default="$(arg initial_positions_file)"/>
@@ -37,4 +39,5 @@
      fake_sensor_commands="$(arg fake_sensor_commands)"
      headless_mode="$(arg headless_mode)"
-     initial_positions="${load_yaml(initial_positions_file)}" />
+     initial_positions="${load_yaml(initial_positions_file)}"
+     ignition="$(arg ignition)" />
 </robot>

File: urdf/ur_macro.xacro (robot description, xacro)
@@ -57,4 +57,5 @@
     fake_sensor_commands:=false
     headless_mode:=false
+    ignition:=false
     initial_positions:=${dict(shoulder_pan_joint=0.0,shoulder_lift_joint=-1.57,elbow_joint=0.0,wrist_1_joint=-1.57,wrist_2_joint=0.0,wrist_3_joint=0.0)}">
     <!-- Load configuration data from the provided .yaml files -->
@@ -95,7 +96,4 @@
           <mesh filename="${base_visual_mesh}"/>
         </geometry>
-        <material name="${base_visual_material_name}">
-          <color rgba="${base_visual_material_color}"/>
-        </material>
       </visual>
       <collision>
@@ -115,7 +113,4 @@
           <mesh filename="${shoulder_visual_mesh}"/>
         </geometry>
-        <material name="${shoulder_visual_material_name}">
-          <color rgba="${shoulder_visual_material_color}"/>
-        </material>
       </visual>
       <collision>
@@ -135,7 +130,4 @@
           <mesh filename="${upper_arm_visual_mesh}"/>
         </geometry>
-        <material name="${upper_arm_visual_material_name}">
-          <color rgba="${upper_arm_visual_material_color}"/>
-        </material>
       </visual>
       <collision>
@@ -155,7 +147,4 @@
           <mesh filename="${forearm_visual_mesh}"/>
         </geometry>
-        <material name="${forearm_visual_material_name}">
-          <color rgba="${forearm_visual_material_color}"/>
-        </material>
       </visual>
       <collision>
@@ -175,7 +164,4 @@
           <mesh filename="${wrist_1_visual_mesh}"/>
         </geometry>
-        <material name="${wrist_1_visual_material_name}">
-          <color rgba="${wrist_1_visual_material_color}"/>
-        </material>
       </visual>
       <collision>
@@ -195,7 +181,4 @@
           <mesh filename="${wrist_2_visual_mesh}"/>
         </geometry>
-        <material name="${wrist_2_visual_material_name}">
-          <color rgba="${wrist_2_visual_material_color}"/>
-        </material>
       </visual>
       <collision>
@@ -215,7 +198,4 @@
           <mesh filename="${wrist_3_visual_mesh}"/>
         </geometry>
-        <material name="${wrist_3_visual_material_name}">
-          <color rgba="${wrist_3_visual_material_color}"/>
-        </material>
       </visual>
       <collision>
@@ -250,5 +230,5 @@
          <safety_controller soft_lower_limit="${shoulder_pan_lower_limit + safety_pos_margin}" soft_upper_limit="${shoulder_pan_upper_limit - safety_pos_margin}" k_position="${safety_k_position}" k_velocity="0.0"/>
       </xacro:if>
-      <dynamics damping="0" friction="0"/>
+      <dynamics damping="5" friction="5"/>
     </joint>
     <joint name="${prefix}shoulder_lift_joint" type="revolute">
@@ -262,5 +242,5 @@
          <safety_controller soft_lower_limit="${shoulder_lift_lower_limit + safety_pos_margin}" soft_upper_limit="${shoulder_lift_upper_limit - safety_pos_margin}" k_position="${safety_k_position}" k_velocity="0.0"/>
       </xacro:if>
-      <dynamics damping="0" friction="0"/>
+      <dynamics damping="5" friction="5"/>
     </joint>
     <joint name="${prefix}elbow_joint" type="revolute">
@@ -274,5 +254,5 @@
          <safety_controller soft_lower_limit="${elbow_joint_lower_limit + safety_pos_margin}" soft_upper_limit="${elbow_joint_upper_limit - safety_pos_margin}" k_position="${safety_k_position}" k_velocity="0.0"/>
       </xacro:if>
-      <dynamics damping="0" friction="0"/>
+      <dynamics damping="5" friction="5"/>
     </joint>
     <joint name="${prefix}wrist_1_joint" type="revolute">
@@ -286,5 +266,5 @@
          <safety_controller soft_lower_limit="${wrist_1_lower_limit + safety_pos_margin}" soft_upper_limit="${wrist_1_upper_limit - safety_pos_margin}" k_position="${safety_k_position}" k_velocity="0.0"/>
       </xacro:if>
-      <dynamics damping="0" friction="0"/>
+      <dynamics damping="5" friction="5"/>
     </joint>
     <joint name="${prefix}wrist_2_joint" type="revolute">
@@ -298,5 +278,5 @@
          <safety_controller soft_lower_limit="${wrist_2_lower_limit + safety_pos_margin}" soft_upper_limit="${wrist_2_upper_limit - safety_pos_margin}" k_position="${safety_k_position}" k_velocity="0.0"/>
       </xacro:if>
-      <dynamics damping="0" friction="0"/>
+      <dynamics damping="5" friction="5"/>
     </joint>
     <joint name="${prefix}wrist_3_joint" type="revolute">
@@ -310,5 +290,5 @@
          <safety_controller soft_lower_limit="${wrist_3_lower_limit + safety_pos_margin}" soft_upper_limit="${wrist_3_upper_limit - safety_pos_margin}" k_position="${safety_k_position}" k_velocity="0.0"/>
       </xacro:if>
-      <dynamics damping="0" friction="0"/>
+      <dynamics damping="5" friction="5"/>
     </joint>
     <!-- ROS-Industrial 'base' frame - base_link to UR 'Base' Coordinates transform -->
@@ -339,4 +319,16 @@
       <child link="${prefix}tool0"/>
     </joint>
+    <!-- Create a world link, and a fixed joint between world and base_link -->
+    <link name="world" />
+    <joint name="${prefix}world_joint"  type="fixed">
+      <origin xyz="0 0 0" rpy="0 0 0" />
+      <parent link="world"/>
+      <child link="${prefix}base_link"/>
+    </joint>
+    <!-- Ignition Gazebo -->
+    <xacro:if value="${ignition}">
+      <!-- Include Ignition Gazebo Plugins -->
+      <xacro:include filename="ur_ignition_plugins.xacro" />
+    </xacro:if>
   </xacro:macro>
 </robot>

Commit message: Revert "Ignition Gazebo simulation for UR robots (#232)" (#241)
This reverts commit 28ef61d366fba93dbb4703537006fc7cb83c0c92.

File: urdf/ur.urdf.xacro (robot description, xacro)
@@ -21,6 +21,4 @@
    <!-- initial position for fake hardware -->
    <xacro:arg name="initial_positions_file" default="$(find ur_description)/config/initial_positions.yaml"/>
-   <!-- Simulation parameter -->
-   <xacro:arg name="ignition" default="false" />
    <!-- convert to property to use substitution in function -->
    <xacro:property name="initial_positions_file" default="$(arg initial_positions_file)"/>
@@ -39,5 +37,4 @@
      fake_sensor_commands="$(arg fake_sensor_commands)"
      headless_mode="$(arg headless_mode)"
-     initial_positions="${load_yaml(initial_positions_file)}"
-     ignition="$(arg ignition)" />
+     initial_positions="${load_yaml(initial_positions_file)}" />
 </robot>

File: urdf/ur_macro.xacro (robot description, xacro)
@@ -57,5 +57,4 @@
     fake_sensor_commands:=false
     headless_mode:=false
-    ignition:=false
     initial_positions:=${dict(shoulder_pan_joint=0.0,shoulder_lift_joint=-1.57,elbow_joint=0.0,wrist_1_joint=-1.57,wrist_2_joint=0.0,wrist_3_joint=0.0)}">
     <!-- Load configuration data from the provided .yaml files -->
@@ -96,4 +95,7 @@
           <mesh filename="${base_visual_mesh}"/>
         </geometry>
+        <material name="${base_visual_material_name}">
+          <color rgba="${base_visual_material_color}"/>
+        </material>
       </visual>
       <collision>
@@ -113,4 +115,7 @@
           <mesh filename="${shoulder_visual_mesh}"/>
         </geometry>
+        <material name="${shoulder_visual_material_name}">
+          <color rgba="${shoulder_visual_material_color}"/>
+        </material>
       </visual>
       <collision>
@@ -130,4 +135,7 @@
           <mesh filename="${upper_arm_visual_mesh}"/>
         </geometry>
+        <material name="${upper_arm_visual_material_name}">
+          <color rgba="${upper_arm_visual_material_color}"/>
+        </material>
       </visual>
       <collision>
@@ -147,4 +155,7 @@
           <mesh filename="${forearm_visual_mesh}"/>
         </geometry>
+        <material name="${forearm_visual_material_name}">
+          <color rgba="${forearm_visual_material_color}"/>
+        </material>
       </visual>
       <collision>
@@ -164,4 +175,7 @@
           <mesh filename="${wrist_1_visual_mesh}"/>
         </geometry>
+        <material name="${wrist_1_visual_material_name}">
+          <color rgba="${wrist_1_visual_material_color}"/>
+        </material>
       </visual>
       <collision>
@@ -181,4 +195,7 @@
           <mesh filename="${wrist_2_visual_mesh}"/>
         </geometry>
+        <material name="${wrist_2_visual_material_name}">
+          <color rgba="${wrist_2_visual_material_color}"/>
+        </material>
       </visual>
       <collision>
@@ -198,4 +215,7 @@
           <mesh filename="${wrist_3_visual_mesh}"/>
         </geometry>
+        <material name="${wrist_3_visual_material_name}">
+          <color rgba="${wrist_3_visual_material_color}"/>
+        </material>
       </visual>
       <collision>
@@ -230,5 +250,5 @@
          <safety_controller soft_lower_limit="${shoulder_pan_lower_limit + safety_pos_margin}" soft_upper_limit="${shoulder_pan_upper_limit - safety_pos_margin}" k_position="${safety_k_position}" k_velocity="0.0"/>
       </xacro:if>
-      <dynamics damping="5" friction="5"/>
+      <dynamics damping="0" friction="0"/>
     </joint>
     <joint name="${prefix}shoulder_lift_joint" type="revolute">
@@ -242,5 +262,5 @@
          <safety_controller soft_lower_limit="${shoulder_lift_lower_limit + safety_pos_margin}" soft_upper_limit="${shoulder_lift_upper_limit - safety_pos_margin}" k_position="${safety_k_position}" k_velocity="0.0"/>
       </xacro:if>
-      <dynamics damping="5" friction="5"/>
+      <dynamics damping="0" friction="0"/>
     </joint>
     <joint name="${prefix}elbow_joint" type="revolute">
@@ -254,5 +274,5 @@
          <safety_controller soft_lower_limit="${elbow_joint_lower_limit + safety_pos_margin}" soft_upper_limit="${elbow_joint_upper_limit - safety_pos_margin}" k_position="${safety_k_position}" k_velocity="0.0"/>
       </xacro:if>
-      <dynamics damping="5" friction="5"/>
+      <dynamics damping="0" friction="0"/>
     </joint>
     <joint name="${prefix}wrist_1_joint" type="revolute">
@@ -266,5 +286,5 @@
          <safety_controller soft_lower_limit="${wrist_1_lower_limit + safety_pos_margin}" soft_upper_limit="${wrist_1_upper_limit - safety_pos_margin}" k_position="${safety_k_position}" k_velocity="0.0"/>
       </xacro:if>
-      <dynamics damping="5" friction="5"/>
+      <dynamics damping="0" friction="0"/>
     </joint>
     <joint name="${prefix}wrist_2_joint" type="revolute">
@@ -278,5 +298,5 @@
          <safety_controller soft_lower_limit="${wrist_2_lower_limit + safety_pos_margin}" soft_upper_limit="${wrist_2_upper_limit - safety_pos_margin}" k_position="${safety_k_position}" k_velocity="0.0"/>
       </xacro:if>
-      <dynamics damping="5" friction="5"/>
+      <dynamics damping="0" friction="0"/>
     </joint>
     <joint name="${prefix}wrist_3_joint" type="revolute">
@@ -290,5 +310,5 @@
          <safety_controller soft_lower_limit="${wrist_3_lower_limit + safety_pos_margin}" soft_upper_limit="${wrist_3_upper_limit - safety_pos_margin}" k_position="${safety_k_position}" k_velocity="0.0"/>
       </xacro:if>
-      <dynamics damping="5" friction="5"/>
+      <dynamics damping="0" friction="0"/>
     </joint>
     <!-- ROS-Industrial 'base' frame - base_link to UR 'Base' Coordinates transform -->
@@ -319,16 +339,4 @@
       <child link="${prefix}tool0"/>
     </joint>
-    <!-- Create a world link, and a fixed joint between world and base_link -->
-    <link name="world" />
-    <joint name="${prefix}world_joint"  type="fixed">
-      <origin xyz="0 0 0" rpy="0 0 0" />
-      <parent link="world"/>
-      <child link="${prefix}base_link"/>
-    </joint>
-    <!-- Ignition Gazebo -->
-    <xacro:if value="${ignition}">
-      <!-- Include Ignition Gazebo Plugins -->
-      <xacro:include filename="ur_ignition_plugins.xacro" />
-    </xacro:if>
   </xacro:macro>
 </robot>

Commit message: Add options to position robot when importing macro.

File: urdf/ur.urdf.xacro (robot description, xacro)
@@ -24,7 +24,11 @@
    <!-- convert to property to use substitution in function -->
    <xacro:property name="initial_positions_file" default="$(arg initial_positions_file)"/>
+   <!-- create link fixed to the "world" -->
+   <link name="world" />
    <!-- arm -->
    <xacro:ur_robot
+     name="$(arg name)"
      prefix="$(arg prefix)"
+     parent="world"
      joint_limits_parameters_file="$(arg joint_limit_params)"
      kinematics_parameters_file="$(arg kinematics_params)"
@@ -39,4 +43,6 @@
      headless_mode="$(arg headless_mode)"
      initial_positions="${load_yaml(initial_positions_file)}"
-     use_tool_communication="$(arg use_tool_communication)" />
+     use_tool_communication="$(arg use_tool_communication)" >
+     <origin xyz="0 0 0" rpy="0 0 0" />          <!-- position robot in the world -->
+   </xacro:ur_robot>
 </robot>

File: urdf/ur_macro.xacro (robot description, xacro)
@@ -45,5 +45,8 @@
   <xacro:include filename="$(find ur_description)/urdf/inc/ur_common.xacro" />
   <xacro:macro name="ur_robot" params="
+    name
     prefix
+    parent
+    *origin
     joint_limits_parameters_file
     kinematics_parameters_file
@@ -74,5 +77,5 @@
     <!-- ros2 control instance -->
     <xacro:ur_ros2_control
-      name="URPositionHardwareInterface" prefix="${prefix}"
+      name="${name}" prefix="${prefix}"
       use_fake_hardware="$(arg use_fake_hardware)"
       initial_positions="${initial_positions}"
@@ -231,4 +234,10 @@
       </xacro:cylinder_inertial>
     </link>
+    <!-- base_joint fixes base_link to the environment -->
+    <joint name="${prefix}base_joint" type="fixed">
+      <xacro:insert_block name="origin" />
+      <parent link="${parent}" />
+      <child link="${prefix}base_link" />
+    </joint>
     <!-- joints - main serial chain -->
     <joint name="${prefix}base_link-base_link_inertia" type="fixed">

Commit message: Remove special urdf files for simulation and update configuration of unified files.

File: urdf/ur.urdf.xacro (robot description, xacro)
@@ -16,8 +16,12 @@
    <xacro:arg name="safety_k_position" default="20"/>
    <!-- ros2_control related parameters -->
+   <xacro:arg name="headless_mode" default="false" />
+   <xacro:arg name="use_tool_communication" default="false" />
+     <!-- Simulation parameters -->
    <xacro:arg name="use_fake_hardware" default="false" />
    <xacro:arg name="fake_sensor_commands" default="false" />
-   <xacro:arg name="headless_mode" default="false" />
-   <xacro:arg name="use_tool_communication" default="false" />
+   <xacro:arg name="sim_gazebo" default="false" />
+   <xacro:arg name="sim_ignition" default="false" />
+   <xacro:arg name="simulation_controllers" default="$(find ur_bringup)/config/ur_controllers.yaml" />
    <!-- initial position for fake hardware -->
    <xacro:arg name="initial_positions_file" default="$(find ur_description)/config/initial_positions.yaml"/>
@@ -41,4 +45,6 @@
      use_fake_hardware="$(arg use_fake_hardware)"
      fake_sensor_commands="$(arg fake_sensor_commands)"
+     sim_gazebo="$(arg sim_gazebo)"
+     sim_ignition="$(arg sim_ignition)"
      headless_mode="$(arg headless_mode)"
      initial_positions="${load_yaml(initial_positions_file)}"
@@ -46,3 +52,24 @@
      <origin xyz="0 0 0" rpy="0 0 0" />          <!-- position robot in the world -->
    </xacro:ur_robot>
+   <xacro:if value="$(arg sim_gazebo)">
+    <!-- Gazebo plugins -->
+    <gazebo reference="world">
+    </gazebo>
+    <gazebo>
+      <plugin filename="libgazebo_ros2_control.so" name="gazebo_ros2_control">
+        <parameters>$(arg simulation_controllers)</parameters>
+      </plugin>
+    </gazebo>
+  </xacro:if>
+  <xacro:if value="$(arg sim_ignition)">
+    <!-- Gazebo plugins -->
+    <gazebo reference="world">
+    </gazebo>
+    <gazebo>
+      <plugin filename="libign_ros2_control-system.so" name="ign_ros2_control::IgnitionROS2ControlPlugin">
+        <parameters>$(arg simulation_controllers)</parameters>
+        <controller_manager_node_name>$(arg prefix)controller_manager</controller_manager_node_name>
+      </plugin>
+    </gazebo>
+  </xacro:if>
 </robot>

File: urdf/ur_macro.xacro (robot description, xacro)
@@ -59,4 +59,6 @@
     use_fake_hardware:=false
     fake_sensor_commands:=false
+    sim_gazebo:=false
+    sim_ignition:=false
     headless_mode:=false
     initial_positions:=${dict(shoulder_pan_joint=0.0,shoulder_lift_joint=-1.57,elbow_joint=0.0,wrist_1_joint=-1.57,wrist_2_joint=0.0,wrist_3_joint=0.0)}
@@ -82,4 +84,6 @@
       fake_sensor_commands="${fake_sensor_commands}"
       headless_mode="${headless_mode}"
+      sim_gazebo="$(arg sim_gazebo)"
+      sim_ignition="$(arg sim_ignition)"
       script_filename="$(arg script_filename)"
       output_recipe_filename="$(arg output_recipe_filename)"
@@ -302,4 +306,10 @@
       <dynamics damping="0" friction="0"/>
     </joint>
+    <link name="${prefix}ft_frame"/>
+    <joint name="${prefix}wrist_3_link-ft_frame" type="fixed">
+      <parent link="${prefix}wrist_3_link"/>
+      <child link="${prefix}ft_frame"/>
+      <origin xyz="0 0 0" rpy="${pi} 0 0"/>
+    </joint>
     <!-- ROS-Industrial 'base' frame - base_link to UR 'Base' Coordinates transform -->
     <link name="${prefix}base"/>

Commit message: Revert test dynamics specification

File: urdf/ur.urdf.xacro (robot description, xacro)
@@ -48,6 +48,4 @@
    <!-- create link fixed to the "world" -->
    <link name="world" />
-   <xacro:property name="joint_dynamics_file" value="$(find ur_description)/config/test_joint_dyn.yaml"/>
-   <xacro:property name="joint_dynamics_dict" value="${xacro.load_yaml(joint_dynamics_file)}"/>
    <!-- arm -->
    <xacro:ur_robot
@@ -59,5 +57,4 @@
      physical_parameters_file="$(arg physical_params)"
      visual_parameters_file="$(arg visual_params)"
-     joint_dynamics="${joint_dynamics_dict}"
      transmission_hw_interface="$(arg transmission_hw_interface)"
      safety_limits="$(arg safety_limits)"

Commit message: Simplify file names

File: urdf/ur.urdf.xacro (robot description, xacro)
@@ -44,9 +44,9 @@
    <!-- initial position for simulations (Fake Hardware, Gazebo, Ignition) -->
    <xacro:arg name="initial_positions_file" default="$(find ur_description)/config/initial_positions.yaml"/>
-   <!-- Default joint dynamics, useful to specialize for simulations -->
-   <xacro:arg name="joint_dynamics_defaults_file" default="$(find ur_description)/config/joint_dynamics_defaults.yaml"/>
+   <!-- Default joint dynamics has friction and damping equal to 0, but useful to specialize for simulations -->
+   <xacro:arg name="joint_dynamics_file" default="$(find ur_description)/config/joint_dynamics.yaml"/>
    <!-- convert to property to use substitution in function -->
    <xacro:property name="initial_positions_file" default="$(arg initial_positions_file)"/>
-   <xacro:property name="joint_dynamics_defaults_file" default="$(arg joint_dynamics_defaults_file)"/>
+   <xacro:property name="joint_dynamics_file" default="$(arg joint_dynamics_file)"/>
    <!-- create link fixed to the "world" -->
    <link name="world" />
@@ -70,5 +70,5 @@
      headless_mode="$(arg headless_mode)"
      initial_positions="${xacro.load_yaml(initial_positions_file)}"
-     joint_dynamics="${xacro.load_yaml(joint_dynamics_defaults_file)}"
+     joint_dynamics="${xacro.load_yaml(joint_dynamics_file)}"
      use_tool_communication="$(arg use_tool_communication)"
      tool_voltage="$(arg tool_voltage)"
