Commit message: Reverted link base_link_inertia rename.

File: urdf/ur_macro.xacro (robot description, xacro)
@@ -132,11 +132,23 @@
     <!-- Placeholder for ros2_control transmission which don't yet exist -->
     <!-- links -  main serial chain -->
-    <link name="${prefix}base_link_fixed"/>
-    <xacro:new_link name="base">
-      <origin xyz="0 0 0" rpy="0 0 ${pi}"/>
+	<!-- Special exception in creation is the base_link_inertia, as naming convention is slightly different from other links which use xacro:new_link. -->
+    <link name="${prefix}base_link"/>
+    <link name="${prefix}base_link_inertia">
+      <visual>
+        <origin xyz="0 0 0" rpy="0 0 ${pi}"/>
+        <geometry>
+          <xacro:get_mesh name="base" type="visual"/>
+        </geometry>
+      </visual>
+      <collision>
+        <origin xyz="0 0 0" rpy="0 0 ${pi}"/>
+        <geometry>
+          <xacro:get_mesh name="base" type="collision"/>
+        </geometry>
+      </collision>
       <xacro:cylinder_inertial radius="${base_inertia_radius}" length="${base_inertia_length}" mass="${base_mass}">
         <origin xyz="0 0 0" rpy="0 0 0" />
       </xacro:cylinder_inertial>
-    </xacro:new_link>
+    </link>
     <xacro:new_link name="shoulder">
       <origin xyz="0 0 0" rpy="0 0 ${pi}"/>
@@ -178,24 +190,23 @@
       </xacro:cylinder_inertial>
     </xacro:new_link>
-    <!-- base_joint fixes base_link_fixed to the environment -->
+    <!-- base_joint fixes base_link to the environment -->
     <joint name="${prefix}base_joint" type="fixed">
       <xacro:insert_block name="origin" />
       <parent link="${parent}" />
-      <child link="${prefix}base_link_fixed" />
+      <child link="${prefix}base_link" />
     </joint>
     <!-- joints - main serial chain -->
-    <joint name="${prefix}base_link_fixed-base_link" type="fixed">
-      <parent link="${prefix}base_link_fixed" />
-      <child link="${prefix}base_link" />
+    <joint name="${prefix}base_link-base_link_inertia" type="fixed">
+      <parent link="${prefix}base_link" />
+      <child link="${prefix}base_link_inertia" />
       <!-- 'base_link' is REP-103 aligned (so X+ forward), while the internal
            frames of the robot/controller have X+ pointing backwards.
-           Use the joint between 'base_link_fixed' and 'base_link' (a dummy
+           Use the joint between 'base_link' and 'base_link_inertia' (a dummy
            link/frame) to introduce the necessary rotation over Z (of pi rad).
       -->
       <origin xyz="0 0 0" rpy="0 0 ${pi}" />
     </joint>
-    <!-- TODO- Rename these conventions to add a xmacro for the creation of new_revolute_joints -->
     <joint name="${prefix}shoulder_pan_joint" type="revolute">
-      <parent link="${prefix}base_link" />
+      <parent link="${prefix}base_link_inertia" />
       <child link="${prefix}shoulder_link" />
       <origin xyz="${shoulder_x} ${shoulder_y} ${shoulder_z}" rpy="${shoulder_roll} ${shoulder_pitch} ${shoulder_yaw}" />
@@ -283,5 +294,5 @@
       -->
       <origin xyz="0 0 0" rpy="0 0 ${pi}"/>
-      <parent link="${prefix}base_link_fixed"/>
+      <parent link="${prefix}base_link"/>
       <child link="${prefix}base"/>
     </joint>

Commit message: Revert new_link macro in "Simplification of xacro code for URDF generation"
This reverts commit parts of 609f1b09c1f256422ec97bf6117e548fba58717a.

File: urdf/ur_macro.xacro (robot description, xacro)
@@ -44,22 +44,4 @@
   <xacro:include filename="$(find ur_description)/urdf/inc/ur_transmissions.xacro" />
   <xacro:include filename="$(find ur_description)/urdf/inc/ur_common.xacro" />
-  <!-- Simplification for link creation -->
-  <xacro:macro name="new_link" params="name *mesh_origin **cylinder">
-    <link name="${prefix}${name}_link">
-      <visual>
-        <xacro:insert_block name="mesh_origin"/>
-        <geometry>
-          <xacro:get_mesh name="${name}" type="visual"/>
-        </geometry>
-      </visual>
-      <collision>
-        <xacro:insert_block name="mesh_origin"/>
-        <geometry>
-          <xacro:get_mesh name="${name}" type="collision"/>
-        </geometry>
-      </collision>
-      <xacro:insert_block name="cylinder"/>
-    </link>
-  </xacro:macro>
   <xacro:macro name="ur_robot" params="
     name
@@ -132,5 +114,4 @@
     <!-- Placeholder for ros2_control transmission which don't yet exist -->
     <!-- links -  main serial chain -->
-	<!-- Special exception in creation is the base_link_inertia, as naming convention is slightly different from other links which use xacro:new_link. -->
     <link name="${prefix}base_link"/>
     <link name="${prefix}base_link_inertia">
@@ -151,43 +132,109 @@
       </xacro:cylinder_inertial>
     </link>
-    <xacro:new_link name="shoulder">
-      <origin xyz="0 0 0" rpy="0 0 ${pi}"/>
+    <link name="${prefix}shoulder_link">
+      <visual>
+        <origin xyz="0 0 0" rpy="0 0 ${pi}"/>
+        <geometry>
+          <xacro:get_mesh name="shoulder" type="visual"/>
+        </geometry>
+      </visual>
+      <collision>
+        <origin xyz="0 0 0" rpy="0 0 ${pi}"/>
+        <geometry>
+          <xacro:get_mesh name="shoulder" type="collision"/>
+        </geometry>
+      </collision>
       <xacro:cylinder_inertial radius="${shoulder_inertia_radius}" length="${shoulder_inertia_length}" mass="${shoulder_mass}">
         <origin xyz="0 0 0" rpy="0 0 0" />
       </xacro:cylinder_inertial>
-    </xacro:new_link>
-    <xacro:new_link name="upper_arm">
-      <origin xyz="0 0 ${shoulder_offset}" rpy="${pi/2} 0 ${-pi/2}"/>
+    </link>
+    <link name="${prefix}upper_arm_link">
+      <visual>
+        <origin xyz="0 0 ${shoulder_offset}" rpy="${pi/2} 0 ${-pi/2}"/>
+        <geometry>
+          <xacro:get_mesh name="upper_arm" type="visual"/>
+        </geometry>
+      </visual>
+      <collision>
+        <origin xyz="0 0 ${shoulder_offset}" rpy="${pi/2} 0 ${-pi/2}"/>
+        <geometry>
+          <xacro:get_mesh name="upper_arm" type="collision"/>
+        </geometry>
+      </collision>
       <xacro:cylinder_inertial radius="${upperarm_inertia_radius}" length="${upperarm_inertia_length}" mass="${upper_arm_mass}">
         <origin xyz="${-0.5 * upperarm_inertia_length} 0.0 ${upper_arm_inertia_offset}" rpy="0 ${pi/2} 0" />
       </xacro:cylinder_inertial>
-    </xacro:new_link>
-    <xacro:new_link name="forearm">
-      <origin xyz="0 0 ${elbow_offset}" rpy="${pi/2} 0 ${-pi/2}"/>
+    </link>
+    <link name="${prefix}forearm_link">
+      <visual>
+        <origin xyz="0 0 ${elbow_offset}" rpy="${pi/2} 0 ${-pi/2}"/>
+        <geometry>
+          <xacro:get_mesh name="forearm" type="visual"/>
+        </geometry>
+      </visual>
+      <collision>
+        <origin xyz="0 0 ${elbow_offset}" rpy="${pi/2} 0 ${-pi/2}"/>
+        <geometry>
+          <xacro:get_mesh name="forearm" type="collision"/>
+        </geometry>
+      </collision>
       <xacro:cylinder_inertial radius="${forearm_inertia_radius}" length="${forearm_inertia_length}"  mass="${forearm_mass}">
         <origin xyz="${-0.5 * forearm_inertia_length} 0.0 ${elbow_offset}" rpy="0 ${pi/2} 0" />
       </xacro:cylinder_inertial>
-    </xacro:new_link>
-    <xacro:new_link name="wrist_1">
-      <xacro:get_visual_params name="wrist_1" type="visual_offset"/>
-      <origin xyz="0 0 ${visual_params}" rpy="${pi/2} 0 0"/>
+    </link>
+    <link name="${prefix}wrist_1_link">
+	  <xacro:get_visual_params name="wrist_1" type="visual_offset"/>
+      <visual>
+      	<origin xyz="0 0 ${visual_params}" rpy="${pi/2} 0 0"/>
+        <geometry>
+          <xacro:get_mesh name="wrist_1" type="visual"/>
+        </geometry>
+      </visual>
+      <collision>
+        <origin xyz="0 0 ${visual_params}" rpy="${pi/2} 0 0"/>
+        <geometry>
+          <xacro:get_mesh name="wrist_1" type="collision"/>
+        </geometry>
+      </collision>
       <xacro:cylinder_inertial radius="${wrist_1_inertia_radius}" length="${wrist_1_inertia_length}"  mass="${wrist_1_mass}">
         <origin xyz="0 0 0" rpy="0 0 0" />
       </xacro:cylinder_inertial>
-    </xacro:new_link>
-    <xacro:new_link name="wrist_2">
-      <xacro:get_visual_params name="wrist_2" type="visual_offset"/>
-      <origin xyz="0 0 ${visual_params}" rpy="0 0 0"/>
+    </link>
+    <link name="${prefix}wrist_2_link">
+	  <xacro:get_visual_params name="wrist_2" type="visual_offset"/>
+      <visual>
+        <origin xyz="0 0 ${visual_params}" rpy="0 0 0"/>
+        <geometry>
+          <xacro:get_mesh name="wrist_2" type="visual"/>
+        </geometry>
+      </visual>
+      <collision>
+        <origin xyz="0 0 ${visual_params}" rpy="0 0 0"/>
+        <geometry>
+          <xacro:get_mesh name="wrist_2" type="collision"/>
+        </geometry>
+      </collision>
       <xacro:cylinder_inertial radius="${wrist_2_inertia_radius}" length="${wrist_2_inertia_length}"  mass="${wrist_2_mass}">
         <origin xyz="0 0 0" rpy="0 0 0" />
       </xacro:cylinder_inertial>
-    </xacro:new_link>
-    <xacro:new_link name="wrist_3">
-      <xacro:get_visual_params name="wrist_3" type="visual_offset"/>
-      <origin xyz="0 0 ${visual_params}" rpy="${pi/2} 0 0"/>
+    </link>
+    <link name="${prefix}wrist_3_link">
+	  <xacro:get_visual_params name="wrist_3" type="visual_offset"/>
+      <visual>
+        <origin xyz="0 0 ${visual_params}" rpy="${pi/2} 0 0"/>
+        <geometry>
+          <xacro:get_mesh name="wrist_3" type="visual"/>
+        </geometry>
+      </visual>
+      <collision>
+        <origin xyz="0 0 ${visual_params}" rpy="${pi/2} 0 0"/>
+        <geometry>
+          <xacro:get_mesh name="wrist_3" type="collision"/>
+        </geometry>
+      </collision>
       <xacro:cylinder_inertial radius="${wrist_3_inertia_radius}" length="${wrist_3_inertia_length}"  mass="${wrist_3_mass}">
         <origin xyz="0.0 0.0 ${-0.5 * wrist_3_inertia_length}" rpy="0 0 0" />
       </xacro:cylinder_inertial>
-    </xacro:new_link>
+    </link>
     <!-- base_joint fixes base_link to the environment -->
     <joint name="${prefix}base_joint" type="fixed">

Commit message: Add friction for Gazebo Classic max_force hack

File: urdf/ur_macro.xacro (robot description, xacro)
@@ -262,4 +262,5 @@
       <origin xyz="0 0 0" rpy="0 0 ${pi}" />
     </joint>
+    <!-- Conditional dynamics tags set the joint friction to 100x the joint's effort limit per discussion at Universal_Robots_ROS2_Gazebo_Simulation/issues/19 -->
     <joint name="${prefix}shoulder_pan_joint" type="revolute">
       <parent link="${prefix}base_link_inertia" />
@@ -272,5 +273,5 @@
          <safety_controller soft_lower_limit="${shoulder_pan_lower_limit + safety_pos_margin}" soft_upper_limit="${shoulder_pan_upper_limit - safety_pos_margin}" k_position="${safety_k_position}" k_velocity="0.0"/>
       </xacro:if>
-      <dynamics damping="0" friction="0"/>
+      <dynamics damping="0" friction="${shoulder_pan_effort_limit*100.0 if sim_gazebo else 0}"/>
     </joint>
     <joint name="${prefix}shoulder_lift_joint" type="revolute">
@@ -284,5 +285,5 @@
          <safety_controller soft_lower_limit="${shoulder_lift_lower_limit + safety_pos_margin}" soft_upper_limit="${shoulder_lift_upper_limit - safety_pos_margin}" k_position="${safety_k_position}" k_velocity="0.0"/>
       </xacro:if>
-      <dynamics damping="0" friction="0"/>
+      <dynamics damping="0" friction="${shoulder_lift_effort_limit*100.0 if sim_gazebo else 0}"/>
     </joint>
     <joint name="${prefix}elbow_joint" type="revolute">
@@ -296,5 +297,5 @@
          <safety_controller soft_lower_limit="${elbow_joint_lower_limit + safety_pos_margin}" soft_upper_limit="${elbow_joint_upper_limit - safety_pos_margin}" k_position="${safety_k_position}" k_velocity="0.0"/>
       </xacro:if>
-      <dynamics damping="0" friction="0"/>
+      <dynamics damping="0" friction="${elbow_joint_effort_limit*100.0 if sim_gazebo else 0}"/>
     </joint>
     <joint name="${prefix}wrist_1_joint" type="revolute">
@@ -308,5 +309,5 @@
          <safety_controller soft_lower_limit="${wrist_1_lower_limit + safety_pos_margin}" soft_upper_limit="${wrist_1_upper_limit - safety_pos_margin}" k_position="${safety_k_position}" k_velocity="0.0"/>
       </xacro:if>
-      <dynamics damping="0" friction="0"/>
+      <dynamics damping="0" friction="${wrist_1_effort_limit*100.0 if sim_gazebo else 0}"/>
     </joint>
     <joint name="${prefix}wrist_2_joint" type="revolute">
@@ -320,5 +321,5 @@
          <safety_controller soft_lower_limit="${wrist_2_lower_limit + safety_pos_margin}" soft_upper_limit="${wrist_2_upper_limit - safety_pos_margin}" k_position="${safety_k_position}" k_velocity="0.0"/>
       </xacro:if>
-      <dynamics damping="0" friction="0"/>
+      <dynamics damping="0" friction="${wrist_2_effort_limit*100.0 if sim_gazebo else 0}"/>
     </joint>
     <joint name="${prefix}wrist_3_joint" type="revolute">
@@ -332,5 +333,5 @@
          <safety_controller soft_lower_limit="${wrist_3_lower_limit + safety_pos_margin}" soft_upper_limit="${wrist_3_upper_limit - safety_pos_margin}" k_position="${safety_k_position}" k_velocity="0.0"/>
       </xacro:if>
-      <dynamics damping="0" friction="0"/>
+      <dynamics damping="0" friction="${wrist_3_effort_limit*100.0 if sim_gazebo else 0}"/>
     </joint>
     <link name="${prefix}ft_frame"/>

Commit message: Update dynamic properties (#195)
* Remove unused dh_parameters
* Rename prop__wrist_2_cog to prop_wrist_2_cog for consistency
* Update mass and cog and use full inertia matrix.
* Update max_efforts (torque limits)
* Remove code and values that are no longer needed.

---------

Co-authored-by: Rune Søe-Knudsen <41109954+urrsk@users.noreply.github.com>
(cherry picked from commit 60e6974c65bf5ebe611c51c022cf2eccf88fae32)

File: urdf/ur_macro.xacro (robot description, xacro)
@@ -163,8 +163,16 @@
         </geometry>
       </collision>
-      <xacro:cylinder_inertial radius="${shoulder_inertia_radius}" length="${shoulder_inertia_length}" mass="${shoulder_mass}">
-        <origin xyz="0 0 0" rpy="0 0 0" />
-      </xacro:cylinder_inertial>
-    </link>
+      <inertial>
+        <mass value="${shoulder_mass}"/>
+        <origin rpy="${shoulder_inertia_rotation}" xyz="${shoulder_cog}"/>
+        <inertia
+            ixx="${shoulder_inertia_ixx}"
+            ixy="${shoulder_inertia_ixy}"
+            ixz="${shoulder_inertia_ixz}"
+            iyy="${shoulder_inertia_iyy}"
+            iyz="${shoulder_inertia_iyz}"
+            izz="${shoulder_inertia_izz}"
+        />
+      </inertial>    </link>
     <link name="${tf_prefix}upper_arm_link">
       <visual>
@@ -180,7 +188,16 @@
         </geometry>
       </collision>
-      <xacro:cylinder_inertial radius="${upperarm_inertia_radius}" length="${upperarm_inertia_length}" mass="${upper_arm_mass}">
-        <origin xyz="${-0.5 * upperarm_inertia_length} 0.0 ${upper_arm_inertia_offset}" rpy="0 ${pi/2} 0" />
-      </xacro:cylinder_inertial>
+      <inertial>
+        <mass value="${upper_arm_mass}"/>
+        <origin rpy="${upper_arm_inertia_rotation}" xyz="${upper_arm_cog}"/>
+        <inertia
+            ixx="${upper_arm_inertia_ixx}"
+            ixy="${upper_arm_inertia_ixy}"
+            ixz="${upper_arm_inertia_ixz}"
+            iyy="${upper_arm_inertia_iyy}"
+            iyz="${upper_arm_inertia_iyz}"
+            izz="${upper_arm_inertia_izz}"
+        />
+      </inertial>
     </link>
     <link name="${tf_prefix}forearm_link">
@@ -197,7 +214,16 @@
         </geometry>
       </collision>
-      <xacro:cylinder_inertial radius="${forearm_inertia_radius}" length="${forearm_inertia_length}"  mass="${forearm_mass}">
-        <origin xyz="${-0.5 * forearm_inertia_length} 0.0 ${elbow_offset}" rpy="0 ${pi/2} 0" />
-      </xacro:cylinder_inertial>
+      <inertial>
+        <mass value="${forearm_mass}"/>
+        <origin rpy="${forearm_inertia_rotation}" xyz="${forearm_cog}"/>
+        <inertia
+            ixx="${forearm_inertia_ixx}"
+            ixy="${forearm_inertia_ixy}"
+            ixz="${forearm_inertia_ixz}"
+            iyy="${forearm_inertia_iyy}"
+            iyz="${forearm_inertia_iyz}"
+            izz="${forearm_inertia_izz}"
+        />
+      </inertial>
     </link>
     <link name="${tf_prefix}wrist_1_link">
@@ -215,7 +241,16 @@
         </geometry>
       </collision>
-      <xacro:cylinder_inertial radius="${wrist_1_inertia_radius}" length="${wrist_1_inertia_length}"  mass="${wrist_1_mass}">
-        <origin xyz="0 0 0" rpy="0 0 0" />
-      </xacro:cylinder_inertial>
+      <inertial>
+        <mass value="${wrist_1_mass}"/>
+        <origin rpy="${wrist_1_inertia_rotation}" xyz="${wrist_1_cog}"/>
+        <inertia
+            ixx="${wrist_1_inertia_ixx}"
+            ixy="${wrist_1_inertia_ixy}"
+            ixz="${wrist_1_inertia_ixz}"
+            iyy="${wrist_1_inertia_iyy}"
+            iyz="${wrist_1_inertia_iyz}"
+            izz="${wrist_1_inertia_izz}"
+        />
+      </inertial>
     </link>
     <link name="${tf_prefix}wrist_2_link">
@@ -233,7 +268,16 @@
         </geometry>
       </collision>
-      <xacro:cylinder_inertial radius="${wrist_2_inertia_radius}" length="${wrist_2_inertia_length}"  mass="${wrist_2_mass}">
-        <origin xyz="0 0 0" rpy="0 0 0" />
-      </xacro:cylinder_inertial>
+      <inertial>
+        <mass value="${wrist_2_mass}"/>
+        <origin rpy="${wrist_2_inertia_rotation}" xyz="${wrist_2_cog}"/>
+        <inertia
+            ixx="${wrist_2_inertia_ixx}"
+            ixy="${wrist_2_inertia_ixy}"
+            ixz="${wrist_2_inertia_ixz}"
+            iyy="${wrist_2_inertia_iyy}"
+            iyz="${wrist_2_inertia_iyz}"
+            izz="${wrist_2_inertia_izz}"
+        />
+      </inertial>
     </link>
     <link name="${tf_prefix}wrist_3_link">
@@ -251,7 +295,16 @@
         </geometry>
       </collision>
-      <xacro:cylinder_inertial radius="${wrist_3_inertia_radius}" length="${wrist_3_inertia_length}"  mass="${wrist_3_mass}">
-        <origin xyz="0.0 0.0 ${-0.5 * wrist_3_inertia_length}" rpy="0 0 0" />
-      </xacro:cylinder_inertial>
+      <inertial>
+        <mass value="${wrist_3_mass}"/>
+        <origin rpy="${wrist_3_inertia_rotation}" xyz="${wrist_3_cog}"/>
+        <inertia
+            ixx="${wrist_3_inertia_ixx}"
+            ixy="${wrist_3_inertia_ixy}"
+            ixz="${wrist_3_inertia_ixz}"
+            iyy="${wrist_3_inertia_iyy}"
+            iyz="${wrist_3_inertia_iyz}"
+            izz="${wrist_3_inertia_izz}"
+        />
+      </inertial>
     </link>
     <!-- base_joint fixes base_link to the environment -->

Commit message: Ur3 infinite wrist (#196)
Change URDF to reflect ur3(e)'s infinite wrist 3 joint

(cherry picked from commit 352a35c19d992973db85b1289ee1747d8ebde148)

File: urdf/ur_macro.xacro (robot description, xacro)
@@ -385,14 +385,22 @@
       <dynamics damping="0" friction="0"/>
     </joint>
-    <joint name="${tf_prefix}wrist_3_joint" type="revolute">
+    <joint name="${tf_prefix}wrist_3_joint" type="${wrist_3_joint_type}">
       <parent link="${tf_prefix}wrist_2_link" />
       <child link="${tf_prefix}wrist_3_link" />
       <origin xyz="${wrist_3_x} ${wrist_3_y} ${wrist_3_z}" rpy="${wrist_3_roll} ${wrist_3_pitch} ${wrist_3_yaw}" />
       <axis xyz="0 0 1" />
-      <limit lower="${wrist_3_lower_limit}" upper="${wrist_3_upper_limit}"
-             effort="${wrist_3_effort_limit}" velocity="${wrist_3_velocity_limit}"/>
-      <xacro:if value="${safety_limits}">
-         <safety_controller soft_lower_limit="${wrist_3_lower_limit + safety_pos_margin}" soft_upper_limit="${wrist_3_upper_limit - safety_pos_margin}" k_position="${safety_k_position}" k_velocity="0.0"/>
-      </xacro:if>
+      <xacro:if value="${wrist_3_joint_type != 'continuous'}">
+        <limit lower="${wrist_3_lower_limit}" upper="${wrist_3_upper_limit}"
+          effort="${wrist_3_effort_limit}" velocity="${wrist_3_velocity_limit}"/>
+        <xacro:if value="${safety_limits}">
+          <safety_controller soft_lower_limit="${wrist_3_lower_limit + safety_pos_margin}" soft_upper_limit="${wrist_3_upper_limit - safety_pos_margin}" k_position="${safety_k_position}" k_velocity="0.0"/>
+        </xacro:if>
+      </xacro:if>
+      <xacro:unless value="${wrist_3_joint_type != 'continuous'}">
+        <limit effort="${wrist_3_effort_limit}" velocity="${wrist_3_velocity_limit}"/>
+        <xacro:if value="${safety_limits}">
+          <safety_controller k_position="${safety_k_position}" k_velocity="0.0"/>
+        </xacro:if>
+      </xacro:unless>
       <dynamics damping="0" friction="0"/>
     </joint>

Commit message: Remove additional base_link_inertia link
The robot's `base` frame is rotated around the `base_link` frame by pi
rad such that `base` is the same as the robot's internal `base` frame
while `base_link` follows REP-103, such that base_link's x+ direction
points forward.

The additional `base_link_inertia` was adding another pi rad which was
compensated again. Removing the `base_link_inertia` frame makes the
kinematic chain less complicated while not changing anything
specifically.

File: urdf/ur_macro.xacro (robot description, xacro)
@@ -65,8 +65,7 @@
       force_abs_paths="${force_abs_paths}"/>
     <!-- links -  main serial chain -->
-    <link name="${tf_prefix}base_link"/>
-    <link name="${tf_prefix}base_link_inertia">
-      <visual>
-        <origin xyz="0 0 0" rpy="0 0 ${pi}"/>
+    <link name="${tf_prefix}base_link">
+      <visual>
+        <origin xyz="0 0 0" rpy="0 0 0"/>
         <geometry>
           <xacro:get_mesh name="base" type="visual"/>
@@ -74,5 +73,5 @@
       </visual>
       <collision>
-        <origin xyz="0 0 0" rpy="0 0 ${pi}"/>
+        <origin xyz="0 0 0" rpy="0 0 0"/>
         <geometry>
           <xacro:get_mesh name="base" type="collision"/>
@@ -254,18 +253,8 @@
     </joint>
     <!-- joints - main serial chain -->
-    <joint name="${tf_prefix}base_link-base_link_inertia" type="fixed">
+    <joint name="${tf_prefix}shoulder_pan_joint" type="revolute">
       <parent link="${tf_prefix}base_link" />
-      <child link="${tf_prefix}base_link_inertia" />
-      <!-- 'base_link' is REP-103 aligned (so X+ forward), while the internal
-           frames of the robot/controller have X+ pointing backwards.
-           Use the joint between 'base_link' and 'base_link_inertia' (a dummy
-           link/frame) to introduce the necessary rotation over Z (of pi rad).
-      -->
-      <origin xyz="0 0 0" rpy="0 0 ${pi}" />
-    </joint>
-    <joint name="${tf_prefix}shoulder_pan_joint" type="revolute">
-      <parent link="${tf_prefix}base_link_inertia" />
       <child link="${tf_prefix}shoulder_link" />
-      <origin xyz="${shoulder_x} ${shoulder_y} ${shoulder_z}" rpy="${shoulder_roll} ${shoulder_pitch} ${shoulder_yaw}" />
+      <origin xyz="${shoulder_x} ${shoulder_y} ${shoulder_z}" rpy="${shoulder_roll} ${shoulder_pitch} ${shoulder_yaw + pi}" />
       <axis xyz="0 0 1" />
       <limit lower="${shoulder_pan_lower_limit}" upper="${shoulder_pan_upper_limit}"
