Commit message: Remove rotation between base_link and kinematic chain
The robot's kinematic chain was rotated around the base_link, mainly
because of historic reasons. For this, an additional link called
`base_link_inertia` was introduced rotated 180 deg around base_link just
as `base`.

This commit removes this additional link which effectively rotates the
whole robot relative to base_link around 180 deg. This also makes
base_link go in line with base which should help reducing a lot of
confusion.

File: urdf/ur_macro.xacro (robot description, xacro)
@@ -65,6 +65,5 @@
       force_abs_paths="${force_abs_paths}"/>
     <!-- links -  main serial chain -->
-    <link name="${tf_prefix}base_link"/>
-    <link name="${tf_prefix}base_link_inertia">
+    <link name="${tf_prefix}base_link">
       <visual>
         <origin xyz="0 0 0" rpy="0 0 ${pi}"/>
@@ -254,16 +253,6 @@
     </joint>
     <!-- joints - main serial chain -->
-    <joint name="${tf_prefix}base_link-base_link_inertia" type="fixed">
+    <joint name="${tf_prefix}shoulder_pan_joint" type="revolute">
       <parent link="${tf_prefix}base_link" />
-      <child link="${tf_prefix}base_link_inertia" />
-      <!-- 'base_link' is REP-103 aligned (so X+ forward), while the internal
-           frames of the robot/controller have X+ pointing backwards.
-           Use the joint between 'base_link' and 'base_link_inertia' (a dummy
-           link/frame) to introduce the necessary rotation over Z (of pi rad).
-      -->
-      <origin xyz="0 0 0" rpy="0 0 ${pi}" />
-    </joint>
-    <joint name="${tf_prefix}shoulder_pan_joint" type="revolute">
-      <parent link="${tf_prefix}base_link_inertia" />
       <child link="${tf_prefix}shoulder_link" />
       <origin xyz="${shoulder_x} ${shoulder_y} ${shoulder_z}" rpy="${shoulder_roll} ${shoulder_pitch} ${shoulder_yaw}" />
@@ -358,5 +347,5 @@
            the UR controller.
       -->
-      <origin xyz="0 0 0" rpy="0 0 ${pi}"/>
+      <origin xyz="0 0 0" rpy="0 0 0"/>
       <parent link="${tf_prefix}base_link"/>
       <child link="${tf_prefix}base"/>

Commit message: エンドエフェクタ・カメラ追加

File: urdf/ur_macro.xacro (robot description, xacro)
@@ -44,4 +44,5 @@
   <xacro:include filename="$(find ur_description)/urdf/inc/ur_transmissions.xacro" />
   <xacro:include filename="$(find ur_description)/urdf/inc/ur_common.xacro" />
+  <xacro:include filename="$(find realsense2_description)/urdf/_d435.urdf.xacro" />
   <xacro:macro name="ur_robot" params="
     name
@@ -314,4 +315,70 @@
       </inertial>
     </link>
+    <link name="endeffector_type5">
+      <visual>
+        <geometry>
+          <mesh filename="package://harvesting_endeffector/type5/ee_type5.stl"/>
+        </geometry>
+      </visual>
+      <collision>
+        <geometry>
+          <mesh filename="package://harvesting_endeffector/type5/ee_type5.stl"/>
+        </geometry>
+      </collision>
+      <inertial>
+        <mass value="0.1"/>
+        <!-- tekitou na atai -->
+        <inertia ixx="0.00042" iyy="0.00042" izz="0.00042" ixy="0" ixz="0" iyz="0" />
+      </inertial>
+    </link>
+    <link name="endeffector_base">
+      <visual>
+        <geometry>
+          <mesh filename="package://harvesting_endeffector/type5/ee_base.stl"/>
+        </geometry>
+      </visual>
+      <collision>
+        <geometry>
+          <mesh filename="package://harvesting_endeffector/type5/ee_base.stl"/>
+        </geometry>
+      </collision>
+      <inertial>
+        <mass value="0.1"/>
+        <!-- tekitou na atai -->
+        <inertia ixx="0.00042" iyy="0.00042" izz="0.00042" ixy="0" ixz="0" iyz="0" />
+      </inertial>
+    </link>
+    <link name="endeffector_cutter">
+      <visual>
+        <geometry>
+          <box size="0.01 0.01 0.01"/>
+        </geometry>
+        <origin xyz="0 0 0" rpy="0 0 0"/>
+        <material name="red">
+          <color rgba="1.0 0.0 0.0 2.0"/>
+        </material>
+      </visual>
+    </link>
+    <link name="realsense_cable">
+      <visual>
+        <geometry>
+          <box size="0.03 0.04 0.02"/>
+        </geometry>
+        <origin xyz="0 0 0" rpy="0 0 0"/>
+        <material name="red">
+          <color rgba="1.0 0.0 0.0 2.0"/>
+        </material>
+      </visual>
+      <collision>
+        <geometry>
+          <box size="0.01 0.05 0.02"/>
+        </geometry>
+      </collision>
+      <inertial>
+        <mass value="0.01"/>
+        <!-- tekitou na atai -->
+        <inertia ixx="0.00042" iyy="0.00042" izz="0.00042" ixy="0" ixz="0" iyz="0" />
+      </inertial>
+    </link>
     <!-- base_joint fixes base_link to the environment -->
     <joint name="${tf_prefix}base_joint" type="fixed">
@@ -440,8 +507,35 @@
     <joint name="${tf_prefix}flange-tool0" type="fixed">
       <!-- default toolframe - X+ left, Y+ up, Z+ front -->
-      <origin xyz="0 0 0" rpy="${pi/2.0} 0 ${pi/2.0}"/>
+      <origin xyz="0 0 0" rpy="${pi/2.0} ${pi} ${pi/2.0}"/>
       <parent link="${tf_prefix}flange"/>
       <child link="${tf_prefix}tool0"/>
     </joint>
+    <joint name="tool0_to_ee_base" type="fixed">
+      <origin xyz="0 0 0.001" rpy="0.0 0.0 ${pi}"/>
+      <parent link="${tf_prefix}tool0"/>
+      <child link="endeffector_base"/>
+    </joint>
+    <xacro:sensor_d435 parent="endeffector_base" name="head_camera">
+      <origin xyz="0 0.074 0.06" rpy="-1.5708 -1.5708 0"/>
+      <xacro:arg name="use_nominal_extrinsics" default="false" />
+      <xacro:if value="$(arg use_nominal_extrinsics)">
+        <arg name="use_nominal_extrinsics" value="true" />
+      </xacro:if>
+    </xacro:sensor_d435>
+    <joint name="camera_to_camera_cable" type="fixed">
+      <origin xyz="-0.02 -0.08 0" rpy="0 0 0"/>
+      <parent link="head_camera_link"/>
+      <child link="realsense_cable"/>
+    </joint>
+    <joint name="eebase_to_ee" type="fixed">
+      <origin xyz="0 0 0.05" rpy="-${pi/2.0} -${pi/2.0} 0"/>
+      <parent link="endeffector_base"/>
+      <child link="endeffector_type5"/>
+    </joint>
+    <joint name="ee_to_cutter" type="fixed">
+      <origin xyz="0.32 -0.01 -0.028" rpy="${pi/2.0} 0 ${pi/2.0}"/>
+      <parent link="endeffector_type5"/>
+      <child link="endeffector_cutter"/>
+    </joint>
   </xacro:macro>
 </robot>

Commit message: fixed model

File: urdf/ur_macro.xacro (robot description, xacro)
@@ -517,6 +517,8 @@
     </joint>
     <xacro:sensor_d435 parent="endeffector_base" name="head_camera">
-      <origin xyz="0 0.074 0.06" rpy="-1.5708 -1.5708 0"/>
-      <xacro:arg name="use_nominal_extrinsics" default="false" />
+      <!-- <origin xyz="0 0.074 0.06" rpy="-1.5708 -1.5708 0"/> -->
+      <origin xyz="0 0.074 0.06" rpy="0.0 -1.4835298641315662 -1.5708346385162237"/>
+      <!-- <origin xyz="0 0.074 0.06" rpy="-1.570834 -1.483529 3.14155050"/> -->
+       <xacro:arg name="use_nominal_extrinsics" default="false" />
       <xacro:if value="$(arg use_nominal_extrinsics)">
         <arg name="use_nominal_extrinsics" value="true" />
@@ -534,5 +536,7 @@
     </joint>
     <joint name="ee_to_cutter" type="fixed">
-      <origin xyz="0.32 -0.01 -0.028" rpy="${pi/2.0} 0 ${pi/2.0}"/>
+      <origin xyz="0.315 -0.01 -0.024" rpy="${pi/2.0} 0 ${pi/2.0}"/>
+      <!-- -0.028 -->
+      <!-- 0.025 -->
       <parent link="endeffector_type5"/>
       <child link="endeffector_cutter"/>

Commit message: add_arm_and_cart_collider

File: urdf/ur_macro.xacro (robot description, xacro)
@@ -381,4 +381,32 @@
       </inertial>
     </link>
+    <link name="cart_collider">
+      <visual>
+        <geometry>
+          <box size="0.8 0.6 0.3"/>
+        </geometry>
+        <origin xyz="0 0 0" rpy="0 0 0"/>
+      </visual>
+      <collision>
+        <geometry>
+          <box size="0.8 0.6 0.3"/>
+        </geometry>
+        <origin xyz="0 0 0" rpy="0 0 0"/>
+      </collision>
+    </link>
+    <link name="arm_collider">
+      <visual>
+        <geometry>
+          <box size="0.3 0.5 0.5"/>
+        </geometry>
+        <origin xyz="0 0 0" rpy="0 0 0"/>
+      </visual>
+      <collision>
+        <geometry>
+          <box size="0.3 0.5 0.5"/>
+        </geometry>
+        <origin xyz="0 0 0" rpy="0 0 0"/>
+      </collision>
+    </link>
     <!-- base_joint fixes base_link to the environment -->
     <joint name="${tf_prefix}base_joint" type="fixed">
@@ -386,4 +414,14 @@
       <parent link="${parent}" />
       <child link="${tf_prefix}base_link" />
+    </joint>
+    <joint name="base_link_to_cart_collider" type="fixed">
+      <origin xyz="-0.25 0 -0.151" rpy="0 0 0"/>
+      <parent link="${tf_prefix}base_link"/>
+      <child link="cart_collider"/>
+    </joint>
+    <joint name="base_link_to_arm_collider" type="fixed">
+      <origin xyz="-0.4 0 0.251" rpy="0 0 0"/>
+      <parent link="${tf_prefix}base_link"/>
+      <child link="arm_collider"/>
     </joint>
     <!-- joints - main serial chain -->
@@ -517,7 +555,6 @@
     </joint>
     <xacro:sensor_d435 parent="endeffector_base" name="head_camera">
-      <!-- <origin xyz="0 0.074 0.06" rpy="-1.5708 -1.5708 0"/> -->
-      <origin xyz="0 0.074 0.06" rpy="0.0 -1.4835298641315662 -1.5708346385162237"/>
-      <!-- <origin xyz="0 0.074 0.06" rpy="-1.570834 -1.483529 3.14155050"/> -->
+      <origin xyz="0 0.074 0.06" rpy="-1.5708 -1.5708 0"/>
+      <!-- <origin xyz="0 0.074 0.06" rpy="0.0 -1.4835298641315662 -1.5708346385162237"/> -->
        <xacro:arg name="use_nominal_extrinsics" default="false" />
       <xacro:if value="$(arg use_nominal_extrinsics)">
@@ -536,5 +573,5 @@
     </joint>
     <joint name="ee_to_cutter" type="fixed">
-      <origin xyz="0.315 -0.01 -0.024" rpy="${pi/2.0} 0 ${pi/2.0}"/>
+      <origin xyz="0.325 -0.01 -0.024" rpy="${pi/2.0} 0 ${pi/2.0}"/>
       <!-- -0.028 -->
       <!-- 0.025 -->

Commit message: add new endeffector

File: urdf/ur_macro.xacro (robot description, xacro)
@@ -315,18 +315,20 @@
       </inertial>
     </link>
-    <link name="endeffector_type5">
-      <visual>
-        <geometry>
-          <mesh filename="package://harvesting_endeffector/type5/ee_type5.stl"/>
-        </geometry>
-      </visual>
-      <collision>
-        <geometry>
-          <mesh filename="package://harvesting_endeffector/type5/ee_type5.stl"/>
+    <!-- link name="endeffector_type5" -->
+    <link name="endeffector_type6" >
+      <visual>
+        <geometry>
+          <!-- mesh filename="package://harvesting_endeffector/type5/ee_type5.stl"/ -->
+          <mesh filename="package://harvesting_endeffector/type6/linear_cutting_endeffector-short_mirrer-main.stl" scale="0.001 0.001 0.001"/>
+        </geometry>
+      </visual>
+      <collision>
+        <geometry>
+          <!-- mesh filename="package://harvesting_endeffector/type5/ee_type5.stl"/ -->
+          <mesh filename="package://harvesting_endeffector/type6/linear_cutting_endeffector-short_mirrer-main.stl" scale="0 0 0"/>
         </geometry>
       </collision>
       <inertial>
         <mass value="0.1"/>
-        <!-- tekitou na atai -->
         <inertia ixx="0.00042" iyy="0.00042" izz="0.00042" ixy="0" ixz="0" iyz="0" />
       </inertial>
@@ -517,6 +519,6 @@
     </joint>
     <xacro:sensor_d435 parent="endeffector_base" name="head_camera">
-      <!-- <origin xyz="0 0.074 0.06" rpy="-1.5708 -1.5708 0"/> -->
-      <origin xyz="0 0.074 0.06" rpy="0.0 -1.4835298641315662 -1.5708346385162237"/>
+      <origin xyz="0 0.074 0.06" rpy="-1.5708 -1.5708 0"/>
+      <!-- <origin xyz="0 0.074 0.06" rpy="0.0 -1.4835298641315662 -1.5708346385162237"/> -->
       <!-- <origin xyz="0 0.074 0.06" rpy="-1.570834 -1.483529 3.14155050"/> -->
        <xacro:arg name="use_nominal_extrinsics" default="false" />
@@ -533,11 +535,14 @@
       <origin xyz="0 0 0.05" rpy="-${pi/2.0} -${pi/2.0} 0"/>
       <parent link="endeffector_base"/>
-      <child link="endeffector_type5"/>
+      <!-- child link="endeffector_type5"/ -->
+      <child link="endeffector_type6"/>
     </joint>
     <joint name="ee_to_cutter" type="fixed">
-      <origin xyz="0.315 -0.01 -0.024" rpy="${pi/2.0} 0 ${pi/2.0}"/>
+      <!-- origin xyz="0.315 -0.01 -0.024" rpy="${pi/2.0} 0 ${pi/2.0}"/ -->
+      <origin xyz="0.18 0.0 0.0" rpy="${pi/2.0} 0 ${pi/2.0}"/>
       <!-- -0.028 -->
       <!-- 0.025 -->
-      <parent link="endeffector_type5"/>
+      <!-- parent link="endeffector_type5"/ -->
+      <parent link="endeffector_type6"/>
       <child link="endeffector_cutter"/>
     </joint>

Commit message: add

File: urdf/ur_macro.xacro (robot description, xacro)
@@ -326,5 +326,5 @@
         <geometry>
           <!-- mesh filename="package://harvesting_endeffector/type5/ee_type5.stl"/ -->
-          <mesh filename="package://harvesting_endeffector/type6/linear_cutting_endeffector-short_mirrer-main.stl" scale="0 0 0"/>
+          <mesh filename="package://harvesting_endeffector/type6/linear_cutting_endeffector-short_mirrer-main.stl" scale="0.001 0.001 0.001"/>
         </geometry>
       </collision>
@@ -337,10 +337,12 @@
       <visual>
         <geometry>
-          <mesh filename="package://harvesting_endeffector/type5/ee_base.stl"/>
-        </geometry>
-      </visual>
-      <collision>
-        <geometry>
-          <mesh filename="package://harvesting_endeffector/type5/ee_base.stl"/>
+          <!-- mesh filename="package://harvesting_endeffector/type5/ee_base.stl"/ -->
+          <mesh filename="package://harvesting_endeffector/type6/EndEffector_Jig.stl" scale="0.001 0.001 0.001"/>
+        </geometry>
+      </visual>
+      <collision>
+        <geometry>
+          <!-- mesh filename="package://harvesting_endeffector/type5/ee_base.stl"/ -->
+          <mesh filename="package://harvesting_endeffector/type6/EndEffector_Jig.stl" scale="0.001 0.001 0.001"/>
         </geometry>
       </collision>
@@ -558,5 +560,5 @@
     <xacro:sensor_d435 parent="endeffector_base" name="head_camera">
       <origin xyz="0 0.074 0.06" rpy="-1.5708 -1.5708 0"/>
-      <!-- <origin xyz="0 0.074 0.06" rpy="0.0 -1.4835298641315662 -1.5708346385162237"/> -->
+      <!-- origin xyz="0 0.074 0.06" rpy="0.0 -1.5271630953540196 -1.570876783818119"/ -->
       <!-- <origin xyz="0 0.074 0.06" rpy="-1.570834 -1.483529 3.14155050"/> -->
        <xacro:arg name="use_nominal_extrinsics" default="false" />
@@ -571,5 +573,5 @@
     </joint>
     <joint name="eebase_to_ee" type="fixed">
-      <origin xyz="0 0 0.05" rpy="-${pi/2.0} -${pi/2.0} 0"/>
+      <origin xyz="0 0 0.105" rpy="-${pi/2.0} -${pi/2.0} 0"/>
       <parent link="endeffector_base"/>
       <!-- child link="endeffector_type5"/ -->
@@ -578,5 +580,5 @@
     <joint name="ee_to_cutter" type="fixed">
       <!-- origin xyz="0.315 -0.01 -0.024" rpy="${pi/2.0} 0 ${pi/2.0}"/ -->
-      <origin xyz="0.18 0.0 0.0" rpy="${pi/2.0} 0 ${pi/2.0}"/>
+      <origin xyz="0.18 -0.01 -0.005" rpy="${pi/2.0} 0 ${pi/2.0}"/>
       <!-- -0.028 -->
       <!-- 0.025 -->

Commit message: add data

File: urdf/ur_macro.xacro (robot description, xacro)
@@ -338,5 +338,5 @@
         <geometry>
           <!-- mesh filename="package://harvesting_endeffector/type5/ee_base.stl"/ -->
-          <mesh filename="package://harvesting_endeffector/type6/EndEffector_Jig.stl" scale="0.001 0.001 0.001"/>
+          <mesh filename="package://harvesting_endeffector/type6/Final.stl" scale="0.001 0.001 0.001"/>
         </geometry>
       </visual>
@@ -344,5 +344,5 @@
         <geometry>
           <!-- mesh filename="package://harvesting_endeffector/type5/ee_base.stl"/ -->
-          <mesh filename="package://harvesting_endeffector/type6/EndEffector_Jig.stl" scale="0.001 0.001 0.001"/>
+          <mesh filename="package://harvesting_endeffector/type6/Final.stl" scale="0.001 0.001 0.001"/>
         </geometry>
       </collision>
@@ -367,5 +367,5 @@
       <visual>
         <geometry>
-          <box size="0.03 0.04 0.02"/>
+          <box size="0 0 0"/>
         </geometry>
         <origin xyz="0 0 0" rpy="0 0 0"/>
@@ -376,5 +376,5 @@
       <collision>
         <geometry>
-          <box size="0.01 0.05 0.02"/>
+          <box size="0 0 0"/>
         </geometry>
       </collision>
@@ -559,5 +559,5 @@
     </joint>
     <xacro:sensor_d435 parent="endeffector_base" name="head_camera">
-      <origin xyz="0 0.074 0.06" rpy="-1.5708 -1.5708 0"/>
+      <origin xyz="0 0.0805 0.018" rpy="-1.5708 -1.5708 0"/>
       <!-- origin xyz="0 0.074 0.06" rpy="0.0 -1.5271630953540196 -1.570876783818119"/ -->
       <!-- <origin xyz="0 0.074 0.06" rpy="-1.570834 -1.483529 3.14155050"/> -->
@@ -573,5 +573,5 @@
     </joint>
     <joint name="eebase_to_ee" type="fixed">
-      <origin xyz="0 0 0.105" rpy="-${pi/2.0} -${pi/2.0} 0"/>
+      <origin xyz="0.01 0.0025 0.107" rpy="-${pi/2.0} -${pi/2.0} 0"/>
       <parent link="endeffector_base"/>
       <!-- child link="endeffector_type5"/ -->

Commit message: new_camera_mount

File: urdf/ur_macro.xacro (robot description, xacro)
@@ -338,5 +338,6 @@
         <geometry>
           <!-- mesh filename="package://harvesting_endeffector/type5/ee_base.stl"/ -->
-          <mesh filename="package://harvesting_endeffector/type6/Final.stl" scale="0.001 0.001 0.001"/>
+          <!--mesh filename="package://harvesting_endeffector/type6/Final.stl" scale="0.001 0.001 0.001"/ -->
+          <mesh filename="package://harvesting_endeffector/type6/EndEffector_inventor_2024smailscale.stl"/>
         </geometry>
       </visual>
@@ -344,5 +345,6 @@
         <geometry>
           <!-- mesh filename="package://harvesting_endeffector/type5/ee_base.stl"/ -->
-          <mesh filename="package://harvesting_endeffector/type6/Final.stl" scale="0.001 0.001 0.001"/>
+          <!-- mesh filename="package://harvesting_endeffector/type6/Final.stl" scale="0.001 0.001 0.001"/ -->
+          <mesh filename="package://harvesting_endeffector/type6/EndEffector_inventor_2024smailscale.stl"/>
         </geometry>
       </collision>
@@ -549,5 +551,5 @@
     <joint name="${tf_prefix}flange-tool0" type="fixed">
       <!-- default toolframe - X+ left, Y+ up, Z+ front -->
-      <origin xyz="0 0 0" rpy="${pi/2.0} ${pi} ${pi/2.0}"/>
+      <origin xyz="0.005 0 0" rpy="${pi/2.0} ${pi} ${pi/2.0}"/>
       <parent link="${tf_prefix}flange"/>
       <child link="${tf_prefix}tool0"/>
@@ -559,5 +561,5 @@
     </joint>
     <xacro:sensor_d435 parent="endeffector_base" name="head_camera">
-      <origin xyz="0 0.0805 0.018" rpy="-1.5708 -1.5708 0"/>
+      <origin xyz="0 0.080 0.014" rpy="-1.5708 -1.5708 0"/>
       <!-- origin xyz="0 0.074 0.06" rpy="0.0 -1.5271630953540196 -1.570876783818119"/ -->
       <!-- <origin xyz="0 0.074 0.06" rpy="-1.570834 -1.483529 3.14155050"/> -->
@@ -573,5 +575,5 @@
     </joint>
     <joint name="eebase_to_ee" type="fixed">
-      <origin xyz="0.01 0.0025 0.107" rpy="-${pi/2.0} -${pi/2.0} 0"/>
+      <origin xyz="0.01 0.0025 0.101" rpy="-${pi/2.0} -${pi/2.0} 0"/>
       <parent link="endeffector_base"/>
       <!-- child link="endeffector_type5"/ -->
