Commit message: Preliminary support for g-series robots
The new mesh files aren't committed, yet.

File: urdf/ur_macro.xacro (robot description, xacro)
@@ -56,4 +56,5 @@
     safety_k_position:=20
     force_abs_paths:=false
+    smart_panel:=''
     ">
     <!-- Load configuration data from the provided .yaml files -->
@@ -64,4 +65,6 @@
       visual_parameters_file="${visual_parameters_file}"
       force_abs_paths="${force_abs_paths}"/>
+    <!-- Empty smart_panel argument means "use visual_parameters.yaml". -->
+    <xacro:property name="smart_panel_enabled" value="${smart_panel if smart_panel != '' else smart_panel_from_visual}"/>
     <!-- links -  main serial chain -->
     <!-- base_link serves as the root of the robot's kinematic tree. It follows REP-103
@@ -401,4 +404,43 @@
       <origin xyz="0 0 0" rpy="0 ${-pi/2.0} ${-pi/2.0}" />
     </joint>
+    <!-- Optional Smart Panel accessory attached to wrist_3_link.
+         Geometry lives in meshes/common/smart_panel so it can be reused
+         across robot models. Joint origin is a placeholder until the
+         real attachment pose is finalized. -->
+    <xacro:if value="${smart_panel_enabled}">
+      <xacro:if value="${force_abs_paths}">
+        <xacro:property name="smart_panel_visual_mesh" value="file://$(find ur_description)/meshes/common/smart_panel/visual/smart_panel.glb"/>
+        <xacro:property name="smart_panel_collision_mesh" value="file://$(find ur_description)/meshes/common/smart_panel/collision/smart_panel.stl"/>
+      </xacro:if>
+      <xacro:unless value="${force_abs_paths}">
+        <xacro:property name="smart_panel_visual_mesh" value="package://ur_description/meshes/common/smart_panel/visual/smart_panel.glb"/>
+        <xacro:property name="smart_panel_collision_mesh" value="package://ur_description/meshes/common/smart_panel/collision/smart_panel.stl"/>
+      </xacro:unless>
+      <link name="${tf_prefix}smart_panel">
+        <visual>
+          <origin xyz="0 0 0" rpy="0 0 0"/>
+          <geometry>
+            <mesh filename="${smart_panel_visual_mesh}"/>
+          </geometry>
+        </visual>
+        <collision>
+          <origin xyz="0 0 0" rpy="0 0 0"/>
+          <geometry>
+            <mesh filename="${smart_panel_collision_mesh}"/>
+          </geometry>
+        </collision>
+        <inertial>
+          <!-- Placeholder inertia until measured Smart Panel properties are available. -->
+          <mass value="0.1"/>
+          <origin xyz="0 0 0" rpy="0 0 0"/>
+          <inertia ixx="0.0001" ixy="0.0" ixz="0.0" iyy="0.0001" iyz="0.0" izz="0.0001"/>
+        </inertial>
+      </link>
+      <joint name="${tf_prefix}wrist_3_link-smart_panel" type="fixed">
+        <parent link="${tf_prefix}wrist_3_link"/>
+        <child link="${tf_prefix}smart_panel"/>
+        <origin xyz="0 0 0" rpy="0 0 0"/>
+      </joint>
+    </xacro:if>
     <!-- ROS-Industrial 'tool0' frame - all-zeros tool frame -->
     <link name="${tf_prefix}tool0"/>

Commit message: Update ur17g-1300 meshes

File: urdf/ur_macro.xacro (robot description, xacro)
@@ -410,9 +410,9 @@
     <xacro:if value="${smart_panel_enabled}">
       <xacro:if value="${force_abs_paths}">
-        <xacro:property name="smart_panel_visual_mesh" value="file://$(find ur_description)/meshes/common/smart_panel/visual/smart_panel.glb"/>
+        <xacro:property name="smart_panel_visual_mesh" value="file://$(find ur_description)/meshes/common/smart_panel/visual/smart_panel.dae"/>
         <xacro:property name="smart_panel_collision_mesh" value="file://$(find ur_description)/meshes/common/smart_panel/collision/smart_panel.stl"/>
       </xacro:if>
       <xacro:unless value="${force_abs_paths}">
-        <xacro:property name="smart_panel_visual_mesh" value="package://ur_description/meshes/common/smart_panel/visual/smart_panel.glb"/>
+        <xacro:property name="smart_panel_visual_mesh" value="package://ur_description/meshes/common/smart_panel/visual/smart_panel.dae"/>
         <xacro:property name="smart_panel_collision_mesh" value="package://ur_description/meshes/common/smart_panel/collision/smart_panel.stl"/>
       </xacro:unless>

Commit message: Add mass and inertia of smart panel (estimated)
The smart panel inertia is estimated based on its shape and mass
assuming homogenious mass distribution inside. The CoG therefore matches
the geometric center.

File: urdf/ur_macro.xacro (robot description, xacro)
@@ -406,6 +406,5 @@
     <!-- Optional Smart Panel accessory attached to wrist_3_link.
          Geometry lives in meshes/common/smart_panel so it can be reused
-         across robot models. Joint origin is a placeholder until the
-         real attachment pose is finalized. -->
+         across robot models. -->
     <xacro:if value="${smart_panel_enabled}">
       <xacro:if value="${force_abs_paths}">
@@ -431,8 +430,10 @@
         </collision>
         <inertial>
-          <!-- Placeholder inertia until measured Smart Panel properties are available. -->
-          <mass value="0.1"/>
-          <origin xyz="0 0 0" rpy="0 0 0"/>
-          <inertia ixx="0.0001" ixy="0.0" ixz="0.0" iyy="0.0001" iyz="0.0" izz="0.0001"/>
+          <!-- Inertia estimated for homogeneous weight distribution and the measured mass of the smart panel. -->
+          <mass value="0.0167"/>
+          <origin xyz="0.045 0 -0.030" rpy="0 0 0"/>
+          <inertia ixx="4.866178e-06" ixy="3.996e-10" ixz="1.595575e-07"
+                   iyy="2.852570e-06" iyz="-1.854789e-09"
+                   izz="2.789305e-06"/>
         </inertial>
       </link>
@@ -440,4 +441,5 @@
         <parent link="${tf_prefix}wrist_3_link"/>
         <child link="${tf_prefix}smart_panel"/>
+        <!-- the mesh is in the correct position relative to wrist_3_link -->
         <origin xyz="0 0 0" rpy="0 0 0"/>
       </joint>

Commit message: Update smart panel's mass as measured

File: urdf/ur_macro.xacro (robot description, xacro)
@@ -431,9 +431,9 @@
         <inertial>
           <!-- Inertia estimated for homogeneous weight distribution and the measured mass of the smart panel. -->
-          <mass value="0.0167"/>
           <origin xyz="0.045 0 -0.030" rpy="0 0 0"/>
-          <inertia ixx="4.866178e-06" ixy="3.996e-10" ixz="1.595575e-07"
-                   iyy="2.852570e-06" iyz="-1.854789e-09"
-                   izz="2.789305e-06"/>
+          <mass value="0.0195"/>
+          <inertia ixx="5.682064e-06" ixy="4.66603e-10" ixz="1.863097e-07"
+                   iyy="3.330845e-06" iyz="-2.165772e-09"
+                   izz="3.256972e-06"/>
         </inertial>
       </link>

Commit message: Add support for g-series robots (#426)
Adds descriptions and meshes for the new g-series robots. We've added new mesh files compared to the UR series that don't use jpeg textures anymore.

As a new argument, the smart-panel can be switched off and on depending on the actual setup.

The smart panel inertia is estimated based on its shape and mass
assuming homogeneous mass distribution inside. The CoG therefore matches
the geometric center.

(cherry picked from commit 970bf8aaed1ffa160ca86ab4bb6c04181f7b592d)

File: urdf/ur_macro.xacro (robot description, xacro)
@@ -56,4 +56,5 @@
     safety_k_position:=20
     force_abs_paths:=false
+    smart_panel:=''
     ">
     <!-- Load configuration data from the provided .yaml files -->
@@ -64,4 +65,6 @@
       visual_parameters_file="${visual_parameters_file}"
       force_abs_paths="${force_abs_paths}"/>
+    <!-- Empty smart_panel argument means "use visual_parameters.yaml". -->
+    <xacro:property name="smart_panel_enabled" value="${smart_panel if smart_panel != '' else smart_panel_from_visual}"/>
     <!-- links -  main serial chain -->
     <!-- base_link serves as the root of the robot's kinematic tree. It follows REP-103
@@ -375,4 +378,45 @@
       <origin xyz="0 0 0" rpy="0 ${-pi/2.0} ${-pi/2.0}" />
     </joint>
+    <!-- Optional Smart Panel accessory attached to wrist_3_link.
+         Geometry lives in meshes/common/smart_panel so it can be reused
+         across robot models. -->
+    <xacro:if value="${smart_panel_enabled}">
+      <xacro:if value="${force_abs_paths}">
+        <xacro:property name="smart_panel_visual_mesh" value="file://$(find ur_description)/meshes/common/smart_panel/visual/smart_panel.dae"/>
+        <xacro:property name="smart_panel_collision_mesh" value="file://$(find ur_description)/meshes/common/smart_panel/collision/smart_panel.stl"/>
+      </xacro:if>
+      <xacro:unless value="${force_abs_paths}">
+        <xacro:property name="smart_panel_visual_mesh" value="package://ur_description/meshes/common/smart_panel/visual/smart_panel.dae"/>
+        <xacro:property name="smart_panel_collision_mesh" value="package://ur_description/meshes/common/smart_panel/collision/smart_panel.stl"/>
+      </xacro:unless>
+      <link name="${tf_prefix}smart_panel">
+        <visual>
+          <origin xyz="0 0 0" rpy="0 0 0"/>
+          <geometry>
+            <mesh filename="${smart_panel_visual_mesh}"/>
+          </geometry>
+        </visual>
+        <collision>
+          <origin xyz="0 0 0" rpy="0 0 0"/>
+          <geometry>
+            <mesh filename="${smart_panel_collision_mesh}"/>
+          </geometry>
+        </collision>
+        <inertial>
+          <!-- Inertia estimated for homogeneous weight distribution and the measured mass of the smart panel. -->
+          <origin xyz="0.045 0 -0.030" rpy="0 0 0"/>
+          <mass value="0.0195"/>
+          <inertia ixx="5.682064e-06" ixy="4.66603e-10" ixz="1.863097e-07"
+                   iyy="3.330845e-06" iyz="-2.165772e-09"
+                   izz="3.256972e-06"/>
+        </inertial>
+      </link>
+      <joint name="${tf_prefix}wrist_3_link-smart_panel" type="fixed">
+        <parent link="${tf_prefix}wrist_3_link"/>
+        <child link="${tf_prefix}smart_panel"/>
+        <!-- the mesh is in the correct position relative to wrist_3_link -->
+        <origin xyz="0 0 0" rpy="0 0 0"/>
+      </joint>
+    </xacro:if>
     <!-- ROS-Industrial 'tool0' frame - all-zeros tool frame -->
     <link name="${tf_prefix}tool0"/>

Commit message: Allow parsing new kilted config format (#432)
This commit allows parsing the new config format used from kilted on.
This allows a more direct backport of new robot models from the default
branch to jazzy. It is fully backwards compatible and can still parse the
"old" format.

(cherry picked from commit 2ca3999ea3f5fbf6e105363d71bdcd84a03d91e9)

# Conflicts:
#	test/test_ur_urdf_xacro.py

File: urdf/ur_macro.xacro (robot description, xacro)
@@ -141,5 +141,5 @@
     <link name="${tf_prefix}base_link_inertia">
       <visual>
-        <origin xyz="0 0 0" rpy="0 0 ${pi}"/>
+        <xacro:mesh_origin name="base" legacy_xyz="0 0 0" legacy_rpy="0 0 ${pi}"/>
         <geometry>
           <xacro:get_mesh name="base" type="visual"/>
@@ -147,5 +147,5 @@
       </visual>
       <collision>
-        <origin xyz="0 0 0" rpy="0 0 ${pi}"/>
+        <xacro:mesh_origin name="base" legacy_xyz="0 0 0" legacy_rpy="0 0 ${pi}"/>
         <geometry>
           <xacro:get_mesh name="base" type="collision"/>
@@ -158,5 +158,5 @@
     <link name="${tf_prefix}shoulder_link">
       <visual>
-        <origin xyz="0 0 0" rpy="0 0 ${pi}"/>
+        <xacro:mesh_origin name="shoulder" legacy_xyz="0 0 0" legacy_rpy="0 0 ${pi}"/>
         <geometry>
           <xacro:get_mesh name="shoulder" type="visual"/>
@@ -164,5 +164,5 @@
       </visual>
       <collision>
-        <origin xyz="0 0 0" rpy="0 0 ${pi}"/>
+        <xacro:mesh_origin name="shoulder" legacy_xyz="0 0 0" legacy_rpy="0 0 ${pi}"/>
         <geometry>
           <xacro:get_mesh name="shoulder" type="collision"/>
@@ -183,5 +183,5 @@
     <link name="${tf_prefix}upper_arm_link">
       <visual>
-        <origin xyz="0 0 ${shoulder_offset}" rpy="${pi/2} 0 ${-pi/2}"/>
+        <xacro:mesh_origin name="upper_arm" legacy_xyz="0 0 ${shoulder_offset}" legacy_rpy="${pi/2} 0 ${-pi/2}"/>
         <geometry>
           <xacro:get_mesh name="upper_arm" type="visual"/>
@@ -189,5 +189,5 @@
       </visual>
       <collision>
-        <origin xyz="0 0 ${shoulder_offset}" rpy="${pi/2} 0 ${-pi/2}"/>
+        <xacro:mesh_origin name="upper_arm" legacy_xyz="0 0 ${shoulder_offset}" legacy_rpy="${pi/2} 0 ${-pi/2}"/>
         <geometry>
           <xacro:get_mesh name="upper_arm" type="collision"/>
@@ -209,5 +209,5 @@
     <link name="${tf_prefix}forearm_link">
       <visual>
-        <origin xyz="0 0 ${elbow_offset}" rpy="${pi/2} 0 ${-pi/2}"/>
+        <xacro:mesh_origin name="forearm" legacy_xyz="0 0 ${elbow_offset}" legacy_rpy="${pi/2} 0 ${-pi/2}"/>
         <geometry>
           <xacro:get_mesh name="forearm" type="visual"/>
@@ -215,5 +215,5 @@
       </visual>
       <collision>
-        <origin xyz="0 0 ${elbow_offset}" rpy="${pi/2} 0 ${-pi/2}"/>
+        <xacro:mesh_origin name="forearm" legacy_xyz="0 0 ${elbow_offset}" legacy_rpy="${pi/2} 0 ${-pi/2}"/>
         <geometry>
           <xacro:get_mesh name="forearm" type="collision"/>
@@ -234,7 +234,8 @@
     </link>
     <link name="${tf_prefix}wrist_1_link">
-	  <xacro:get_visual_params name="wrist_1" type="visual_offset"/>
-      <visual>
-      	<origin xyz="0 0 ${visual_params}" rpy="${pi/2} 0 0"/>
+      <xacro:get_visual_params name="wrist_1" type="visual_offset"/>
+      <xacro:property name="wrist_1_legacy_offset" value="${visual_params}"/>
+      <visual>
+        <xacro:mesh_origin name="wrist_1" legacy_xyz="0 0 ${wrist_1_legacy_offset}" legacy_rpy="${pi/2} 0 0"/>
         <geometry>
           <xacro:get_mesh name="wrist_1" type="visual"/>
@@ -242,5 +243,5 @@
       </visual>
       <collision>
-        <origin xyz="0 0 ${visual_params}" rpy="${pi/2} 0 0"/>
+        <xacro:mesh_origin name="wrist_1" legacy_xyz="0 0 ${wrist_1_legacy_offset}" legacy_rpy="${pi/2} 0 0"/>
         <geometry>
           <xacro:get_mesh name="wrist_1" type="collision"/>
@@ -261,7 +262,8 @@
     </link>
     <link name="${tf_prefix}wrist_2_link">
-          <xacro:get_visual_params name="wrist_2" type="visual_offset"/>
-      <visual>
-        <origin xyz="0 0 ${visual_params}" rpy="0 0 0"/>
+      <xacro:get_visual_params name="wrist_2" type="visual_offset"/>
+      <xacro:property name="wrist_2_legacy_offset" value="${visual_params}"/>
+      <visual>
+        <xacro:mesh_origin name="wrist_2" legacy_xyz="0 0 ${wrist_2_legacy_offset}" legacy_rpy="0 0 0"/>
         <geometry>
           <xacro:get_mesh name="wrist_2" type="visual"/>
@@ -269,5 +271,5 @@
       </visual>
       <collision>
-        <origin xyz="0 0 ${visual_params}" rpy="0 0 0"/>
+        <xacro:mesh_origin name="wrist_2" legacy_xyz="0 0 ${wrist_2_legacy_offset}" legacy_rpy="0 0 0"/>
         <geometry>
           <xacro:get_mesh name="wrist_2" type="collision"/>
@@ -296,5 +298,5 @@
       </xacro:if>
       <visual>
-        <origin xyz="${mesh_offset}" rpy="${pi/2} 0 0"/>
+        <xacro:mesh_origin name="wrist_3" legacy_xyz="${mesh_offset}" legacy_rpy="${pi/2} 0 0"/>
         <geometry>
           <xacro:get_mesh name="wrist_3" type="visual"/>
@@ -302,5 +304,5 @@
       </visual>
       <collision>
-        <origin xyz="${mesh_offset}" rpy="${pi/2} 0 0"/>
+        <xacro:mesh_origin name="wrist_3" legacy_xyz="${mesh_offset}" legacy_rpy="${pi/2} 0 0"/>
         <geometry>
           <xacro:get_mesh name="wrist_3" type="collision"/>
