Commit message: WIP: Split ros2_control and kinematics description
This commit separates the description into a pure description of the robot's
visuals, kinematics and the control structure.

This is by far not at a finished state.

File: ur_description/urdf/inc/ur_common.xacro (robot description, xacro)
@@ -36,4 +36,9 @@
     <xacro:get_mesh_path/>
     <mesh filename="${mesh}"/>
+  </xacro:macro>
+  <xacro:macro name="get_kinematics_hash" params="kinematics_parameters_file">
+    <xacro:property name="config_kinematics_parameters" value="${xacro.load_yaml(kinematics_parameters_file)}"/>
+    <xacro:property name="sec_kinematics" value="${config_kinematics_parameters['kinematics']}" />
+    <xacro:property name="kinematics_hash" value="${sec_kinematics['hash']}" scope="parent"/>
   </xacro:macro>
   <xacro:macro name="read_model_data" params="joint_limits_parameters_file kinematics_parameters_file physical_parameters_file visual_parameters_file force_abs_paths">
@@ -168,6 +173,4 @@
     <xacro:property name="forearm_radius" value="${sec_inertia_parameters['forearm_radius']}" scope="parent"/>
     <xacro:property name="wrist_radius" value="${sec_inertia_parameters['wrist_radius']}" scope="parent"/>
-    <!--KINEMATICS HASH-->
-    <xacro:property name="kinematics_hash" value="${sec_kinematics['hash']}" scope="parent"/>
   </xacro:macro>
 </robot>

File: ur_description/urdf/ur_macro.xacro (robot description, xacro)
@@ -42,5 +42,4 @@
      - Muhammad Asif Rana
   -->
-  <xacro:include filename="$(find ur_description)/urdf/inc/ur_transmissions.xacro" />
   <xacro:include filename="$(find ur_description)/urdf/inc/ur_common.xacro" />
   <xacro:macro name="ur_robot" params="
@@ -53,35 +52,9 @@
     physical_parameters_file
     visual_parameters_file
-    transmission_hw_interface:=hardware_interface/PositionJointInterface
     safety_limits:=false
     safety_pos_margin:=0.15
     safety_k_position:=20
-    use_fake_hardware:=false
-    fake_sensor_commands:=false
-    sim_gazebo:=false
-    sim_ignition:=false
-    headless_mode:=false
-    initial_positions:=${dict(shoulder_pan_joint=0.0,shoulder_lift_joint=-1.57,elbow_joint=0.0,wrist_1_joint=-1.57,wrist_2_joint=0.0,wrist_3_joint=0.0)}
-    use_tool_communication:=false
-    tool_voltage:=0
-    tool_parity:=0
-    tool_baud_rate:=115200
-    tool_stop_bits:=1
-    tool_rx_idle_chars:=1.5
-    tool_tx_idle_chars:=3.5
-    tool_device_name:=/tmp/ttyUR
-    tool_tcp_port:=54321
-    robot_ip:=0.0.0.0
-    script_filename:=to_be_filled_by_ur_robot_driver
-    output_recipe_filename:=to_be_filled_by_ur_robot_driver
-    input_recipe_filename:=to_be_filled_by_ur_robot_driver
-    reverse_port:=50001
-    script_sender_port:=50002
-    reverse_ip:=0.0.0.0
-    script_command_port:=50004
-    trajectory_port:=50003
-    non_blocking_read:=false
-    keep_alive_count:=2"
-    >
+    force_abs_paths:=false
+    ">
     <!-- Load configuration data from the provided .yaml files -->
     <xacro:read_model_data
@@ -90,42 +63,5 @@
       physical_parameters_file="${physical_parameters_file}"
       visual_parameters_file="${visual_parameters_file}"
-      force_abs_paths="${sim_gazebo or sim_ignition}"/>
-    <!-- ros2 control include -->
-    <xacro:include filename="$(find ur_description)/urdf/ur.ros2_control.xacro" />
-    <!-- ros2 control instance -->
-    <xacro:ur_ros2_control
-      name="${name}"
-      use_fake_hardware="${use_fake_hardware}"
-      initial_positions="${initial_positions}"
-      fake_sensor_commands="${fake_sensor_commands}"
-      headless_mode="${headless_mode}"
-      sim_gazebo="${sim_gazebo}"
-      sim_ignition="${sim_ignition}"
-      script_filename="${script_filename}"
-      output_recipe_filename="${output_recipe_filename}"
-      input_recipe_filename="${input_recipe_filename}"
-      tf_prefix="${tf_prefix}"
-      hash_kinematics="${kinematics_hash}"
-      robot_ip="${robot_ip}"
-      use_tool_communication="${use_tool_communication}"
-      tool_voltage="${tool_voltage}"
-      tool_parity="${tool_parity}"
-      tool_baud_rate="${tool_baud_rate}"
-      tool_stop_bits="${tool_stop_bits}"
-      tool_rx_idle_chars="${tool_rx_idle_chars}"
-      tool_tx_idle_chars="${tool_tx_idle_chars}"
-      tool_device_name="${tool_device_name}"
-      tool_tcp_port="${tool_tcp_port}"
-      reverse_port="${reverse_port}"
-      script_sender_port="${script_sender_port}"
-      reverse_ip="${reverse_ip}"
-      script_command_port="${script_command_port}"
-      trajectory_port="${trajectory_port}"
-      non_blocking_read="${non_blocking_read}"
-      keep_alive_count="${keep_alive_count}"
-      />
-    <!-- Add URDF transmission elements (for ros_control) -->
-    <!--<xacro:ur_arm_transmission prefix="${prefix}" hw_interface="${transmission_hw_interface}" />-->
-    <!-- Placeholder for ros2_control transmission which don't yet exist -->
+      force_abs_paths="${force_abs_paths}"/>
     <!-- links -  main serial chain -->
     <link name="${tf_prefix}base_link"/>

File: ur_ros2_control_support/urdf/ur.urdf.xacro (robot description, xacro)
@@ -4,5 +4,5 @@
    <xacro:arg name="name" default="ur"/>
    <!-- import main macro -->
-   <xacro:include filename="$(find ur_description)/urdf/ur_macro.xacro"/>
+   <xacro:include filename="$(find ur_ros2_control_support)/urdf/ur_macro.xacro"/>
    <!-- possible 'ur_type' values: ur3, ur3e, ur5, ur5e, ur10, ur10e, ur16e -->
    <!-- the default value should raise an error in case this was called without defining the type -->
@@ -49,5 +49,5 @@
    <link name="world" />
    <!-- arm -->
-   <xacro:ur_robot
+   <xacro:ur_robot_ros2_controlled
      name="$(arg name)"
      tf_prefix="$(arg tf_prefix)"
@@ -84,5 +84,5 @@
      >
      <origin xyz="0 0 0" rpy="0 0 0" />          <!-- position robot in the world -->
-   </xacro:ur_robot>
+   </xacro:ur_robot_ros2_controlled>
    <xacro:if value="$(arg sim_gazebo)">
     <!-- Gazebo plugins -->
