Commit message: Joint limits parameters for Moveit planning (#187)
* Change names of joints in the limits yaml.

* Change accordingly field names in the xacro.

* Adapt moveit-based launch files to use LaunchContext.

* Add auxiliary python module for launch files simplification. Add support for degrees and radians constructors in yaml.

* Fix pre-commit.

* Add auxiliary module to servo test.

* Remove unneccessary imports.

File: urdf/inc/ur_common.xacro (robot description, xacro)
@@ -34,28 +34,28 @@
     <xacro:property name="sec_kinematics" value="${config_kinematics_parameters['kinematics']}" />
     <!-- JOINTS LIMIT PARAMETERS -->
-    <xacro:property name="shoulder_pan_lower_limit" value="${sec_limits['shoulder_pan']['min_position']}" scope="parent"/>
-    <xacro:property name="shoulder_pan_upper_limit" value="${sec_limits['shoulder_pan']['max_position']}" scope="parent"/>
-    <xacro:property name="shoulder_pan_velocity_limit" value="${sec_limits['shoulder_pan']['max_velocity']}" scope="parent"/>
-    <xacro:property name="shoulder_pan_effort_limit" value="${sec_limits['shoulder_pan']['max_effort']}" scope="parent"/>
-    <xacro:property name="shoulder_lift_lower_limit" value="${sec_limits['shoulder_lift']['min_position']}" scope="parent"/>
-    <xacro:property name="shoulder_lift_upper_limit" value="${sec_limits['shoulder_lift']['max_position']}" scope="parent"/>
-    <xacro:property name="shoulder_lift_velocity_limit" value="${sec_limits['shoulder_lift']['max_velocity']}" scope="parent"/>
-    <xacro:property name="shoulder_lift_effort_limit" value="${sec_limits['shoulder_lift']['max_effort']}" scope="parent"/>
+    <xacro:property name="shoulder_pan_lower_limit" value="${sec_limits['shoulder_pan_joint']['min_position']}" scope="parent"/>
+    <xacro:property name="shoulder_pan_upper_limit" value="${sec_limits['shoulder_pan_joint']['max_position']}" scope="parent"/>
+    <xacro:property name="shoulder_pan_velocity_limit" value="${sec_limits['shoulder_pan_joint']['max_velocity']}" scope="parent"/>
+    <xacro:property name="shoulder_pan_effort_limit" value="${sec_limits['shoulder_pan_joint']['max_effort']}" scope="parent"/>
+    <xacro:property name="shoulder_lift_lower_limit" value="${sec_limits['shoulder_lift_joint']['min_position']}" scope="parent"/>
+    <xacro:property name="shoulder_lift_upper_limit" value="${sec_limits['shoulder_lift_joint']['max_position']}" scope="parent"/>
+    <xacro:property name="shoulder_lift_velocity_limit" value="${sec_limits['shoulder_lift_joint']['max_velocity']}" scope="parent"/>
+    <xacro:property name="shoulder_lift_effort_limit" value="${sec_limits['shoulder_lift_joint']['max_effort']}" scope="parent"/>
     <xacro:property name="elbow_joint_lower_limit" value="${sec_limits['elbow_joint']['min_position']}" scope="parent"/>
     <xacro:property name="elbow_joint_upper_limit" value="${sec_limits['elbow_joint']['max_position']}" scope="parent"/>
     <xacro:property name="elbow_joint_velocity_limit" value="${sec_limits['elbow_joint']['max_velocity']}" scope="parent"/>
     <xacro:property name="elbow_joint_effort_limit" value="${sec_limits['elbow_joint']['max_effort']}" scope="parent"/>
-    <xacro:property name="wrist_1_lower_limit" value="${sec_limits['wrist_1']['min_position']}" scope="parent"/>
-    <xacro:property name="wrist_1_upper_limit" value="${sec_limits['wrist_1']['max_position']}" scope="parent"/>
-    <xacro:property name="wrist_1_velocity_limit" value="${sec_limits['wrist_1']['max_velocity']}" scope="parent"/>
-    <xacro:property name="wrist_1_effort_limit" value="${sec_limits['wrist_1']['max_effort']}" scope="parent"/>
-    <xacro:property name="wrist_2_lower_limit" value="${sec_limits['wrist_2']['min_position']}" scope="parent"/>
-    <xacro:property name="wrist_2_upper_limit" value="${sec_limits['wrist_2']['max_position']}" scope="parent"/>
-    <xacro:property name="wrist_2_velocity_limit" value="${sec_limits['wrist_2']['max_velocity']}" scope="parent"/>
-    <xacro:property name="wrist_2_effort_limit" value="${sec_limits['wrist_2']['max_effort']}" scope="parent"/>
-    <xacro:property name="wrist_3_lower_limit" value="${sec_limits['wrist_3']['min_position']}" scope="parent"/>
-    <xacro:property name="wrist_3_upper_limit" value="${sec_limits['wrist_3']['max_position']}" scope="parent"/>
-    <xacro:property name="wrist_3_velocity_limit" value="${sec_limits['wrist_3']['max_velocity']}" scope="parent"/>
-    <xacro:property name="wrist_3_effort_limit" value="${sec_limits['wrist_3']['max_effort']}" scope="parent"/>
+    <xacro:property name="wrist_1_lower_limit" value="${sec_limits['wrist_1_joint']['min_position']}" scope="parent"/>
+    <xacro:property name="wrist_1_upper_limit" value="${sec_limits['wrist_1_joint']['max_position']}" scope="parent"/>
+    <xacro:property name="wrist_1_velocity_limit" value="${sec_limits['wrist_1_joint']['max_velocity']}" scope="parent"/>
+    <xacro:property name="wrist_1_effort_limit" value="${sec_limits['wrist_1_joint']['max_effort']}" scope="parent"/>
+    <xacro:property name="wrist_2_lower_limit" value="${sec_limits['wrist_2_joint']['min_position']}" scope="parent"/>
+    <xacro:property name="wrist_2_upper_limit" value="${sec_limits['wrist_2_joint']['max_position']}" scope="parent"/>
+    <xacro:property name="wrist_2_velocity_limit" value="${sec_limits['wrist_2_joint']['max_velocity']}" scope="parent"/>
+    <xacro:property name="wrist_2_effort_limit" value="${sec_limits['wrist_2_joint']['max_effort']}" scope="parent"/>
+    <xacro:property name="wrist_3_lower_limit" value="${sec_limits['wrist_3_joint']['min_position']}" scope="parent"/>
+    <xacro:property name="wrist_3_upper_limit" value="${sec_limits['wrist_3_joint']['max_position']}" scope="parent"/>
+    <xacro:property name="wrist_3_velocity_limit" value="${sec_limits['wrist_3_joint']['max_velocity']}" scope="parent"/>
+    <xacro:property name="wrist_3_effort_limit" value="${sec_limits['wrist_3_joint']['max_effort']}" scope="parent"/>
     <!-- DH PARAMETERS -->
     <xacro:property name="d1" value="${sec_dh_parameters['d1']}" scope="parent"/>

Commit message: Use xacro-resolved mesh filenames
using the package://-notation is not correctly interpreted by all clients (e.g. gazebo)
Using $(find pkgname)/x/y/z.stl gets not translated properly during xacro processing.

As implemented in this commit, the mesh paths get translated to absolute paths
during xacro processing and therefore the result is usable by many clients
(such as RViz, Gazebo)

File: urdf/inc/ur_common.xacro (robot description, xacro)
@@ -152,40 +152,41 @@
     <!-- Mesh files -->
     <xacro:property name="base_mesh" value="${sec_mesh_files['base']}"/>
-    <xacro:property name="base_visual_mesh" value="${base_mesh['visual']['mesh']}" scope="parent"/>
+    <xacro:property name="base_visual_mesh" value="file://$(find ${base_mesh['visual']['mesh']['package']})/${base_mesh['visual']['mesh']['path']}" scope="parent"/>
     <xacro:property name="base_visual_material_name" value="${base_mesh['visual']['material']['name']}" scope="parent"/>
     <xacro:property name="base_visual_material_color" value="${base_mesh['visual']['material']['color']}" scope="parent"/>
-    <xacro:property name="base_collision_mesh" value="${base_mesh['collision']['mesh']}" scope="parent"/>
+    <xacro:property name="base_collision_mesh" value="file://$(find ${base_mesh['collision']['mesh']['package']})/${base_mesh['collision']['mesh']['path']}" scope="parent"/>
     <xacro:property name="shoulder_mesh" value="${sec_mesh_files['shoulder']}"/>
-    <xacro:property name="shoulder_visual_mesh" value="${shoulder_mesh['visual']['mesh']}" scope="parent"/>
+    <xacro:property name="shoulder_visual_mesh" value="file://$(find ${shoulder_mesh['visual']['mesh']['package']})/${shoulder_mesh['visual']['mesh']['path']}" scope="parent"/>
     <xacro:property name="shoulder_visual_material_name" value="${shoulder_mesh['visual']['material']['name']}" scope="parent"/>
     <xacro:property name="shoulder_visual_material_color" value="${shoulder_mesh['visual']['material']['color']}" scope="parent"/>
-    <xacro:property name="shoulder_collision_mesh" value="${shoulder_mesh['collision']['mesh']}" scope="parent"/>
+    <xacro:property name="shoulder_collision_mesh" value="file://$(find ${shoulder_mesh['collision']['mesh']['package']})/${shoulder_mesh['collision']['mesh']['path']}" scope="parent"/>
     <xacro:property name="upper_arm_mesh" value="${sec_mesh_files['upper_arm']}"/>
-    <xacro:property name="upper_arm_visual_mesh" value="${upper_arm_mesh['visual']['mesh']}" scope="parent"/>
+    <xacro:property name="upper_arm_visual_mesh" value="file://$(find ${upper_arm_mesh['visual']['mesh']['package']})/${upper_arm_mesh['visual']['mesh']['path']}" scope="parent"/>
     <xacro:property name="upper_arm_visual_material_name" value="${upper_arm_mesh['visual']['material']['name']}" scope="parent"/>
     <xacro:property name="upper_arm_visual_material_color" value="${upper_arm_mesh['visual']['material']['color']}" scope="parent"/>
     <xacro:property name="upper_arm_collision_mesh" value="${upper_arm_mesh['collision']['mesh']}" scope="parent"/>
+    <xacro:property name="upper_arm_collision_mesh" value="file://$(find ${upper_arm_mesh['collision']['mesh']['package']})/${upper_arm_mesh['collision']['mesh']['path']}" scope="parent"/>
     <xacro:property name="forearm_mesh" value="${sec_mesh_files['forearm']}"/>
-    <xacro:property name="forearm_visual_mesh" value="${forearm_mesh['visual']['mesh']}" scope="parent"/>
+    <xacro:property name="forearm_visual_mesh" value="file://$(find ${forearm_mesh['visual']['mesh']['package']})/${forearm_mesh['visual']['mesh']['path']}" scope="parent"/>
     <xacro:property name="forearm_visual_material_name" value="${forearm_mesh['visual']['material']['name']}" scope="parent"/>
     <xacro:property name="forearm_visual_material_color" value="${forearm_mesh['visual']['material']['color']}" scope="parent"/>
-    <xacro:property name="forearm_collision_mesh" value="${forearm_mesh['collision']['mesh']}" scope="parent"/>
+    <xacro:property name="forearm_collision_mesh" value="file://$(find ${forearm_mesh['collision']['mesh']['package']})/${forearm_mesh['collision']['mesh']['path']}" scope="parent"/>
     <xacro:property name="wrist_1_mesh" value="${sec_mesh_files['wrist_1']}"/>
-    <xacro:property name="wrist_1_visual_mesh" value="${wrist_1_mesh['visual']['mesh']}" scope="parent"/>
+    <xacro:property name="wrist_1_visual_mesh" value="file://$(find ${wrist_1_mesh['visual']['mesh']['package']})/${wrist_1_mesh['visual']['mesh']['path']}" scope="parent"/>
     <xacro:property name="wrist_1_visual_material_name" value="${wrist_1_mesh['visual']['material']['name']}" scope="parent"/>
     <xacro:property name="wrist_1_visual_material_color" value="${wrist_1_mesh['visual']['material']['color']}" scope="parent"/>
-    <xacro:property name="wrist_1_collision_mesh" value="${wrist_1_mesh['collision']['mesh']}" scope="parent"/>
+    <xacro:property name="wrist_1_collision_mesh" value="file://$(find ${wrist_1_mesh['collision']['mesh']['package']})/${wrist_1_mesh['collision']['mesh']['path']}" scope="parent"/>
     <xacro:property name="wrist_1_visual_offset" value="${wrist_1_mesh['visual_offset']}" scope="parent"/>
     <xacro:property name="wrist_2_mesh" value="${sec_mesh_files['wrist_2']}"/>
-    <xacro:property name="wrist_2_visual_mesh" value="${wrist_2_mesh['visual']['mesh']}" scope="parent"/>
+    <xacro:property name="wrist_2_visual_mesh" value="file://$(find ${wrist_2_mesh['visual']['mesh']['package']})/${wrist_2_mesh['visual']['mesh']['path']}" scope="parent"/>
     <xacro:property name="wrist_2_visual_material_name" value="${wrist_2_mesh['visual']['material']['name']}" scope="parent"/>
     <xacro:property name="wrist_2_visual_material_color" value="${wrist_2_mesh['visual']['material']['color']}" scope="parent"/>
-    <xacro:property name="wrist_2_collision_mesh" value="${wrist_2_mesh['collision']['mesh']}" scope="parent"/>
+    <xacro:property name="wrist_2_collision_mesh" value="file://$(find ${wrist_2_mesh['collision']['mesh']['package']})/${wrist_2_mesh['collision']['mesh']['path']}" scope="parent"/>
     <xacro:property name="wrist_2_visual_offset" value="${wrist_2_mesh['visual_offset']}" scope="parent"/>
     <xacro:property name="wrist_3_mesh" value="${sec_mesh_files['wrist_3']}"/>
-    <xacro:property name="wrist_3_visual_mesh" value="${wrist_3_mesh['visual']['mesh']}" scope="parent"/>
+    <xacro:property name="wrist_3_visual_mesh" value="file://$(find ${wrist_3_mesh['visual']['mesh']['package']})/${wrist_3_mesh['visual']['mesh']['path']}" scope="parent"/>
     <xacro:property name="wrist_3_visual_material_name" value="${wrist_3_mesh['visual']['material']['name']}" scope="parent"/>
     <xacro:property name="wrist_3_visual_material_color" value="${wrist_3_mesh['visual']['material']['color']}" scope="parent"/>
-    <xacro:property name="wrist_3_collision_mesh" value="${wrist_3_mesh['collision']['mesh']}" scope="parent"/>
+    <xacro:property name="wrist_3_collision_mesh" value="file://$(find ${wrist_3_mesh['collision']['mesh']['package']})/${wrist_3_mesh['collision']['mesh']['path']}" scope="parent"/>
     <xacro:property name="wrist_3_visual_offset" value="${wrist_3_mesh['visual_offset']}" scope="parent"/>
     <!--KINEMATICS HASH-->

Commit message: Remove materials
They were at best unnecessary, with gazebo they were even breaking things

File: urdf/inc/ur_common.xacro (robot description, xacro)
@@ -153,39 +153,25 @@
     <xacro:property name="base_mesh" value="${sec_mesh_files['base']}"/>
     <xacro:property name="base_visual_mesh" value="file://$(find ${base_mesh['visual']['mesh']['package']})/${base_mesh['visual']['mesh']['path']}" scope="parent"/>
-    <xacro:property name="base_visual_material_name" value="${base_mesh['visual']['material']['name']}" scope="parent"/>
-    <xacro:property name="base_visual_material_color" value="${base_mesh['visual']['material']['color']}" scope="parent"/>
     <xacro:property name="base_collision_mesh" value="file://$(find ${base_mesh['collision']['mesh']['package']})/${base_mesh['collision']['mesh']['path']}" scope="parent"/>
     <xacro:property name="shoulder_mesh" value="${sec_mesh_files['shoulder']}"/>
     <xacro:property name="shoulder_visual_mesh" value="file://$(find ${shoulder_mesh['visual']['mesh']['package']})/${shoulder_mesh['visual']['mesh']['path']}" scope="parent"/>
-    <xacro:property name="shoulder_visual_material_name" value="${shoulder_mesh['visual']['material']['name']}" scope="parent"/>
-    <xacro:property name="shoulder_visual_material_color" value="${shoulder_mesh['visual']['material']['color']}" scope="parent"/>
     <xacro:property name="shoulder_collision_mesh" value="file://$(find ${shoulder_mesh['collision']['mesh']['package']})/${shoulder_mesh['collision']['mesh']['path']}" scope="parent"/>
     <xacro:property name="upper_arm_mesh" value="${sec_mesh_files['upper_arm']}"/>
     <xacro:property name="upper_arm_visual_mesh" value="file://$(find ${upper_arm_mesh['visual']['mesh']['package']})/${upper_arm_mesh['visual']['mesh']['path']}" scope="parent"/>
-    <xacro:property name="upper_arm_visual_material_name" value="${upper_arm_mesh['visual']['material']['name']}" scope="parent"/>
-    <xacro:property name="upper_arm_visual_material_color" value="${upper_arm_mesh['visual']['material']['color']}" scope="parent"/>
     <xacro:property name="upper_arm_collision_mesh" value="${upper_arm_mesh['collision']['mesh']}" scope="parent"/>
     <xacro:property name="upper_arm_collision_mesh" value="file://$(find ${upper_arm_mesh['collision']['mesh']['package']})/${upper_arm_mesh['collision']['mesh']['path']}" scope="parent"/>
     <xacro:property name="forearm_mesh" value="${sec_mesh_files['forearm']}"/>
     <xacro:property name="forearm_visual_mesh" value="file://$(find ${forearm_mesh['visual']['mesh']['package']})/${forearm_mesh['visual']['mesh']['path']}" scope="parent"/>
-    <xacro:property name="forearm_visual_material_name" value="${forearm_mesh['visual']['material']['name']}" scope="parent"/>
-    <xacro:property name="forearm_visual_material_color" value="${forearm_mesh['visual']['material']['color']}" scope="parent"/>
     <xacro:property name="forearm_collision_mesh" value="file://$(find ${forearm_mesh['collision']['mesh']['package']})/${forearm_mesh['collision']['mesh']['path']}" scope="parent"/>
     <xacro:property name="wrist_1_mesh" value="${sec_mesh_files['wrist_1']}"/>
     <xacro:property name="wrist_1_visual_mesh" value="file://$(find ${wrist_1_mesh['visual']['mesh']['package']})/${wrist_1_mesh['visual']['mesh']['path']}" scope="parent"/>
-    <xacro:property name="wrist_1_visual_material_name" value="${wrist_1_mesh['visual']['material']['name']}" scope="parent"/>
-    <xacro:property name="wrist_1_visual_material_color" value="${wrist_1_mesh['visual']['material']['color']}" scope="parent"/>
     <xacro:property name="wrist_1_collision_mesh" value="file://$(find ${wrist_1_mesh['collision']['mesh']['package']})/${wrist_1_mesh['collision']['mesh']['path']}" scope="parent"/>
     <xacro:property name="wrist_1_visual_offset" value="${wrist_1_mesh['visual_offset']}" scope="parent"/>
     <xacro:property name="wrist_2_mesh" value="${sec_mesh_files['wrist_2']}"/>
     <xacro:property name="wrist_2_visual_mesh" value="file://$(find ${wrist_2_mesh['visual']['mesh']['package']})/${wrist_2_mesh['visual']['mesh']['path']}" scope="parent"/>
-    <xacro:property name="wrist_2_visual_material_name" value="${wrist_2_mesh['visual']['material']['name']}" scope="parent"/>
-    <xacro:property name="wrist_2_visual_material_color" value="${wrist_2_mesh['visual']['material']['color']}" scope="parent"/>
     <xacro:property name="wrist_2_collision_mesh" value="file://$(find ${wrist_2_mesh['collision']['mesh']['package']})/${wrist_2_mesh['collision']['mesh']['path']}" scope="parent"/>
     <xacro:property name="wrist_2_visual_offset" value="${wrist_2_mesh['visual_offset']}" scope="parent"/>
     <xacro:property name="wrist_3_mesh" value="${sec_mesh_files['wrist_3']}"/>
     <xacro:property name="wrist_3_visual_mesh" value="file://$(find ${wrist_3_mesh['visual']['mesh']['package']})/${wrist_3_mesh['visual']['mesh']['path']}" scope="parent"/>
-    <xacro:property name="wrist_3_visual_material_name" value="${wrist_3_mesh['visual']['material']['name']}" scope="parent"/>
-    <xacro:property name="wrist_3_visual_material_color" value="${wrist_3_mesh['visual']['material']['color']}" scope="parent"/>
     <xacro:property name="wrist_3_collision_mesh" value="file://$(find ${wrist_3_mesh['collision']['mesh']['package']})/${wrist_3_mesh['collision']['mesh']['path']}" scope="parent"/>
     <xacro:property name="wrist_3_visual_offset" value="${wrist_3_mesh['visual_offset']}" scope="parent"/>

File: urdf/ur_macro.xacro (robot description, xacro)
@@ -100,7 +100,4 @@
           <mesh filename="${base_visual_mesh}"/>
         </geometry>
-        <material name="${base_visual_material_name}">
-          <color rgba="${base_visual_material_color}"/>
-        </material>
       </visual>
       <collision>
@@ -120,7 +117,4 @@
           <mesh filename="${shoulder_visual_mesh}"/>
         </geometry>
-        <material name="${shoulder_visual_material_name}">
-          <color rgba="${shoulder_visual_material_color}"/>
-        </material>
       </visual>
       <collision>
@@ -140,7 +134,4 @@
           <mesh filename="${upper_arm_visual_mesh}"/>
         </geometry>
-        <material name="${upper_arm_visual_material_name}">
-          <color rgba="${upper_arm_visual_material_color}"/>
-        </material>
       </visual>
       <collision>
@@ -160,7 +151,4 @@
           <mesh filename="${forearm_visual_mesh}"/>
         </geometry>
-        <material name="${forearm_visual_material_name}">
-          <color rgba="${forearm_visual_material_color}"/>
-        </material>
       </visual>
       <collision>
@@ -180,7 +168,4 @@
           <mesh filename="${wrist_1_visual_mesh}"/>
         </geometry>
-        <material name="${wrist_1_visual_material_name}">
-          <color rgba="${wrist_1_visual_material_color}"/>
-        </material>
       </visual>
       <collision>
@@ -200,7 +185,4 @@
           <mesh filename="${wrist_2_visual_mesh}"/>
         </geometry>
-        <material name="${wrist_2_visual_material_name}">
-          <color rgba="${wrist_2_visual_material_color}"/>
-        </material>
       </visual>
       <collision>
@@ -220,7 +202,4 @@
           <mesh filename="${wrist_3_visual_mesh}"/>
         </geometry>
-        <material name="${wrist_3_visual_material_name}">
-          <color rgba="${wrist_3_visual_material_color}"/>
-        </material>
       </visual>
       <collision>
