Commit message: Set joint dyn properties, optionally from file

File: urdf/inc/ur_common.xacro (robot description, xacro)
@@ -37,5 +37,5 @@
     <mesh filename="${mesh}"/>
   </xacro:macro>
-  <xacro:macro name="read_model_data" params="joint_limits_parameters_file kinematics_parameters_file physical_parameters_file visual_parameters_file force_abs_paths">
+  <xacro:macro name="read_model_data" params="joint_limits_parameters_file kinematics_parameters_file physical_parameters_file visual_parameters_file joint_dynamics_file:=None force_abs_paths">
     <xacro:property name="force_abs_paths" value="${force_abs_paths}" scope="parent"/>
     <!-- Read .yaml files from disk, load content into properties -->
@@ -44,4 +44,5 @@
     <xacro:property name="config_physical_parameters" value="${xacro.load_yaml(physical_parameters_file)}"/>
     <xacro:property name="config_visual_parameters" value="${xacro.load_yaml(visual_parameters_file)}"/>
+    <xacro:property name="config_joint_dynamics" value="${xacro.load_yaml(joint_dynamics_file) if joint_dynamics_file else None}" scope="parent"/>
     <!-- Extract subsections from yaml dictionaries -->
     <xacro:property name="sec_limits" value="${config_joint_limit_parameters['joint_limits']}"/>
@@ -51,4 +52,5 @@
     <xacro:property name="sec_mesh_files" value="${config_visual_parameters['mesh_files']}" scope="parent"/>
     <xacro:property name="sec_kinematics" value="${config_kinematics_parameters['kinematics']}" />
+    <xacro:property name="sec_joint_dynamics" value="${config_joint_dynamics['joint_dynamics'] if joint_dynamics_file else None}" scope="parent"/>
     <!-- JOINTS LIMIT PARAMETERS -->
     <xacro:property name="shoulder_pan_lower_limit" value="${sec_limits['shoulder_pan_joint']['min_position']}" scope="parent"/>
@@ -76,4 +78,17 @@
     <xacro:property name="wrist_3_velocity_limit" value="${sec_limits['wrist_3_joint']['max_velocity']}" scope="parent"/>
     <xacro:property name="wrist_3_effort_limit" value="${sec_limits['wrist_3_joint']['max_effort']}" scope="parent"/>
+    <!-- JOINT DYNAMICS PARAMETERS -->
+    <xacro:property name="shoulder_pan_damping" value="${sec_joint_dynamics['shoulder_pan_joint']['damping'] if sec_joint_dynamics else 0}" scope="parent"/>
+    <xacro:property name="shoulder_pan_friction" value="${sec_joint_dynamics['shoulder_pan_joint']['friction'] if sec_joint_dynamics else 0}" scope="parent"/>
+    <xacro:property name="shoulder_lift_damping" value="${sec_joint_dynamics['shoulder_lift_joint']['damping'] if sec_joint_dynamics else 0}" scope="parent"/>
+    <xacro:property name="shoulder_lift_friction" value="${sec_joint_dynamics['shoulder_lift_joint']['friction'] if sec_joint_dynamics else 0}" scope="parent"/>
+    <xacro:property name="elbow_joint_damping" value="${sec_joint_dynamics['elbow_joint']['damping'] if sec_joint_dynamics else 0}" scope="parent"/>
+    <xacro:property name="elbow_joint_friction" value="${sec_joint_dynamics['elbow_joint']['friction'] if sec_joint_dynamics else 0}" scope="parent"/>
+    <xacro:property name="wrist_1_damping" value="${sec_joint_dynamics['wrist_1_joint']['damping'] if sec_joint_dynamics else 0}" scope="parent"/>
+    <xacro:property name="wrist_1_friction" value="${sec_joint_dynamics['wrist_1_joint']['friction'] if sec_joint_dynamics else 0}" scope="parent"/>
+    <xacro:property name="wrist_2_damping" value="${sec_joint_dynamics['wrist_2_joint']['damping'] if sec_joint_dynamics else 0}" scope="parent"/>
+    <xacro:property name="wrist_2_friction" value="${sec_joint_dynamics['wrist_2_joint']['friction'] if sec_joint_dynamics else 0}" scope="parent"/>
+    <xacro:property name="wrist_3_damping" value="${sec_joint_dynamics['wrist_3_joint']['damping'] if sec_joint_dynamics else 0}" scope="parent"/>
+    <xacro:property name="wrist_3_friction" value="${sec_joint_dynamics['wrist_3_joint']['friction'] if sec_joint_dynamics else 0}" scope="parent"/>
     <!-- DH PARAMETERS -->
     <xacro:property name="d1" value="${sec_dh_parameters['d1']}" scope="parent"/>

Commit message: Pass joint dynamics as default-empty dict()

File: urdf/inc/ur_common.xacro (robot description, xacro)
@@ -37,5 +37,5 @@
     <mesh filename="${mesh}"/>
   </xacro:macro>
-  <xacro:macro name="read_model_data" params="joint_limits_parameters_file kinematics_parameters_file physical_parameters_file visual_parameters_file joint_dynamics_file:=None force_abs_paths">
+  <xacro:macro name="read_model_data" params="joint_limits_parameters_file kinematics_parameters_file physical_parameters_file visual_parameters_file joint_dynamics:=${dict()} force_abs_paths">
     <xacro:property name="force_abs_paths" value="${force_abs_paths}" scope="parent"/>
     <!-- Read .yaml files from disk, load content into properties -->
@@ -44,5 +44,5 @@
     <xacro:property name="config_physical_parameters" value="${xacro.load_yaml(physical_parameters_file)}"/>
     <xacro:property name="config_visual_parameters" value="${xacro.load_yaml(visual_parameters_file)}"/>
-    <xacro:property name="config_joint_dynamics" value="${xacro.load_yaml(joint_dynamics_file) if joint_dynamics_file else None}" scope="parent"/>
+    <xacro:property name="config_joint_dynamics" value="${joint_dynamics}" scope="parent"/>
     <!-- Extract subsections from yaml dictionaries -->
     <xacro:property name="sec_limits" value="${config_joint_limit_parameters['joint_limits']}"/>
@@ -52,5 +52,5 @@
     <xacro:property name="sec_mesh_files" value="${config_visual_parameters['mesh_files']}" scope="parent"/>
     <xacro:property name="sec_kinematics" value="${config_kinematics_parameters['kinematics']}" />
-    <xacro:property name="sec_joint_dynamics" value="${config_joint_dynamics['joint_dynamics'] if joint_dynamics_file else None}" scope="parent"/>
+    <xacro:property name="sec_joint_dynamics" value="${config_joint_dynamics['joint_dynamics'] if joint_dynamics else dict()}" scope="parent"/>
     <!-- JOINTS LIMIT PARAMETERS -->
     <xacro:property name="shoulder_pan_lower_limit" value="${sec_limits['shoulder_pan_joint']['min_position']}" scope="parent"/>

File: urdf/ur.urdf.xacro (robot description, xacro)
@@ -48,4 +48,6 @@
    <!-- create link fixed to the "world" -->
    <link name="world" />
+   <xacro:property name="joint_dynamics_file" value="$(find ur_description)/config/test_joint_dyn.yaml"/>
+   <xacro:property name="joint_dynamics_dict" value="${xacro.load_yaml(joint_dynamics_file)}"/>
    <!-- arm -->
    <xacro:ur_robot
@@ -57,4 +59,5 @@
      physical_parameters_file="$(arg physical_params)"
      visual_parameters_file="$(arg visual_params)"
+     joint_dynamics="${joint_dynamics_dict}"
      transmission_hw_interface="$(arg transmission_hw_interface)"
      safety_limits="$(arg safety_limits)"

File: urdf/ur_macro.xacro (robot description, xacro)
@@ -53,4 +53,5 @@
     physical_parameters_file
     visual_parameters_file
+    joint_dynamics:=${dict()}
     transmission_hw_interface:=hardware_interface/PositionJointInterface
     safety_limits:=false
@@ -86,4 +87,5 @@
       physical_parameters_file="${physical_parameters_file}"
       visual_parameters_file="${visual_parameters_file}"
+      joint_dynamics="${joint_dynamics}"
       force_abs_paths="${sim_gazebo or sim_ignition}"/>
     <!-- ros2 control include -->
@@ -272,5 +274,5 @@
          <safety_controller soft_lower_limit="${shoulder_pan_lower_limit + safety_pos_margin}" soft_upper_limit="${shoulder_pan_upper_limit - safety_pos_margin}" k_position="${safety_k_position}" k_velocity="0.0"/>
       </xacro:if>
-      <dynamics damping="0" friction="0"/>
+      <dynamics damping="${shoulder_pan_damping}" friction="${shoulder_pan_friction}"/>
     </joint>
     <joint name="${prefix}shoulder_lift_joint" type="revolute">
@@ -284,5 +286,5 @@
          <safety_controller soft_lower_limit="${shoulder_lift_lower_limit + safety_pos_margin}" soft_upper_limit="${shoulder_lift_upper_limit - safety_pos_margin}" k_position="${safety_k_position}" k_velocity="0.0"/>
       </xacro:if>
-      <dynamics damping="0" friction="0"/>
+      <dynamics damping="${shoulder_lift_damping}" friction="${shoulder_lift_friction}"/>
     </joint>
     <joint name="${prefix}elbow_joint" type="revolute">
@@ -296,5 +298,5 @@
          <safety_controller soft_lower_limit="${elbow_joint_lower_limit + safety_pos_margin}" soft_upper_limit="${elbow_joint_upper_limit - safety_pos_margin}" k_position="${safety_k_position}" k_velocity="0.0"/>
       </xacro:if>
-      <dynamics damping="0" friction="0"/>
+      <dynamics damping="${elbow_joint_damping}" friction="${elbow_joint_friction}"/>
     </joint>
     <joint name="${prefix}wrist_1_joint" type="revolute">
@@ -308,5 +310,5 @@
          <safety_controller soft_lower_limit="${wrist_1_lower_limit + safety_pos_margin}" soft_upper_limit="${wrist_1_upper_limit - safety_pos_margin}" k_position="${safety_k_position}" k_velocity="0.0"/>
       </xacro:if>
-      <dynamics damping="0" friction="0"/>
+      <dynamics damping="${wrist_1_damping}" friction="${wrist_1_friction}"/>
     </joint>
     <joint name="${prefix}wrist_2_joint" type="revolute">
@@ -320,5 +322,5 @@
          <safety_controller soft_lower_limit="${wrist_2_lower_limit + safety_pos_margin}" soft_upper_limit="${wrist_2_upper_limit - safety_pos_margin}" k_position="${safety_k_position}" k_velocity="0.0"/>
       </xacro:if>
-      <dynamics damping="0" friction="0"/>
+      <dynamics damping="${wrist_2_damping}" friction="${wrist_2_friction}"/>
     </joint>
     <joint name="${prefix}wrist_3_joint" type="revolute">
@@ -332,5 +334,5 @@
          <safety_controller soft_lower_limit="${wrist_3_lower_limit + safety_pos_margin}" soft_upper_limit="${wrist_3_upper_limit - safety_pos_margin}" k_position="${safety_k_position}" k_velocity="0.0"/>
       </xacro:if>
-      <dynamics damping="0" friction="0"/>
+      <dynamics damping="${wrist_3_damping}" friction="${wrist_3_friction}"/>
     </joint>
     <link name="${prefix}ft_frame"/>

Commit message: Mimic initial_positions with dynamics defaults

File: urdf/inc/ur_common.xacro (robot description, xacro)
@@ -37,5 +37,5 @@
     <mesh filename="${mesh}"/>
   </xacro:macro>
-  <xacro:macro name="read_model_data" params="joint_limits_parameters_file kinematics_parameters_file physical_parameters_file visual_parameters_file joint_dynamics:=${dict()} force_abs_paths">
+  <xacro:macro name="read_model_data" params="joint_limits_parameters_file kinematics_parameters_file physical_parameters_file visual_parameters_file joint_dynamics force_abs_paths">
     <xacro:property name="force_abs_paths" value="${force_abs_paths}" scope="parent"/>
     <!-- Read .yaml files from disk, load content into properties -->
@@ -52,5 +52,5 @@
     <xacro:property name="sec_mesh_files" value="${config_visual_parameters['mesh_files']}" scope="parent"/>
     <xacro:property name="sec_kinematics" value="${config_kinematics_parameters['kinematics']}" />
-    <xacro:property name="sec_joint_dynamics" value="${config_joint_dynamics['joint_dynamics'] if joint_dynamics else dict()}" scope="parent"/>
+    <xacro:property name="sec_joint_dynamics" value="${config_joint_dynamics['joint_dynamics']}" scope="parent"/>
     <!-- JOINTS LIMIT PARAMETERS -->
     <xacro:property name="shoulder_pan_lower_limit" value="${sec_limits['shoulder_pan_joint']['min_position']}" scope="parent"/>
@@ -79,16 +79,16 @@
     <xacro:property name="wrist_3_effort_limit" value="${sec_limits['wrist_3_joint']['max_effort']}" scope="parent"/>
     <!-- JOINT DYNAMICS PARAMETERS -->
-    <xacro:property name="shoulder_pan_damping" value="${sec_joint_dynamics['shoulder_pan_joint']['damping'] if sec_joint_dynamics else 0}" scope="parent"/>
-    <xacro:property name="shoulder_pan_friction" value="${sec_joint_dynamics['shoulder_pan_joint']['friction'] if sec_joint_dynamics else 0}" scope="parent"/>
-    <xacro:property name="shoulder_lift_damping" value="${sec_joint_dynamics['shoulder_lift_joint']['damping'] if sec_joint_dynamics else 0}" scope="parent"/>
-    <xacro:property name="shoulder_lift_friction" value="${sec_joint_dynamics['shoulder_lift_joint']['friction'] if sec_joint_dynamics else 0}" scope="parent"/>
-    <xacro:property name="elbow_joint_damping" value="${sec_joint_dynamics['elbow_joint']['damping'] if sec_joint_dynamics else 0}" scope="parent"/>
-    <xacro:property name="elbow_joint_friction" value="${sec_joint_dynamics['elbow_joint']['friction'] if sec_joint_dynamics else 0}" scope="parent"/>
-    <xacro:property name="wrist_1_damping" value="${sec_joint_dynamics['wrist_1_joint']['damping'] if sec_joint_dynamics else 0}" scope="parent"/>
-    <xacro:property name="wrist_1_friction" value="${sec_joint_dynamics['wrist_1_joint']['friction'] if sec_joint_dynamics else 0}" scope="parent"/>
-    <xacro:property name="wrist_2_damping" value="${sec_joint_dynamics['wrist_2_joint']['damping'] if sec_joint_dynamics else 0}" scope="parent"/>
-    <xacro:property name="wrist_2_friction" value="${sec_joint_dynamics['wrist_2_joint']['friction'] if sec_joint_dynamics else 0}" scope="parent"/>
-    <xacro:property name="wrist_3_damping" value="${sec_joint_dynamics['wrist_3_joint']['damping'] if sec_joint_dynamics else 0}" scope="parent"/>
-    <xacro:property name="wrist_3_friction" value="${sec_joint_dynamics['wrist_3_joint']['friction'] if sec_joint_dynamics else 0}" scope="parent"/>
+    <xacro:property name="shoulder_pan_damping" value="${sec_joint_dynamics['shoulder_pan_joint']['damping']}" scope="parent"/>
+    <xacro:property name="shoulder_pan_friction" value="${sec_joint_dynamics['shoulder_pan_joint']['friction']}" scope="parent"/>
+    <xacro:property name="shoulder_lift_damping" value="${sec_joint_dynamics['shoulder_lift_joint']['damping']}" scope="parent"/>
+    <xacro:property name="shoulder_lift_friction" value="${sec_joint_dynamics['shoulder_lift_joint']['friction']}" scope="parent"/>
+    <xacro:property name="elbow_joint_damping" value="${sec_joint_dynamics['elbow_joint']['damping']}" scope="parent"/>
+    <xacro:property name="elbow_joint_friction" value="${sec_joint_dynamics['elbow_joint']['friction']}" scope="parent"/>
+    <xacro:property name="wrist_1_damping" value="${sec_joint_dynamics['wrist_1_joint']['damping']}" scope="parent"/>
+    <xacro:property name="wrist_1_friction" value="${sec_joint_dynamics['wrist_1_joint']['friction']}" scope="parent"/>
+    <xacro:property name="wrist_2_damping" value="${sec_joint_dynamics['wrist_2_joint']['damping']}" scope="parent"/>
+    <xacro:property name="wrist_2_friction" value="${sec_joint_dynamics['wrist_2_joint']['friction']}" scope="parent"/>
+    <xacro:property name="wrist_3_damping" value="${sec_joint_dynamics['wrist_3_joint']['damping']}" scope="parent"/>
+    <xacro:property name="wrist_3_friction" value="${sec_joint_dynamics['wrist_3_joint']['friction']}" scope="parent"/>
     <!-- DH PARAMETERS -->
     <xacro:property name="d1" value="${sec_dh_parameters['d1']}" scope="parent"/>

File: urdf/ur.urdf.xacro (robot description, xacro)
@@ -44,6 +44,9 @@
    <!-- initial position for simulations (Fake Hardware, Gazebo, Ignition) -->
    <xacro:arg name="initial_positions_file" default="$(find ur_description)/config/initial_positions.yaml"/>
+   <!-- Default joint dynamics, useful to specialize for simulations -->
+   <xacro:arg name="joint_dynamics_defaults_file" default="$(find ur_description)/config/joint_dynamics_defaults.yaml"/>
    <!-- convert to property to use substitution in function -->
    <xacro:property name="initial_positions_file" default="$(arg initial_positions_file)"/>
+   <xacro:property name="joint_dynamics_defaults_file" default="$(arg joint_dynamics_defaults_file)"/>
    <!-- create link fixed to the "world" -->
    <link name="world" />
@@ -67,4 +70,5 @@
      headless_mode="$(arg headless_mode)"
      initial_positions="${xacro.load_yaml(initial_positions_file)}"
+     joint_dynamics="${xacro.load_yaml(joint_dynamics_defaults_file)}"
      use_tool_communication="$(arg use_tool_communication)"
      tool_voltage="$(arg tool_voltage)"

File: urdf/ur_macro.xacro (robot description, xacro)
@@ -53,5 +53,4 @@
     physical_parameters_file
     visual_parameters_file
-    joint_dynamics:=${dict()}
     transmission_hw_interface:=hardware_interface/PositionJointInterface
     safety_limits:=false
@@ -64,4 +63,5 @@
     headless_mode:=false
     initial_positions:=${dict(shoulder_pan_joint=0.0,shoulder_lift_joint=-1.57,elbow_joint=0.0,wrist_1_joint=-1.57,wrist_2_joint=0.0,wrist_3_joint=0.0)}
+    joint_dynamics:=${dict(shoulder_pan_joint=dict(damping=0.0, friction=0.0), shoulder_lift_joint=dict(damping=0.0, friction=0.0), elbow_joint=dict(damping=0.0, friction=0.0), wrist_1_joint=dict(damping=0.0, friction=0.0), wrist_2_joint=dict(damping=0.0, friction=0.0), wrist_3_joint=dict(damping=0.0, friction=0.0))}
     use_tool_communication:=false
     tool_voltage:=0

Commit message: Change URDF to reflect ur3(e)'s infinite wrist 3 joint

File: urdf/inc/ur_common.xacro (robot description, xacro)
@@ -71,6 +71,8 @@
     <xacro:property name="wrist_2_velocity_limit" value="${sec_limits['wrist_2_joint']['max_velocity']}" scope="parent"/>
     <xacro:property name="wrist_2_effort_limit" value="${sec_limits['wrist_2_joint']['max_effort']}" scope="parent"/>
-    <xacro:property name="wrist_3_lower_limit" value="${sec_limits['wrist_3_joint']['min_position']}" scope="parent"/>
-    <xacro:property name="wrist_3_upper_limit" value="${sec_limits['wrist_3_joint']['max_position']}" scope="parent"/>
+    <xacro:if value="${sec_limits['wrist_3_joint']['has_position_limits']}">
+      <xacro:property name="wrist_3_lower_limit" value="${sec_limits['wrist_3_joint']['min_position']}" scope="parent"/>
+      <xacro:property name="wrist_3_upper_limit" value="${sec_limits['wrist_3_joint']['max_position']}" scope="parent"/>
+    </xacro:if>
     <xacro:property name="wrist_3_velocity_limit" value="${sec_limits['wrist_3_joint']['max_velocity']}" scope="parent"/>
     <xacro:property name="wrist_3_effort_limit" value="${sec_limits['wrist_3_joint']['max_effort']}" scope="parent"/>

File: urdf/ur_macro.xacro (robot description, xacro)
@@ -64,4 +64,6 @@
       visual_parameters_file="${visual_parameters_file}"
       force_abs_paths="${force_abs_paths}"/>
+    <xacro:property name="config_joint_limit_parameters" value="${xacro.load_yaml(joint_limits_parameters_file)}"/>
+    <xacro:property name="sec_limits" value="${config_joint_limit_parameters['joint_limits']}"/>
     <!-- links -  main serial chain -->
     <link name="${tf_prefix}base_link"/>
@@ -318,16 +320,31 @@
       <dynamics damping="0" friction="0"/>
     </joint>
-    <joint name="${tf_prefix}wrist_3_joint" type="revolute">
-      <parent link="${tf_prefix}wrist_2_link" />
-      <child link="${tf_prefix}wrist_3_link" />
-      <origin xyz="${wrist_3_x} ${wrist_3_y} ${wrist_3_z}" rpy="${wrist_3_roll} ${wrist_3_pitch} ${wrist_3_yaw}" />
-      <axis xyz="0 0 1" />
-      <limit lower="${wrist_3_lower_limit}" upper="${wrist_3_upper_limit}"
-             effort="${wrist_3_effort_limit}" velocity="${wrist_3_velocity_limit}"/>
-      <xacro:if value="${safety_limits}">
-         <safety_controller soft_lower_limit="${wrist_3_lower_limit + safety_pos_margin}" soft_upper_limit="${wrist_3_upper_limit - safety_pos_margin}" k_position="${safety_k_position}" k_velocity="0.0"/>
-      </xacro:if>
-      <dynamics damping="0" friction="0"/>
-    </joint>
+    <xacro:if value="${sec_limits['wrist_3_joint']['has_position_limits']}">
+      <joint name="${tf_prefix}wrist_3_joint" type="revolute">
+        <parent link="${tf_prefix}wrist_2_link" />
+        <child link="${tf_prefix}wrist_3_link" />
+        <origin xyz="${wrist_3_x} ${wrist_3_y} ${wrist_3_z}" rpy="${wrist_3_roll} ${wrist_3_pitch} ${wrist_3_yaw}" />
+        <axis xyz="0 0 1" />
+        <limit lower="${wrist_3_lower_limit}" upper="${wrist_3_upper_limit}"
+              effort="${wrist_3_effort_limit}" velocity="${wrist_3_velocity_limit}"/>
+        <xacro:if value="${safety_limits}">
+          <safety_controller soft_lower_limit="${wrist_3_lower_limit + safety_pos_margin}" soft_upper_limit="${wrist_3_upper_limit - safety_pos_margin}" k_position="${safety_k_position}" k_velocity="0.0"/>
+        </xacro:if>
+        <dynamics damping="0" friction="0"/>
+      </joint>
+    </xacro:if>
+    <xacro:unless value="${sec_limits['wrist_3_joint']['has_position_limits']}">
+      <joint name="${tf_prefix}wrist_3_joint" type="continuous">
+        <parent link="${tf_prefix}wrist_2_link" />
+        <child link="${tf_prefix}wrist_3_link" />
+        <origin xyz="${wrist_3_x} ${wrist_3_y} ${wrist_3_z}" rpy="${wrist_3_roll} ${wrist_3_pitch} ${wrist_3_yaw}" />
+        <axis xyz="0 0 1" />
+        <limit effort="${wrist_3_effort_limit}" velocity="${wrist_3_velocity_limit}"/>
+        <xacro:if value="${safety_limits}">
+          <safety_controller k_position="${safety_k_position}" k_velocity="0.0"/>
+        </xacro:if>
+        <dynamics damping="0" friction="0"/>
+      </joint>
+    </xacro:unless>
     <link name="${tf_prefix}ft_frame"/>
     <joint name="${tf_prefix}wrist_3_link-ft_frame" type="fixed">

Commit message: Remove unused dh_parameters

File: urdf/inc/ur_common.xacro (robot description, xacro)
@@ -46,5 +46,4 @@
     <!-- Extract subsections from yaml dictionaries -->
     <xacro:property name="sec_limits" value="${config_joint_limit_parameters['joint_limits']}"/>
-    <xacro:property name="sec_dh_parameters" value="${config_physical_parameters['dh_parameters']}"/>
     <xacro:property name="sec_offsets" value="${config_physical_parameters['offsets']}"/>
     <xacro:property name="sec_inertia_parameters" value="${config_physical_parameters['inertia_parameters']}" />
@@ -76,11 +75,4 @@
     <xacro:property name="wrist_3_velocity_limit" value="${sec_limits['wrist_3_joint']['max_velocity']}" scope="parent"/>
     <xacro:property name="wrist_3_effort_limit" value="${sec_limits['wrist_3_joint']['max_effort']}" scope="parent"/>
-    <!-- DH PARAMETERS -->
-    <xacro:property name="d1" value="${sec_dh_parameters['d1']}" scope="parent"/>
-    <xacro:property name="a2" value="${sec_dh_parameters['a2']}" scope="parent"/>
-    <xacro:property name="a3" value="${sec_dh_parameters['a3']}" scope="parent"/>
-    <xacro:property name="d4" value="${sec_dh_parameters['d4']}" scope="parent"/>
-    <xacro:property name="d5" value="${sec_dh_parameters['d5']}" scope="parent"/>
-    <xacro:property name="d6" value="${sec_dh_parameters['d6']}" scope="parent"/>
     <!-- kinematics -->
     <xacro:property name="shoulder_x" value="${sec_kinematics['shoulder']['x']}" scope="parent"/>
